File: Hardware/Boards/heatingHeader.brd (EAGLE design)
At the start: 45.4 x 30.5 mm, 26 parts, among them IC1 DS1820

Commit message: a
Parts:
- removed R6: 8.2, resistor:R6332
- R5: value 100 -> 1K
- moved PAD6 3.81 mm to (20.3, 3.81)
- moved PAD7 3.81 mm to (24.1, 3.81)
Connections:
- removed net N$11: PAD6.1, R7.1, U$2.15
- removed net N$17: JP2.2, PAD1.1, R6.1, U$1.VDD, U$2.1
- new net N$9: PAD6.1, R7.1, U$2.2
- net N$1: now also U$2.8; no longer U$2.2
- net N$2: now also JP2.2, PAD1.1, U$1.VDD, U$2.1; no longer R6.2
- net N$28: no longer U$2.10
- net N$3: now also U$2.15; no longer U$2.3
Changed lines of the file:
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@@
 <element name="PAD4" library="wirepad" package="5-2,5" value="WIREPADSMD5-2,5" x="38.1" y="3.81" rot="MR0"/>
 <element name="PAD5" library="wirepad" package="5-2,5" value="WIREPADSMD5-2,5" x="27.94" y="3.81" rot="MR0"/>
-<element name="R5" library="resistor" package="R1206" value="100" x="-20.32" y="43.18"/>
-<element name="R6" library="resistor" package="R6332" value="8.2" x="-25.4" y="43.18"/>
-<element name="PAD6" library="wirepad" package="5-2,5" value="WIREPADSMD5-2,5" x="24.13" y="3.81" rot="MR0"/>
-<element name="PAD7" library="wirepad" package="5-2,5" value="WIREPADSMD5-2,5" x="20.32" y="3.81" rot="MR0"/>
+<element name="R5" library="resistor" package="R1206" value="1K" x="-20.32" y="43.18"/>
+<element name="PAD6" library="wirepad" package="5-2,5" value="WIREPADSMD5-2,5" x="20.32" y="3.81" rot="MR0"/>
+<element name="PAD7" library="wirepad" package="5-2,5" value="WIREPADSMD5-2,5" x="24.13" y="3.81" rot="MR0"/>
 <element name="R7" library="resistor" package="R1206" value="100 K" x="-33.02" y="36.83"/>
 </elements>
@@
 <wire x1="6.25" y1="9.22" x2="21.205" y2="14.155" width="0" layer="19" extent="1-1"/>
 <wire x1="43.18" y1="26.67" x2="21.205" y2="14.155" width="0" layer="19" extent="1-1"/>
-<wire x1="20.32" y1="3.81" x2="43.18" y2="26.67" width="0" layer="19" extent="1-1"/>
-<wire x1="-29.53" y1="42.08" x2="20.32" y2="3.81" width="0" layer="19" extent="1-1"/>
+<wire x1="24.13" y1="3.81" x2="43.18" y2="26.67" width="0" layer="19" extent="1-1"/>
+<wire x1="-29.53" y1="42.08" x2="24.13" y2="3.81" width="0" layer="19" extent="1-1"/>
 <wire x1="-34.61" y1="42.08" x2="-29.53" y2="42.08" width="0" layer="19" extent="1-1"/>
-<wire x1="40.64" y1="15.24" x2="20.32" y2="3.81" width="0" layer="19" extent="1-1"/>
+<wire x1="40.64" y1="15.24" x2="24.13" y2="3.81" width="0" layer="19" extent="1-1"/>
 <wire x1="-19.59" y1="21.59" x2="40.64" y2="15.24" width="0" layer="19" extent="1-1"/>
 <wire x1="34.29" y1="2.54" x2="-29.53" y2="42.08" width="0" layer="19" extent="1-1"/>
-</signal>
-<signal name="N$17">
-<contactref element="U$2" pad="1"/>
-<contactref element="U$1" pad="VDD"/>
-<contactref element="JP2" pad="2"/>
-<contactref element="PAD1" pad="1"/>
-<contactref element="R6" pad="1"/>
-<wire x1="7.55" y1="9.22" x2="21.205" y2="21.405" width="0" layer="19" extent="1-1"/>
-<wire x1="40.64" y1="12.7" x2="7.55" y2="9.22" width="0" layer="19" extent="1-1"/>
-<wire x1="2.54" y1="26.67" x2="40.64" y2="12.7" width="0" layer="19" extent="1-1"/>
-<wire x1="-28.2" y1="43.18" x2="2.54" y2="26.67" width="0" layer="19" extent="1-1"/>
 </signal>
 <signal name="N$18">
@@
 <signal name="N$28">
 <contactref element="R5" pad="2"/>
-<contactref element="U$2" pad="10"/>
 <contactref element="U$2" pad="12"/>
 <contactref element="R7" pad="2"/>
-<wire x1="26.405" y1="14.155" x2="27.055" y2="21.405" width="0" layer="19" extent="1-1"/>
-<wire x1="-31.598" y1="36.83" x2="26.405" y2="14.155" width="0" layer="19" extent="1-1"/>
-<wire x1="-18.898" y1="43.18" x2="-31.598" y2="36.83" width="0" layer="19" extent="1-1"/>
+<wire x1="-18.898" y1="43.18" x2="26.405" y2="14.155" width="0" layer="19" extent="1-16"/>
+<wire x1="-31.598" y1="36.83" x2="-18.898" y2="43.18" width="0" layer="19" extent="1-1"/>
 </signal>
 <signal name="N$30">
@@
 <contactref element="R4" pad="2"/>
 <contactref element="U$2" pad="5"/>
-<wire x1="-44.602" y1="36.83" x2="23.805" y2="21.405" width="0" layer="19" extent="1-1"/>
-<wire x1="-13.818" y1="43.18" x2="-44.602" y2="36.83" width="0" layer="19" extent="1-1"/>
+<wire x1="-13.818" y1="43.18" x2="23.805" y2="21.405" width="0" layer="19" extent="1-16"/>
+<wire x1="-44.602" y1="36.83" x2="-13.818" y2="43.18" width="0" layer="19" extent="1-1"/>
 </signal>
 <signal name="N$3">
 <contactref element="IC1" pad="3"/>
-<contactref element="U$2" pad="3"/>
-<wire x1="31.75" y1="2.54" x2="22.505" y2="21.405" width="0" layer="19" extent="1-1"/>
+<contactref element="U$2" pad="15"/>
+<wire x1="31.75" y1="2.54" x2="24.455" y2="14.155" width="0" layer="19" extent="16-16"/>
 </signal>
 <signal name="N$1">
 <contactref element="IC1" pad="2"/>
-<contactref element="U$2" pad="2"/>
-<wire x1="33.02" y1="4.445" x2="21.855" y2="21.405" width="0" layer="19" extent="1-1"/>
+<contactref element="U$2" pad="8"/>
+<wire x1="33.02" y1="4.445" x2="25.755" y2="21.405" width="0" layer="19" extent="16-16"/>
 </signal>
 <signal name="N$7">
@@
 <contactref element="D4" pad="C"/>
 <contactref element="T3" pad="E"/>
-<contactref element="R6" pad="2"/>
 <contactref element="U$2" pad="7"/>
-<wire x1="-35.02" y1="21.59" x2="25.105" y2="21.405" width="0" layer="19" extent="1-1"/>
+<contactref element="U$2" pad="1"/>
+<contactref element="U$1" pad="VDD"/>
+<contactref element="JP2" pad="2"/>
+<contactref element="PAD1" pad="1"/>
+<wire x1="25.105" y1="21.405" x2="40.64" y2="12.7" width="0" layer="19" extent="16-16"/>
+<wire x1="21.205" y1="21.405" x2="25.105" y2="21.405" width="0" layer="19" extent="16-16"/>
+<wire x1="7.55" y1="9.22" x2="21.205" y2="21.405" width="0" layer="19" extent="16-16"/>
+<wire x1="2.54" y1="26.67" x2="7.55" y2="9.22" width="0" layer="19" extent="1-16"/>
+<wire x1="-35.02" y1="21.59" x2="2.54" y2="26.67" width="0" layer="19" extent="1-1"/>
 <wire x1="-46.45" y1="21.59" x2="-35.02" y2="21.59" width="0" layer="19" extent="1-1"/>
 <wire x1="-44.77" y1="42.08" x2="-46.45" y2="21.59" width="0" layer="19" extent="1-1"/>
 <wire x1="-39.69" y1="42.08" x2="-44.77" y2="42.08" width="0" layer="19" extent="1-1"/>
-<wire x1="-22.6" y1="43.18" x2="-39.69" y2="42.08" width="0" layer="19" extent="1-1"/>
 </signal>
 <signal name="N$6">
@@
 <wire x1="14.05" y1="9.22" x2="25.755" y2="14.155" width="0" layer="19" extent="1-1"/>
 </signal>
-<signal name="N$11">
+<signal name="N$9">
+<contactref element="U$2" pad="2"/>
 <contactref element="R7" pad="1"/>
 <contactref element="PAD6" pad="1"/>
-<contactref element="U$2" pad="15"/>
-<wire x1="-34.442" y1="36.83" x2="24.455" y2="14.155" width="0" layer="19" extent="1-1"/>
-<wire x1="24.13" y1="3.81" x2="-34.442" y2="36.83" width="0" layer="19" extent="1-1"/>
+<wire x1="20.32" y1="3.81" x2="21.855" y2="21.405" width="0" layer="19" extent="16-16"/>
+<wire x1="-34.442" y1="36.83" x2="21.855" y2="21.405" width="0" layer="19" extent="1-16"/>
 </signal>
 </signals>

Commit message: a
Parts:
- added S1: (no value), switch-dil:SD4-01
- moved U$2 8.03 mm to (31.8, 15.2)
Connections:
- new net N$10: S1.2, U$2.3
- net N$5: now also S1.1
Changed lines of the file:
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@@
 <elements>
 <element name="U$1" library="rfm70" package="RFM70" value="RFM70" x="6.35" y="-5.08" rot="MR180"/>
-<element name="U$2" library="microchip" package="SSOP20" value="PIC16F690" x="24.13" y="17.78" rot="MR180"/>
+<element name="U$2" library="microchip" package="SSOP20" value="PIC16F690" x="31.75" y="15.24" rot="MR180"/>
 <element name="JP2" library="pinhead" package="1X05" value="Prog" x="40.64" y="15.24" rot="MR90"/>
 <element name="IC1" library="ds1820" package="TO-92" value="DS1820" x="33.02" y="2.54" rot="MR0"/>
@@
 <element name="PAD7" library="wirepad" package="5-2,5" value="WIREPADSMD5-2,5" x="24.13" y="3.81" rot="MR0"/>
 <element name="R7" library="resistor" package="R1206" value="100 K" x="-33.02" y="36.83"/>
+<element name="S1" library="switch-dil" package="SD4-01" value="" x="21.59" y="16.51">
+<attribute name="OC_NEWARK" value="unknown" x="21.59" y="16.51" size="1.778" layer="27" display="off"/>
+<attribute name="MPN" value="" x="21.59" y="16.51" size="1.778" layer="27" display="off"/>
+<attribute name="MF" value="" x="21.59" y="16.51" size="1.778" layer="27" display="off"/>
+<attribute name="OC_FARNELL" value="unknown" x="21.59" y="16.51" size="1.778" layer="27" display="off"/>
+</element>
 </elements>
 <signals>
@@
 <contactref element="PAD2" pad="1"/>
 <contactref element="PAD7" pad="1"/>
-<wire x1="21.205" y1="14.155" x2="-46.26" y2="5.08" width="0" layer="19" extent="1-1"/>
-<wire x1="6.25" y1="9.22" x2="21.205" y2="14.155" width="0" layer="19" extent="1-1"/>
-<wire x1="43.18" y1="26.67" x2="21.205" y2="14.155" width="0" layer="19" extent="1-1"/>
-<wire x1="24.13" y1="3.81" x2="43.18" y2="26.67" width="0" layer="19" extent="1-1"/>
-<wire x1="-29.53" y1="42.08" x2="24.13" y2="3.81" width="0" layer="19" extent="1-1"/>
+<contactref element="S1" pad="1"/>
+<wire x1="40.64" y1="15.24" x2="43.18" y2="26.67" width="0" layer="19" extent="1-1"/>
+<wire x1="34.29" y1="2.54" x2="40.64" y2="15.24" width="0" layer="19" extent="1-1"/>
+<wire x1="24.13" y1="3.81" x2="34.29" y2="2.54" width="0" layer="19" extent="16-16"/>
+<wire x1="28.825" y1="11.615" x2="24.13" y2="3.81" width="0" layer="19" extent="16-16"/>
+<wire x1="6.25" y1="9.22" x2="28.825" y2="11.615" width="0" layer="19" extent="16-16"/>
+<wire x1="-19.59" y1="21.59" x2="6.25" y2="9.22" width="0" layer="19" extent="1-16"/>
+<wire x1="-29.53" y1="42.08" x2="-19.59" y2="21.59" width="0" layer="19" extent="1-1"/>
 <wire x1="-34.61" y1="42.08" x2="-29.53" y2="42.08" width="0" layer="19" extent="1-1"/>
-<wire x1="40.64" y1="15.24" x2="24.13" y2="3.81" width="0" layer="19" extent="1-1"/>
-<wire x1="-19.59" y1="21.59" x2="40.64" y2="15.24" width="0" layer="19" extent="1-1"/>
-<wire x1="34.29" y1="2.54" x2="-29.53" y2="42.08" width="0" layer="19" extent="1-1"/>
+<wire x1="-46.26" y1="5.08" x2="-19.59" y2="21.59" width="0" layer="19" extent="1-1"/>
+<wire x1="21.59" y1="12.7" x2="-46.26" y2="5.08" width="0" layer="19" extent="1-1"/>
 </signal>
 <signal name="N$18">
 <contactref element="U$2" pad="19"/>
 <contactref element="JP2" pad="4"/>
-<wire x1="40.64" y1="17.78" x2="21.855" y2="14.155" width="0" layer="19" extent="1-1"/>
+<wire x1="40.64" y1="17.78" x2="29.475" y2="11.615" width="0" layer="19" extent="1-1"/>
 </signal>
 <signal name="N$19">
 <contactref element="U$2" pad="18"/>
 <contactref element="JP2" pad="5"/>
-<wire x1="40.64" y1="20.32" x2="22.505" y2="14.155" width="0" layer="19" extent="1-1"/>
+<wire x1="40.64" y1="20.32" x2="30.125" y2="11.615" width="0" layer="19" extent="1-1"/>
 </signal>
 <signal name="N$16">
 <contactref element="U$2" pad="17"/>
 <contactref element="U$1" pad="CE"/>
-<wire x1="8.85" y1="9.22" x2="23.155" y2="14.155" width="0" layer="19" extent="1-1"/>
+<wire x1="8.85" y1="9.22" x2="30.775" y2="11.615" width="0" layer="19" extent="1-1"/>
 </signal>
 <signal name="N$20">
 <contactref element="U$2" pad="16"/>
 <contactref element="U$1" pad="CSN"/>
-<wire x1="10.15" y1="9.22" x2="23.805" y2="14.155" width="0" layer="19" extent="1-1"/>
+<wire x1="10.15" y1="9.22" x2="31.425" y2="11.615" width="0" layer="19" extent="1-1"/>
 </signal>
 <signal name="N$21">
 <contactref element="U$2" pad="14"/>
 <contactref element="U$1" pad="IRQ"/>
-<wire x1="15.35" y1="9.22" x2="25.105" y2="14.155" width="0" layer="19" extent="1-1"/>
+<wire x1="15.35" y1="9.22" x2="32.725" y2="11.615" width="0" layer="19" extent="1-1"/>
 </signal>
 <signal name="N$22">
 <contactref element="U$2" pad="11"/>
 <contactref element="U$1" pad="SCK"/>
-<wire x1="11.45" y1="9.22" x2="27.055" y2="14.155" width="0" layer="19" extent="1-1"/>
+<wire x1="11.45" y1="9.22" x2="34.675" y2="11.615" width="0" layer="19" extent="1-1"/>
 </signal>
 <signal name="N$23">
 <contactref element="U$2" pad="9"/>
 <contactref element="U$1" pad="MOSI"/>
-<wire x1="12.75" y1="9.22" x2="26.405" y2="21.405" width="0" layer="19" extent="1-1"/>
+<wire x1="12.75" y1="9.22" x2="34.025" y2="18.865" width="0" layer="19" extent="1-1"/>
 </signal>
 <signal name="N$25">
 <contactref element="U$2" pad="4"/>
 <contactref element="JP2" pad="1"/>
-<wire x1="40.64" y1="10.16" x2="23.155" y2="21.405" width="0" layer="19" extent="1-1"/>
+<wire x1="40.64" y1="10.16" x2="30.775" y2="18.865" width="0" layer="19" extent="1-1"/>
 </signal>
 <signal name="N$28">
@@
 <contactref element="U$2" pad="12"/>
 <contactref element="R7" pad="2"/>
-<wire x1="-18.898" y1="43.18" x2="26.405" y2="14.155" width="0" layer="19" extent="1-16"/>
+<wire x1="-18.898" y1="43.18" x2="34.025" y2="11.615" width="0" layer="19" extent="1-16"/>
 <wire x1="-31.598" y1="36.83" x2="-18.898" y2="43.18" width="0" layer="19" extent="1-1"/>
 </signal>
@@
 <contactref element="R1" pad="1"/>
 <contactref element="R3" pad="2"/>
-<wire x1="-39.522" y1="36.83" x2="24.455" y2="21.405" width="0" layer="19" extent="1-1"/>
+<wire x1="-39.522" y1="36.83" x2="32.075" y2="18.865" width="0" layer="19" extent="1-1"/>
 <wire x1="-46.838" y1="36.83" x2="-39.522" y2="36.83" width="0" layer="19" extent="1-1"/>
 </signal>
@@
 <contactref element="R4" pad="2"/>
 <contactref element="U$2" pad="5"/>
-<wire x1="-13.818" y1="43.18" x2="23.805" y2="21.405" width="0" layer="19" extent="1-16"/>
+<wire x1="-13.818" y1="43.18" x2="31.425" y2="18.865" width="0" layer="19" extent="1-16"/>
 <wire x1="-44.602" y1="36.83" x2="-13.818" y2="43.18" width="0" layer="19" extent="1-1"/>
 </signal>
@@
 <contactref element="IC1" pad="3"/>
 <contactref element="U$2" pad="15"/>
-<wire x1="31.75" y1="2.54" x2="24.455" y2="14.155" width="0" layer="19" extent="16-16"/>
+<wire x1="31.75" y1="2.54" x2="32.075" y2="11.615" width="0" layer="19" extent="16-16"/>
 </signal>
 <signal name="N$1">
 <contactref element="IC1" pad="2"/>
 <contactref element="U$2" pad="8"/>
-<wire x1="33.02" y1="4.445" x2="25.755" y2="21.405" width="0" layer="19" extent="16-16"/>
+<wire x1="33.02" y1="4.445" x2="33.375" y2="18.865" width="0" layer="19" extent="16-16"/>
 </signal>
 <signal name="N$7">
@@
 <contactref element="JP2" pad="2"/>
 <contactref element="PAD1" pad="1"/>
-<wire x1="25.105" y1="21.405" x2="40.64" y2="12.7" width="0" layer="19" extent="16-16"/>
-<wire x1="21.205" y1="21.405" x2="25.105" y2="21.405" width="0" layer="19" extent="16-16"/>
-<wire x1="7.55" y1="9.22" x2="21.205" y2="21.405" width="0" layer="19" extent="16-16"/>
+<wire x1="32.725" y1="18.865" x2="40.64" y2="12.7" width="0" layer="19" extent="16-16"/>
+<wire x1="28.825" y1="18.865" x2="32.725" y2="18.865" width="0" layer="19" extent="16-16"/>
+<wire x1="7.55" y1="9.22" x2="28.825" y2="18.865" width="0" layer="19" extent="16-16"/>
 <wire x1="2.54" y1="26.67" x2="7.55" y2="9.22" width="0" layer="19" extent="1-16"/>
 <wire x1="-35.02" y1="21.59" x2="2.54" y2="26.67" width="0" layer="19" extent="1-1"/>
@@
 <contactref element="U$1" pad="MISO"/>
 <contactref element="U$2" pad="13"/>
-<wire x1="14.05" y1="9.22" x2="25.755" y2="14.155" width="0" layer="19" extent="1-1"/>
+<wire x1="14.05" y1="9.22" x2="33.375" y2="11.615" width="0" layer="19" extent="1-1"/>
 </signal>
 <signal name="N$9">
@@
 <contactref element="R7" pad="1"/>
 <contactref element="PAD6" pad="1"/>
-<wire x1="20.32" y1="3.81" x2="21.855" y2="21.405" width="0" layer="19" extent="16-16"/>
-<wire x1="-34.442" y1="36.83" x2="21.855" y2="21.405" width="0" layer="19" extent="1-16"/>
+<wire x1="20.32" y1="3.81" x2="29.475" y2="18.865" width="0" layer="19" extent="16-16"/>
+<wire x1="-34.442" y1="36.83" x2="29.475" y2="18.865" width="0" layer="19" extent="1-16"/>
+</signal>
+<signal name="N$10">
+<contactref element="S1" pad="2"/>
+<contactref element="U$2" pad="3"/>
+<wire x1="30.125" y1="18.865" x2="21.59" y2="20.32" width="0" layer="19" extent="16-16"/>
 </signal>
 </signals>
