File: Hardware/Boards/rolety.brd (EAGLE design)
At the start: 23.8 x 45.7 mm, 28 parts, among them IC1 LNK304, IC2 MCP1703DB, K2 FRS1B, K3 FRS1B, T1 BC846, T2 BC846

Commit message: a
Parts:
- added S1: (no value), switch-dil:SD4-01
- moved L1 15.7 mm to (16.0, 38.1)
- moved T2 14.9 mm to (3.71, 24.5)
- moved D4 13.9 mm to (1.54, 35.4)
- moved C1 6.30 mm to (7.20, 29.3)
- moved D3 6.12 mm to (4.98, 37.1), turned to 270 degrees
- moved T1 4.82 mm to (3.30, 29.5)
- moved IC2 4.54 mm to (13.4, 26.0), turned to 270 degrees
- moved C2 3.69 mm to (9.85, 35.8)
- moved U$1 3.31 mm to (26.6, 33.5)
- moved U$2 2.10 mm to (17.0, 34.8)
- moved JP2 1.24 mm to (16.7, 42.0)
- moved IC1 1.12 mm to (21.2, 26.1)
- moved C3 0.93 mm to (21.3, 2.54)
- moved C4 0.68 mm to (15.9, 2.54)
- moved JP1 0.50 mm to (6.77, 2.79)
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Connections:
- net N$33: now also S1.2
- net N$5: now also S1.1
Other:
- board size 23.8 x 45.7 mm -> 23.8 x 43.8 mm
