File: Hardware/Boards/spinac.brd (EAGLE design)
At the start: 56.8 x 22.9 mm, 26 parts, among them IC1 LNK304, IC2 MCP1703DB, IC4 DS1820, K1 G5L, T1 BC846

Commit message: a
Parts:
- moved JP2 39.6 mm to (6.35, 27.9)
- moved IC4 22.6 mm to (39.4, 3.81)
- moved U$2 21.6 mm to (29.2, 8.89)
- moved U$1 21.3 mm to (34.3, -3.81)
- moved L1 20.5 mm to (21.6, 27.9), turned to 180 degrees
- moved C4 20.5 mm to (2.54, 2.54)
- moved JP1 17.7 mm to (40.6, 14.0), turned to 270 degrees
- moved IC1 15.7 mm to (33.0, 26.7)
- moved B1 11.5 mm to (39.4, 25.4)
- moved C1 10.2 mm to (30.5, 19.1), turned to 0 degrees
- moved K1 4.58 mm to (14.0, 11.4), turned to 270 degrees
- moved C3 4.58 mm to (2.54, 22.9)
- moved IC2 3.59 mm to (14.0, 12.7), turned to 90 degrees
Other:
- board size 56.8 x 22.9 mm -> 42.9 x 30.5 mm

Commit message: a
Parts:
- added S1: (no value), switch-dil:SD4-01
- moved JP1 38.6 mm to (2.18, 10.9)
- moved C4 37.1 mm to (33.0, 23.7)
- moved IC4 36.7 mm to (2.76, 1.01), turned to 0 degrees
- moved B1 29.5 mm to (12.3, 13.6)
- moved L1 18.6 mm to (37.7, 18.6), turned to 270 degrees
- moved JP3 14.8 mm to (3.96, 24.9), turned to 180 degrees
- moved U$2 13.2 mm to (26.6, 21.8)
- moved U$1 10.9 mm to (23.5, -2.39), flipped to the bottom
- moved IC1 8.49 mm to (36.6, 19.0)
- moved JP2 8.36 mm to (14.1, 24.9)
- moved IC2 8.27 mm to (13.4, 4.45)
- moved T1 6.33 mm to (6.88, 13.2)
- moved C1 4.21 mm to (28.7, 15.2)
- moved C3 2.40 mm to (2.54, 20.5), turned to 270 degrees
- moved K1 1.03 mm to (13.4, 10.5)
Connections:
- net N$33: now also S1.2
- net N$5: now also S1.1
Other:
- board size 42.9 x 30.5 mm -> 39.8 x 26.5 mm
