File: Hardware/Boards/tempThermostat.brd (EAGLE design)
At the start: 30.1 x 20.3 mm, 21 parts, among them IC1 DS1820

Commit message: a
Parts:
- added S1: (no value), switch-dil:SD4-01
- moved U$2 42.8 mm to (8.89, 14.0), flipped to the bottom
- moved JP1 1.27 mm to (25.4, 17.8)
Connections:
- new net N$6: S1.2, U$2.3
- net N$5: now also S1.1
Changed lines of the file:
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@@
 <elements>
 <element name="U$1" library="rfm70" package="RFM70" value="RFM70" x="6.35" y="24.13"/>
-<element name="U$2" library="microchip" package="SSOP20" value="PIC16F690" x="-33.02" y="5.08"/>
+<element name="U$2" library="microchip" package="SSOP20" value="PIC16F690" x="8.89" y="13.97" rot="MR0"/>
 <element name="JP2" library="pinhead" package="1X05" value="Prog" x="2.54" y="12.7" rot="R90"/>
 <element name="IC1" library="ds1820" package="TO-92" value="DS1820" x="27.94" y="8.89" rot="R90"/>
 <element name="LSP1" library="solpad" package="LSP11" value="LSP11" x="15.24" y="2.54"/>
 <element name="LSP2" library="solpad" package="LSP11" value="LSP11" x="2.54" y="2.54"/>
-<element name="JP1" library="pinhead" package="1X03" value="" x="25.4" y="16.51"/>
+<element name="JP1" library="pinhead" package="1X03" value="" x="25.4" y="17.78"/>
 <element name="T1" library="transistor" package="SOT23-BEC" value="" x="-39.37" y="27.94"/>
 <element name="T2" library="transistor" package="SOT23-BEC" value="" x="-15.24" y="34.29"/>
@@
 <element name="D3" library="diode" package="SMA" value="MBRA340T3" x="-40.64" y="-21.59"/>
 <element name="D4" library="diode" package="SMA" value="MBRA340T3" x="-40.64" y="-30.48"/>
+<element name="S1" library="switch-dil" package="SD4-01" value="" x="8.89" y="5.08" rot="R90">
+<attribute name="OC_NEWARK" value="unknown" x="8.89" y="5.08" size="1.778" layer="27" rot="R90" display="off"/>
+<attribute name="MPN" value="" x="8.89" y="5.08" size="1.778" layer="27" rot="R90" display="off"/>
+<attribute name="MF" value="" x="8.89" y="5.08" size="1.778" layer="27" rot="R90" display="off"/>
+<attribute name="OC_FARNELL" value="unknown" x="8.89" y="5.08" size="1.778" layer="27" rot="R90" display="off"/>
+</element>
 </elements>
 <signals>
@@
 <contactref element="D2" pad="A"/>
 <contactref element="D1" pad="A"/>
+<contactref element="S1" pad="1"/>
+<wire x1="-38.64" y1="-12.7" x2="12.7" y2="5.08" width="0" layer="19" extent="1-1"/>
 <wire x1="-38.64" y1="-3.81" x2="-38.64" y2="-12.7" width="0" layer="19" extent="1-1"/>
-<wire x1="-35.945" y1="8.705" x2="-38.64" y2="-3.81" width="0" layer="19" extent="1-1"/>
-<wire x1="-38.42" y1="26.84" x2="-35.945" y2="8.705" width="0" layer="19" extent="1-1"/>
+<wire x1="11.815" y1="17.595" x2="-38.64" y2="-3.81" width="0" layer="19" extent="1-1"/>
+<wire x1="-38.42" y1="26.84" x2="11.815" y2="17.595" width="0" layer="19" extent="1-1"/>
 <wire x1="-14.29" y1="33.19" x2="-38.42" y2="26.84" width="0" layer="19" extent="1-1"/>
 <wire x1="2.54" y1="12.7" x2="-14.29" y2="33.19" width="0" layer="19" extent="1-1"/>
@@
 <contactref element="U$1" pad="MISO"/>
 <contactref element="U$2" pad="13"/>
-<wire x1="14.05" y1="9.83" x2="-31.395" y2="8.705" width="0" layer="19" extent="1-1"/>
+<wire x1="14.05" y1="9.83" x2="7.265" y2="17.595" width="0" layer="19" extent="1-1"/>
 </signal>
 <signal name="N$17">
@@
 <contactref element="JP2" pad="2"/>
 <contactref element="LSP1" pad="MP"/>
-<wire x1="7.55" y1="9.83" x2="-35.945" y2="1.455" width="0" layer="19" extent="1-1"/>
+<wire x1="7.55" y1="9.83" x2="11.815" y2="10.345" width="0" layer="19" extent="1-1"/>
 <wire x1="2.54" y1="10.16" x2="7.55" y2="9.83" width="0" layer="19" extent="1-1"/>
 <wire x1="15.24" y1="2.54" x2="2.54" y2="10.16" width="0" layer="19" extent="1-1"/>
@@
 <contactref element="U$2" pad="19"/>
 <contactref element="JP2" pad="4"/>
-<wire x1="2.54" y1="15.24" x2="-35.295" y2="8.705" width="0" layer="19" extent="1-1"/>
+<wire x1="2.54" y1="15.24" x2="11.165" y2="17.595" width="0" layer="19" extent="1-1"/>
 </signal>
 <signal name="N$19">
 <contactref element="U$2" pad="18"/>
 <contactref element="JP2" pad="5"/>
-<wire x1="2.54" y1="17.78" x2="-34.645" y2="8.705" width="0" layer="19" extent="1-1"/>
+<wire x1="2.54" y1="17.78" x2="10.515" y2="17.595" width="0" layer="19" extent="1-1"/>
 </signal>
 <signal name="N$16">
 <contactref element="U$2" pad="17"/>
 <contactref element="U$1" pad="CE"/>
-<wire x1="8.85" y1="9.83" x2="-33.995" y2="8.705" width="0" layer="19" extent="1-1"/>
+<wire x1="8.85" y1="9.83" x2="9.865" y2="17.595" width="0" layer="19" extent="1-1"/>
 </signal>
 <signal name="N$20">
 <contactref element="U$2" pad="16"/>
 <contactref element="U$1" pad="CSN"/>
-<wire x1="10.15" y1="9.83" x2="-33.345" y2="8.705" width="0" layer="19" extent="1-1"/>
+<wire x1="10.15" y1="9.83" x2="9.215" y2="17.595" width="0" layer="19" extent="1-1"/>
 </signal>
 <signal name="N$21">
 <contactref element="U$2" pad="14"/>
 <contactref element="U$1" pad="IRQ"/>
-<wire x1="15.35" y1="9.83" x2="-32.045" y2="8.705" width="0" layer="19" extent="1-1"/>
+<wire x1="15.35" y1="9.83" x2="7.915" y2="17.595" width="0" layer="19" extent="1-1"/>
 </signal>
 <signal name="N$22">
 <contactref element="U$2" pad="11"/>
 <contactref element="U$1" pad="SCK"/>
-<wire x1="11.45" y1="9.83" x2="-30.095" y2="8.705" width="0" layer="19" extent="1-1"/>
+<wire x1="11.45" y1="9.83" x2="5.965" y2="17.595" width="0" layer="19" extent="1-1"/>
 </signal>
 <signal name="N$23">
 <contactref element="U$2" pad="9"/>
 <contactref element="U$1" pad="MOSI"/>
-<wire x1="12.75" y1="9.83" x2="-30.745" y2="1.455" width="0" layer="19" extent="1-1"/>
+<wire x1="12.75" y1="9.83" x2="6.615" y2="10.345" width="0" layer="19" extent="1-1"/>
 </signal>
 <signal name="N$25">
 <contactref element="U$2" pad="4"/>
 <contactref element="JP2" pad="1"/>
-<wire x1="2.54" y1="7.62" x2="-33.995" y2="1.455" width="0" layer="19" extent="1-1"/>
+<wire x1="2.54" y1="7.62" x2="9.865" y2="10.345" width="0" layer="19" extent="1-1"/>
 </signal>
 <signal name="N$28">
@@
 <contactref element="R1" pad="1"/>
 <contactref element="R3" pad="2"/>
-<wire x1="-43.332" y1="20.32" x2="-32.695" y2="1.455" width="0" layer="19" extent="1-1"/>
+<wire x1="-43.332" y1="20.32" x2="8.565" y2="10.345" width="0" layer="19" extent="1-1"/>
 <wire x1="-18.898" y1="29.21" x2="-43.332" y2="20.32" width="0" layer="19" extent="1-1"/>
 </signal>
@@
 <contactref element="R2" pad="1"/>
 <contactref element="R4" pad="2"/>
-<wire x1="-23.978" y1="29.21" x2="-32.045" y2="1.455" width="0" layer="19" extent="1-1"/>
+<wire x1="-23.978" y1="29.21" x2="7.915" y2="10.345" width="0" layer="19" extent="1-1"/>
 <wire x1="-16.662" y1="29.21" x2="-23.978" y2="29.21" width="0" layer="19" extent="1-1"/>
 </signal>
@@
 <contactref element="IC1" pad="3"/>
 <contactref element="U$2" pad="5"/>
-<wire x1="27.94" y1="10.16" x2="-33.345" y2="1.455" width="0" layer="19" extent="1-1"/>
+<wire x1="27.94" y1="10.16" x2="9.215" y2="10.345" width="0" layer="19" extent="1-1"/>
 </signal>
 <signal name="N$1">
 <contactref element="IC1" pad="2"/>
 <contactref element="U$2" pad="2"/>
-<wire x1="26.035" y1="8.89" x2="-35.295" y2="1.455" width="0" layer="19" extent="1-1"/>
+<wire x1="26.035" y1="8.89" x2="11.165" y2="10.345" width="0" layer="19" extent="1-1"/>
 </signal>
 <signal name="N$2">
 <contactref element="JP1" pad="3"/>
 <contactref element="U$3" pad="P$2"/>
-<wire x1="27.94" y1="16.51" x2="22.86" y2="6.35" width="0" layer="19" extent="1-1"/>
+<wire x1="27.94" y1="17.78" x2="22.86" y2="6.35" width="0" layer="19" extent="1-1"/>
 </signal>
 <signal name="N$7">
@@
 <contactref element="JP1" pad="1"/>
 <contactref element="U$3" pad="P$4"/>
-<wire x1="22.86" y1="16.51" x2="22.86" y2="10.75" width="0" layer="19" extent="1-1"/>
+<wire x1="22.86" y1="17.78" x2="22.86" y2="10.75" width="0" layer="19" extent="1-1"/>
 </signal>
 <signal name="N$10">
 <contactref element="JP1" pad="2"/>
 <contactref element="U$3" pad="P$3"/>
-<wire x1="25.4" y1="16.51" x2="22.86" y2="8.55" width="0" layer="19" extent="1-1"/>
+<wire x1="25.4" y1="17.78" x2="22.86" y2="8.55" width="0" layer="19" extent="1-1"/>
+</signal>
+<signal name="N$6">
+<contactref element="S1" pad="2"/>
+<contactref element="U$2" pad="3"/>
+<wire x1="10.515" y1="10.345" x2="5.08" y2="5.08" width="0" layer="19" extent="1-1"/>
 </signal>
 </signals>
