File: Hardware/Schemas/raspi.sch (EAGLE design)
At the start: 4 parts

Commit message: a
Parts:
- added S1: (no value), switch-dil:SD4-01
Connections:
- new net N$1: S1.2, U$2.RA5/T1CKI/OSC1/CLKIN
- net N$5: now also S1.1
Changed lines of the file:
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@@
 <part name="JP2" library="pinhead" deviceset="PINHD-1X5" device="" value="Prog"/>
 <part name="JP1" library="pinhead" deviceset="PINHD-2X5" device="" value="Raspi"/>
+<part name="S1" library="switch-dil" deviceset="SD4-01" device=""/>
 </parts>
 <sheets>
@@
 <instance part="JP2" gate="A" x="162.56" y="121.92"/>
 <instance part="JP1" gate="A" x="43.18" y="78.74"/>
+<instance part="S1" gate="1" x="73.66" y="45.72"/>
 </instances>
 <busses>
@@
 <net name="N$5" class="0">
 <segment>
-<wire x1="66.04" y1="30.48" x2="132.08" y2="30.48" width="0.1524" layer="91"/>
+<wire x1="66.04" y1="30.48" x2="73.66" y2="30.48" width="0.1524" layer="91"/>
+<wire x1="73.66" y1="30.48" x2="132.08" y2="30.48" width="0.1524" layer="91"/>
 <wire x1="132.08" y1="30.48" x2="177.8" y2="30.48" width="0.1524" layer="91"/>
 <pinref part="U$2" gate="G$1" pin="VSS"/>
@@
 <wire x1="48.26" y1="78.74" x2="66.04" y2="78.74" width="0.1524" layer="91"/>
 <wire x1="66.04" y1="78.74" x2="66.04" y2="30.48" width="0.1524" layer="91"/>
+<pinref part="S1" gate="1" pin="1"/>
+<wire x1="73.66" y1="38.1" x2="73.66" y2="30.48" width="0.1524" layer="91"/>
+<junction x="73.66" y="30.48"/>
 </segment>
 </net>
@@
 </segment>
 </net>
+<net name="N$1" class="0">
+<segment>
+<pinref part="S1" gate="1" pin="2"/>
+<wire x1="73.66" y1="53.34" x2="73.66" y2="139.7" width="0.1524" layer="91"/>
+<pinref part="U$2" gate="G$1" pin="RA5/T1CKI/OSC1/CLKIN"/>
+<wire x1="119.38" y1="119.38" x2="119.38" y2="139.7" width="0.1524" layer="91"/>
+<wire x1="119.38" y1="139.7" x2="73.66" y2="139.7" width="0.1524" layer="91"/>
+</segment>
+</net>
