File: Hardware/Schemas/tempSensor.sch (EAGLE design)
At the start: 6 parts, among them IC1 DS1820

Commit message: a
Parts:
- added S1: (no value), switch-dil:SD4-01
Connections:
- new net N$2: S1.2, U$2.RA4/AN3/T1G/OSC2/CLKOUT
- net N$5: now also S1.1
Changed lines of the file:
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@@
 <part name="LSP1" library="solpad" deviceset="LSP11" device=""/>
 <part name="LSP2" library="solpad" deviceset="LSP11" device=""/>
+<part name="S1" library="switch-dil" deviceset="SD4-01" device=""/>
 </parts>
 <sheets>
@@
 <instance part="LSP1" gate="1" x="86.36" y="48.26"/>
 <instance part="LSP2" gate="1" x="101.6" y="48.26"/>
+<instance part="S1" gate="1" x="68.58" y="55.88"/>
 </instances>
 <busses>
@@
 <pinref part="IC1" gate="G$1" pin="GND"/>
 <wire x1="58.42" y1="91.44" x2="58.42" y2="30.48" width="0.1524" layer="91"/>
-<wire x1="58.42" y1="30.48" x2="101.6" y2="30.48" width="0.1524" layer="91"/>
+<wire x1="58.42" y1="30.48" x2="68.58" y2="30.48" width="0.1524" layer="91"/>
 <junction x="132.08" y="30.48"/>
 <pinref part="LSP2" gate="1" pin="MP"/>
+<wire x1="68.58" y1="30.48" x2="101.6" y2="30.48" width="0.1524" layer="91"/>
 <wire x1="101.6" y1="30.48" x2="132.08" y2="30.48" width="0.1524" layer="91"/>
 <wire x1="101.6" y1="45.72" x2="101.6" y2="30.48" width="0.1524" layer="91"/>
+<pinref part="S1" gate="1" pin="1"/>
+<wire x1="68.58" y1="48.26" x2="68.58" y2="30.48" width="0.1524" layer="91"/>
+<junction x="68.58" y="30.48"/>
 </segment>
 </net>
@@
 </segment>
 </net>
+<net name="N$2" class="0">
+<segment>
+<pinref part="S1" gate="1" pin="2"/>
+<wire x1="68.58" y1="63.5" x2="73.66" y2="63.5" width="0.1524" layer="91"/>
+<wire x1="73.66" y1="63.5" x2="73.66" y2="139.7" width="0.1524" layer="91"/>
+<pinref part="U$2" gate="G$1" pin="RA4/AN3/T1G/OSC2/CLKOUT"/>
+<wire x1="73.66" y1="139.7" x2="121.92" y2="139.7" width="0.1524" layer="91"/>
+<wire x1="121.92" y1="139.7" x2="121.92" y2="119.38" width="0.1524" layer="91"/>
+</segment>
+</net>
