File: Hardware/Schemas/tempThermostat.sch (EAGLE design)
At the start: 21 parts, among them IC1 DS1820

Commit message: a
Parts:
- added S1: (no value), switch-dil:SD4-01
Connections:
- new net N$6: S1.2, U$2.RA4/AN3/T1G/OSC2/CLKOUT
- net N$5: now also S1.1
Changed lines of the file:
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@@
 <part name="D3" library="diode" deviceset="MBRA340T3" device=""/>
 <part name="D4" library="diode" deviceset="MBRA340T3" device=""/>
+<part name="S1" library="switch-dil" deviceset="SD4-01" device=""/>
 </parts>
 <sheets>
@@
 <instance part="D3" gate="G$1" x="40.64" y="114.3" rot="R90"/>
 <instance part="D4" gate="G$1" x="27.94" y="114.3" rot="R90"/>
+<instance part="S1" gate="1" x="73.66" y="76.2"/>
 </instances>
 <busses>
@@
 <pinref part="IC1" gate="G$1" pin="GND"/>
 <wire x1="58.42" y1="91.44" x2="58.42" y2="86.36" width="0.1524" layer="91"/>
-<wire x1="58.42" y1="86.36" x2="58.42" y2="30.48" width="0.1524" layer="91"/>
+<wire x1="58.42" y1="86.36" x2="58.42" y2="60.96" width="0.1524" layer="91"/>
+<wire x1="58.42" y1="60.96" x2="58.42" y2="30.48" width="0.1524" layer="91"/>
 <wire x1="58.42" y1="30.48" x2="101.6" y2="30.48" width="0.1524" layer="91"/>
 <junction x="132.08" y="30.48"/>
@@
 <junction x="40.64" y="86.36"/>
 <junction x="25.4" y="86.36"/>
+<pinref part="S1" gate="1" pin="1"/>
+<wire x1="73.66" y1="68.58" x2="73.66" y2="60.96" width="0.1524" layer="91"/>
+<wire x1="73.66" y1="60.96" x2="58.42" y2="60.96" width="0.1524" layer="91"/>
+<junction x="58.42" y="60.96"/>
 </segment>
 </net>
@@
 </segment>
 </net>
+<net name="N$6" class="0">
+<segment>
+<pinref part="S1" gate="1" pin="2"/>
+<wire x1="73.66" y1="83.82" x2="73.66" y2="139.7" width="0.1524" layer="91"/>
+<pinref part="U$2" gate="G$1" pin="RA4/AN3/T1G/OSC2/CLKOUT"/>
+<wire x1="73.66" y1="139.7" x2="121.92" y2="139.7" width="0.1524" layer="91"/>
+<wire x1="121.92" y1="139.7" x2="121.92" y2="119.38" width="0.1524" layer="91"/>
+</segment>
+</net>
