File: Hardware/SchemasBoard/heatingHeader.brd (EAGLE design)
At the start: 45.5 x 30.5 mm, 30 parts, among them IC1 DS1820

Commit message: a
Parts:
- added Q1: BSS123, transistor-small-signal:SOT23
- moved JP1 3.35 mm to (35.1, 26.9)
- moved D3 0.80 mm to (36.2, 21.8)
Connections:
- new net N$11: JP1.1, Q1.3
- new net N$28: Q1.1, U$2.12
- net VDD: now also Q1.2; no longer JP1.1
Routing:
- net N$28: track 0.00 -> 36.1 mm, vias 0 -> 2
- net GND: track 186.9 -> 160.4 mm
- net N$15: track 55.9 -> 47.9 mm, vias 3 -> 2
- net VDD: track 97.8 -> 104.0 mm, vias 2 -> 3
- net N$2: track 40.9 -> 45.3 mm
- net N$27: track 31.4 -> 34.8 mm
- net N$11: track 0.00 -> 1.43 mm
- net N$13: track 20.2 -> 19.2 mm

Commit message: a
Parts:
- added R6: 4K7, resistor:R1206W
Connections:
- net N$25: now also R6.1
- net VDD: now also R6.2
Routing:
- net N$25: track 38.8 -> 65.9 mm, vias 1 -> 2
- net VDD: track 104.0 -> 111.3 mm, vias 3 -> 4
Changed lines of the file:
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@@
 <element name="C2" library="resistor" package="C2012" value="100nF" x="12.2" y="27.4" rot="MR0"/>
 <element name="Q1" library="transistor-small-signal" package="SOT23" value="BSS123" x="31.3" y="26.9" rot="MR90"/>
+<element name="R6" library="resistor" package="R1206W" value="4K7" x="3.3" y="1.5" rot="MR0"/>
 </elements>
 <signals>
@@
 <wire x1="35.4" y1="10.2" x2="34" y2="8.8" width="0.3048" layer="1"/>
 <wire x1="34" y1="8.8" x2="28.6" y2="8.8" width="0.3048" layer="1"/>
-<wire x1="28.6" y1="8.8" x2="20.8" y2="17.2" width="0.3048" layer="1"/>
+<wire x1="28.6" y1="8.8" x2="28.37205625" y2="9.045478125" width="0.3048" layer="1"/>
+<wire x1="28.37205625" y1="9.045478125" x2="20.8" y2="17.2" width="0.3048" layer="1"/>
 <wire x1="20.8" y1="17.2" x2="15.4" y2="17.2" width="0.3048" layer="1"/>
 <wire x1="15.4" y1="17.2" x2="11.1" y2="21.6" width="0.3048" layer="1"/>
@@
 <wire x1="12.24" y1="22.9" x2="12.245" y2="22.905" width="0.4064" layer="16"/>
 <wire x1="40.76" y1="10.2" x2="40.79" y2="10.17" width="0.4064" layer="1"/>
+<contactref element="R6" pad="1"/>
+<wire x1="4.799" y1="1.5" x2="10.1" y2="1.5" width="0.3048" layer="16"/>
+<wire x1="10.1" y1="1.5" x2="10.1" y2="2.1" width="0.3048" layer="16"/>
+<wire x1="10.1" y1="2.1" x2="15.5" y2="2.1" width="0.3048" layer="16"/>
+<via x="15.5" y="2.1" extent="1-16" drill="0.6"/>
+<wire x1="15.5" y1="2.1" x2="21.426578125" y2="2.1" width="0.3048" layer="1"/>
+<wire x1="21.426578125" y1="2.1" x2="28.37205625" y2="9.045478125" width="0.3048" layer="1"/>
 </signal>
 <signal name="N$30">
@@
 <wire x1="1.8" y1="25.6" x2="2.06" y2="25.6" width="0.3048" layer="1"/>
 <wire x1="2.06" y1="25.6" x2="2.06" y2="27.21" width="0.3048" layer="1"/>
+<contactref element="R6" pad="2"/>
+<wire x1="1.801" y1="1.5" x2="1.6" y2="1.5" width="0.3048" layer="16"/>
+<wire x1="1.6" y1="1.5" x2="1.6" y2="3.5" width="0.3048" layer="16"/>
+<via x="1.6" y="3.5" extent="1-16" drill="0.6"/>
+<wire x1="1.6" y1="3.5" x2="1.7" y2="3.5" width="0.3048" layer="1"/>
+<wire x1="1.7" y1="3.5" x2="1.7" y2="8.5" width="0.3048" layer="1"/>
 <wire x1="40.9" y1="12.7" x2="40.79" y2="12.71" width="0" layer="19" extent="1-1"/>
 </signal>

Commit message: a
Parts:
- Q1: value BSS123 -> BSS84
- moved R6 6.10 mm to (3.10, 7.60), turned to 90 degrees
- moved Q1 0.20 mm to (31.1, 26.9)
Routing:
- net N$25: track 65.9 -> 76.6 mm
- net VDD: track 111.3 -> 100.8 mm, vias 4 -> 3
- net N$3: track 49.7 -> 58.7 mm
- net N$16: track 35.4 -> 41.6 mm
- net N$30: track 14.1 -> 16.1 mm
- net N$31: track 8.18 -> 6.60 mm
- net N$15: track 47.9 -> 46.4 mm
- net N$1: track 43.3 -> 42.7 mm
- net GND: track 160.4 -> 160.9 mm
