File: Hardware/SchemasBoard/heatingHeader.brd (EAGLE design)
At the start: 45.5 x 30.5 mm, 36 parts, among them IC1 DS1820, T5 BC846

Commit message: dfg
Parts:
- removed R9: 1K, resistor:R1206
- removed T5: BC846, transistor:SOT23
Connections:
- removed net N$11: R9.2, U$2.8
- removed net N$28: T5.3, U$1.GND
- removed net N$5: R9.1, T5.1
- net GND: now also U$1.GND; no longer T5.2
Routing:
- net N$11: track 41.2 -> 0.00 mm, vias 2 -> 0
- net N$28: track 7.35 -> 0.00 mm, vias 2 -> 0
- net N$5: track 2.07 -> 0.00 mm
- net GND: track 172.3 -> 170.9 mm
