File: Hardware/SchemasBoard/pc.brd (EAGLE design)
At the start: 14.9 x 24.1 mm, 10 parts

Commit message: aa
Parts:
- removed S1: (no value), switch-dil:SD4-01
- added S2: DTSM-3, switch-tact:DTSM-3
Connections:
- net GND: now also S2.1; no longer S1.1
- net N$1: now also S2.2; no longer S1.2
Routing:
- net N$1: track 7.47 -> 6.46 mm
Changed lines of the file:
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@@
 <element name="PAD3" library="wirepad" package="5-1,8" value="WIREPADSMD5-1,8" x="10.16" y="3.81"/>
 <element name="PAD4" library="wirepad" package="5-1,8" value="WIREPADSMD5-1,8" x="12.7" y="3.81"/>
-<element name="S1" library="switch-dil" package="SD4-01" value="" x="9.800034375" y="16.987021875">
-<attribute name="OC_NEWARK" value="unknown" x="9.800034375" y="16.987021875" size="1.778" layer="27" display="off"/>
-<attribute name="MPN" value="" x="9.800034375" y="16.987021875" size="1.778" layer="27" display="off"/>
-<attribute name="MF" value="" x="9.800034375" y="16.987021875" size="1.778" layer="27" display="off"/>
-<attribute name="OC_FARNELL" value="unknown" x="9.800034375" y="16.987021875" size="1.778" layer="27" display="off"/>
-</element>
 <element name="C1" library="resistor" package="C2012" value="100nF" x="2.3622" y="12.2809" rot="MR0"/>
 <element name="C2" library="resistor" package="SMC_A" value="1uF" x="13.9827" y="4.7752" rot="MR90"/>
+<element name="S2" library="switch-tact" package="DTSM-3" value="DTSM-3" x="1.4859" y="-11.4935"/>
 </elements>
 <signals>
@@
 <contactref element="JP2" pad="3"/>
 <contactref element="PAD4" pad="1"/>
-<contactref element="S1" pad="1"/>
 <wire x1="10.8458" y1="18.4531" x2="10.8712" y2="21.971" width="0.3048" layer="16"/>
 <wire x1="10.8712" y1="21.971" x2="10.287" y2="22.5552" width="0.3048" layer="16"/>
@@
 <wire x1="10.8458" y1="18.4531" x2="12.027790625" y2="17.5387" width="0.3048" layer="16"/>
 <wire x1="12.027790625" y1="17.5387" x2="13.488290625" y2="16.51" width="0.3048" layer="16"/>
+<contactref element="S2" pad="1"/>
+<wire x1="13.5636" y1="7.5819" x2="13.488290625" y2="16.51" width="0" layer="19" extent="16-16"/>
+<wire x1="2.44" y1="10.441" x2="12.7" y2="7.5819" width="0" layer="19" extent="16-16"/>
+<wire x1="-1.2141" y1="-11.4935" x2="12.0904" y2="3.8354" width="0" layer="19" extent="1-1"/>
 </signal>
 <signal name="N$12">
@@
 </signal>
 <signal name="N$1">
-<contactref element="S1" pad="2"/>
 <contactref element="U$2" pad="2"/>
 <wire x1="6.3009" y1="14.7773" x2="6.2992" y2="14.779" width="0.254" layer="16"/>
@@
 <via x="6.2992" y="16.2814" extent="1-16" drill="0.6"/>
 <wire x1="6.2992" y1="16.2814" x2="9.800034375" y2="19.782234375" width="0.254" layer="1"/>
-<wire x1="9.800034375" y1="19.782234375" x2="9.800034375" y2="20.797021875" width="0.254" layer="1"/>
+<contactref element="S2" pad="2"/>
+<wire x1="4.1859" y1="-11.4935" x2="6.3009" y2="14.7773" width="0" layer="19" extent="1-16"/>
 </signal>
 </signals>
