File: Hardware/SchemasBoard/pc.brd (EAGLE design)
At the start: 14.9 x 24.1 mm, 10 parts

Commit message: a
Routing:
- net GND: track 19.0 -> 23.9 mm
Changed lines of the file:
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@@
 <contactref element="PAD4" pad="1"/>
 <contactref element="S1" pad="1"/>
-<wire x1="13.488290625" y1="16.51" x2="12.7889" y2="16.51" width="0.3048" layer="16"/>
-<wire x1="12.7889" y1="16.51" x2="10.8458" y2="18.4531" width="0.3048" layer="16"/>
 <wire x1="10.8458" y1="18.4531" x2="10.8712" y2="21.971" width="0.3048" layer="16"/>
 <wire x1="10.8712" y1="21.971" x2="10.287" y2="22.5552" width="0.3048" layer="16"/>
@@
 <contactref element="C1" pad="2"/>
 <contactref element="C2" pad="-"/>
-<wire x1="13.8303" y1="5.9436" x2="13.7541" y2="5.8039" width="0.4064" layer="1"/>
-<wire x1="13.7541" y1="5.8039" x2="12.0904" y2="3.8354" width="0.4064" layer="1"/>
+<wire x1="13.7541" y1="5.8039" x2="13.136665625" y2="5.073346875" width="0.4064" layer="1"/>
+<wire x1="13.136665625" y1="5.073346875" x2="12.0904" y2="3.8354" width="0.4064" layer="1"/>
 <wire x1="12.0904" y1="3.8354" x2="12.7" y2="3.8354" width="0.4064" layer="1"/>
 <wire x1="12.7" y1="3.8354" x2="12.7" y2="3.81" width="0.4064" layer="1"/>
@@
 <wire x1="1.5494" y1="11.3919" x2="1.5494" y2="12.2437" width="0.4064" layer="16"/>
 <wire x1="1.5494" y1="12.2437" x2="1.5122" y2="12.2809" width="0.4064" layer="16"/>
-<via x="12.7889" y="16.51" extent="1-16" drill="0.6" shape="square"/>
-<wire x1="13.8303" y1="5.9436" x2="13.9827" y2="6.2752" width="0" layer="19" extent="1-16"/>
+<wire x1="13.9827" y1="6.2752" x2="13.5636" y2="6.2752" width="0.3048" layer="16"/>
+<wire x1="13.5636" y1="6.2752" x2="13.5636" y2="7.5819" width="0.3048" layer="16"/>
+<wire x1="13.5636" y1="7.5819" x2="12.7" y2="7.5819" width="0.3048" layer="16"/>
+<wire x1="12.7" y1="7.5819" x2="12.7" y2="7.4549" width="0.3048" layer="16"/>
+<via x="12.7" y="7.4549" extent="1-16" drill="0.6"/>
+<wire x1="12.7" y1="7.4549" x2="12.7" y2="5.5100125" width="0.3048" layer="1"/>
+<wire x1="12.7" y1="5.5100125" x2="13.136665625" y2="5.073346875" width="0.3048" layer="1"/>
+<wire x1="10.8458" y1="18.4531" x2="12.027790625" y2="17.5387" width="0.3048" layer="16"/>
+<wire x1="12.027790625" y1="17.5387" x2="13.488290625" y2="16.51" width="0.3048" layer="16"/>
 </signal>
 <signal name="N$12">

Commit message: aa
Parts:
- removed S1: (no value), switch-dil:SD4-01
- added S2: DTSM-3, switch-tact:DTSM-3
Connections:
- net GND: now also S2.1; no longer S1.1
- net N$1: now also S2.2; no longer S1.2
Routing:
- net GND: track 23.9 -> 26.4 mm, vias 2 -> 3
- net N$1: track 7.47 -> 9.75 mm, vias 1 -> 2
- net VDD: track 56.7 -> 58.3 mm
Changed lines of the file:
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@@
 <element name="PAD3" library="wirepad" package="5-1,8" value="WIREPADSMD5-1,8" x="10.16" y="3.81"/>
 <element name="PAD4" library="wirepad" package="5-1,8" value="WIREPADSMD5-1,8" x="12.7" y="3.81"/>
-<element name="S1" library="switch-dil" package="SD4-01" value="" x="9.800034375" y="16.987021875">
-<attribute name="OC_NEWARK" value="unknown" x="9.800034375" y="16.987021875" size="1.778" layer="27" display="off"/>
-<attribute name="MPN" value="" x="9.800034375" y="16.987021875" size="1.778" layer="27" display="off"/>
-<attribute name="MF" value="" x="9.800034375" y="16.987021875" size="1.778" layer="27" display="off"/>
-<attribute name="OC_FARNELL" value="unknown" x="9.800034375" y="16.987021875" size="1.778" layer="27" display="off"/>
-</element>
 <element name="C1" library="resistor" package="C2012" value="100nF" x="2.3622" y="12.2809" rot="MR0"/>
 <element name="C2" library="resistor" package="SMC_A" value="1uF" x="13.9827" y="4.7752" rot="MR90"/>
+<element name="S2" library="switch-tact" package="DTSM-3" value="DTSM-3" x="9.7663" y="17.7292" rot="MR90"/>
 </elements>
 <signals>
@@
 <contactref element="JP2" pad="3"/>
 <contactref element="PAD4" pad="1"/>
-<contactref element="S1" pad="1"/>
-<wire x1="10.8458" y1="18.4531" x2="10.8712" y2="21.971" width="0.3048" layer="16"/>
-<wire x1="10.8712" y1="21.971" x2="10.287" y2="22.5552" width="0.3048" layer="16"/>
+<wire x1="11.0871" y1="18.415" x2="11.0744" y2="21.9329" width="0.3048" layer="16"/>
+<wire x1="11.0744" y1="21.9329" x2="10.287" y2="22.5552" width="0.3048" layer="16"/>
 <wire x1="10.287" y1="22.5552" x2="7.2517" y2="22.5552" width="0.3048" layer="16"/>
 <wire x1="7.2517" y1="22.5552" x2="6.9636" y2="22.5846" width="0.3048" layer="16"/>
@@
 <wire x1="12.7" y1="7.4549" x2="12.7" y2="5.5100125" width="0.3048" layer="1"/>
 <wire x1="12.7" y1="5.5100125" x2="13.136665625" y2="5.073346875" width="0.3048" layer="1"/>
-<wire x1="10.8458" y1="18.4531" x2="12.027790625" y2="17.5387" width="0.3048" layer="16"/>
-<wire x1="12.027790625" y1="17.5387" x2="13.488290625" y2="16.51" width="0.3048" layer="16"/>
+<wire x1="11.0871" y1="18.415" x2="12.065890625" y2="17.6022" width="0.3048" layer="16"/>
+<wire x1="12.065890625" y1="17.6022" x2="13.488290625" y2="16.51" width="0.3048" layer="16"/>
+<contactref element="S2" pad="1"/>
+<wire x1="9.7663" y1="15.0292" x2="9.7917" y2="15.0292" width="0.4064" layer="16"/>
+<wire x1="9.7917" y1="15.0292" x2="9.7917" y2="13.4112" width="0.3048" layer="16"/>
+<via x="9.7917" y="13.4112" extent="1-16" drill="0.6"/>
+<wire x1="8.9408" y1="13.4239" x2="9.7917" y2="13.4112" width="0.3048" layer="1"/>
+<wire x1="9.7917" y1="13.4112" x2="9.7917" y2="13.4239" width="0.3048" layer="1"/>
 </signal>
 <signal name="N$12">
@@
 <contactref element="U$2" pad="13"/>
 <wire x1="9.5034" y1="9.0041" x2="9.7701" y2="9.7447" width="0.3048" layer="16"/>
-<wire x1="9.7701" y1="9.7447" x2="10.9093" y2="10.7696" width="0.3048" layer="16"/>
-<wire x1="10.9093" y1="10.7696" x2="10.9093" y2="15.7226" width="0.3048" layer="16"/>
-<wire x1="10.9093" y1="15.7226" x2="7.3152" y2="19.3167" width="0.3048" layer="16"/>
+<wire x1="9.7701" y1="9.7447" x2="10.9728" y2="10.7696" width="0.3048" layer="16"/>
+<wire x1="10.9728" y1="10.7696" x2="10.9728" y2="16.7386" width="0.3048" layer="16"/>
+<wire x1="10.9728" y1="16.7386" x2="7.3152" y2="19.3167" width="0.3048" layer="16"/>
 <wire x1="7.3152" y1="19.3167" x2="2.921" y2="19.3167" width="0.3048" layer="16"/>
 <wire x1="2.921" y1="19.3167" x2="2.413" y2="20.0152" width="0.3048" layer="16"/>
@@
 <contactref element="PAD1" pad="1"/>
 <wire x1="13.488290625" y1="13.97" x2="11.9126" y2="13.97" width="0.3048" layer="1"/>
-<wire x1="11.9126" y1="13.97" x2="10.6045" y2="15.2781" width="0.3048" layer="1"/>
-<wire x1="10.6045" y1="15.2781" x2="9.6139" y2="15.2781" width="0.3048" layer="1"/>
-<via x="9.6139" y="15.2781" extent="1-16" drill="0.6"/>
-<wire x1="9.6139" y1="15.2781" x2="9.0932" y2="14.7574" width="0.3048" layer="16"/>
-<wire x1="9.0932" y1="14.7574" x2="7.9121" y2="14.7574" width="0.3048" layer="16"/>
+<wire x1="11.9126" y1="13.97" x2="11.0109" y2="12.9413" width="0.3048" layer="1"/>
+<wire x1="11.0109" y1="12.9413" x2="9.4107" y2="12.192" width="0.3048" layer="1"/>
+<via x="9.4107" y="12.192" extent="1-16" drill="0.6"/>
+<wire x1="9.4107" y1="12.192" x2="7.9375" y2="12.9921" width="0.3048" layer="16"/>
+<wire x1="7.9375" y1="12.9921" x2="7.9121" y2="14.7574" width="0.3048" layer="16"/>
 <wire x1="7.9121" y1="14.7574" x2="7.4803" y2="15.1892" width="0.3048" layer="16"/>
 <wire x1="7.4803" y1="15.1892" x2="6.9469" y2="15.1892" width="0.3048" layer="16"/>
@@
 <wire x1="6.9509" y1="15.5107" x2="7.239" y2="15.7988" width="0.3048" layer="16"/>
 <wire x1="7.239" y1="15.7988" x2="7.239" y2="15.8369" width="0.3048" layer="16"/>
-<wire x1="7.239" y1="15.8369" x2="7.4676" y2="16.0655" width="0.3048" layer="16"/>
-<wire x1="7.4676" y1="16.0655" x2="7.4676" y2="16.5481" width="0.3048" layer="16"/>
-<wire x1="7.4676" y1="16.5481" x2="6.7564" y2="17.7673" width="0.3048" layer="16"/>
+<wire x1="7.239" y1="15.8369" x2="7.2644" y2="16.51" width="0.3048" layer="16"/>
+<wire x1="7.2644" y1="16.51" x2="7.2644" y2="16.9926" width="0.3048" layer="16"/>
+<wire x1="7.2644" y1="16.9926" x2="6.7564" y2="17.7673" width="0.3048" layer="16"/>
 <wire x1="6.7564" y1="17.7673" x2="0.254" y2="17.8181" width="0.3048" layer="16"/>
 <wire x1="0.254" y1="17.8181" x2="0.2159" y2="7.4549" width="0.3048" layer="16"/>
@@
 <contactref element="JP2" pad="4"/>
 <wire x1="13.488290625" y1="19.05" x2="12.7635" y2="19.05" width="0.3048" layer="16"/>
-<wire x1="12.7635" y1="19.05" x2="11.4554" y2="20.3581" width="0.3048" layer="16"/>
-<wire x1="11.4554" y1="20.3581" x2="11.4681" y2="22.3266" width="0.3048" layer="16"/>
-<wire x1="11.4681" y1="22.3266" x2="10.4902" y2="23.2537" width="0.3048" layer="16"/>
+<wire x1="12.7635" y1="19.05" x2="11.5824" y2="20.3581" width="0.3048" layer="16"/>
+<wire x1="11.5824" y1="20.3581" x2="11.5697" y2="22.3266" width="0.3048" layer="16"/>
+<wire x1="11.5697" y1="22.3266" x2="10.4902" y2="23.2537" width="0.3048" layer="16"/>
 <wire x1="10.4902" y1="23.2537" x2="6.5405" y2="23.2537" width="0.3048" layer="16"/>
 <wire x1="6.5405" y1="23.2537" x2="6.3009" y2="23.0268" width="0.3048" layer="16"/>
@@
 <wire x1="10.8034" y1="9.0041" x2="11.557" y2="9.0041" width="0.3048" layer="16"/>
 <wire x1="11.557" y1="9.0041" x2="11.557" y2="10.6553" width="0.3048" layer="16"/>
-<wire x1="11.557" y1="10.6553" x2="11.54" y2="15.9682" width="0.3048" layer="16"/>
-<wire x1="11.54" y1="15.9682" x2="7.5692" y2="19.939" width="0.3048" layer="16"/>
+<wire x1="11.557" y1="10.6553" x2="11.54" y2="17.1493" width="0.3048" layer="16"/>
+<wire x1="11.54" y1="17.1493" x2="7.5692" y2="19.939" width="0.3048" layer="16"/>
 <wire x1="7.5692" y1="19.939" x2="3.2131" y2="19.939" width="0.3048" layer="16"/>
 <wire x1="3.2131" y1="19.939" x2="3.0607" y2="20.3581" width="0.3048" layer="16"/>
@@
 </signal>
 <signal name="N$1">
-<contactref element="S1" pad="2"/>
 <contactref element="U$2" pad="2"/>
-<wire x1="6.3009" y1="14.7773" x2="6.2992" y2="14.779" width="0.254" layer="16"/>
-<wire x1="6.2992" y1="14.779" x2="6.2992" y2="16.2814" width="0.254" layer="16"/>
-<via x="6.2992" y="16.2814" extent="1-16" drill="0.6"/>
-<wire x1="6.2992" y1="16.2814" x2="9.800034375" y2="19.782234375" width="0.254" layer="1"/>
-<wire x1="9.800034375" y1="19.782234375" x2="9.800034375" y2="20.797021875" width="0.254" layer="1"/>
+<contactref element="S2" pad="2"/>
+<wire x1="6.3009" y1="14.7773" x2="6.2992" y2="14.7773" width="0.3048" layer="16"/>
+<wire x1="6.2992" y1="14.7773" x2="6.2992" y2="16.4719" width="0.3048" layer="16"/>
+<via x="6.2992" y="16.4719" extent="1-16" drill="0.6"/>
+<wire x1="6.2992" y1="16.4719" x2="6.2992" y2="19.7231" width="0.3048" layer="1"/>
+<wire x1="6.2992" y1="19.7231" x2="8.2677" y2="21.6916" width="0.3048" layer="1"/>
+<via x="8.2677" y="21.6916" extent="1-16" drill="0.6"/>
+<wire x1="8.2677" y1="21.6916" x2="8.5039" y2="21.6916" width="0.3048" layer="16"/>
+<wire x1="8.5039" y1="21.6916" x2="9.7663" y2="20.4292" width="0.3048" layer="16"/>
 </signal>
 </signals>

Commit message: aaa
Parts:
- removed JP2: Prog, pinhead:1X05
- added U$3: PROGRAMMINGHEADERDIP, rfm70:PROGHEADER
Connections:
- removed net N$19: JP2.5, U$2.18
- new net N$2: U$2.18, U$3.PGC
- net GND: now also U$3.GND; no longer JP2.3
- net N$18: now also U$3.PGD; no longer JP2.4
- net N$25: now also U$3.MCLR; no longer JP2.1
- net VDD: now also U$3.VDD; no longer JP2.2
Routing:
- net N$2: track 0.00 -> 10.5 mm
- net N$19: track 10.3 -> 0.00 mm
- net N$25: track 10.4 -> 11.2 mm
Changed lines of the file:
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@@
 <layers>
 <layer number="1" name="Top" color="4" fill="1" visible="yes" active="yes"/>
-<layer number="16" name="Bottom" color="1" fill="1" visible="yes" active="yes"/>
+<layer number="16" name="Bottom" color="1" fill="1" visible="no" active="yes"/>
 <layer number="17" name="Pads" color="2" fill="1" visible="yes" active="yes"/>
 <layer number="18" name="Vias" color="2" fill="1" visible="yes" active="yes"/>
@@
 <element name="U$1" library="rfm70" package="RFM70" value="RFM70" x="1.8034" y="-5.2959" rot="MR180"/>
 <element name="U$2" library="microchip" package="SSOP20" value="PIC16F690" x="4.0259" y="18.4023" rot="MR0"/>
-<element name="JP2" library="pinhead" package="1X05" value="Prog" x="13.488290625" y="16.51" rot="R90"/>
 <element name="PAD1" library="wirepad" package="5-1,8" value="WIREPADSMD5-1,8" x="2.54" y="3.81"/>
 <element name="PAD2" library="wirepad" package="5-1,8" value="WIREPADSMD5-1,8" x="7.62" y="3.81"/>
@@
 <element name="C2" library="resistor" package="SMC_A" value="1uF" x="13.9827" y="4.7752" rot="MR90"/>
 <element name="S2" library="switch-tact" package="DTSM-3" value="DTSM-3" x="9.7663" y="17.7292" rot="MR90"/>
+<element name="U$3" library="rfm70" package="PROGHEADER" value="PROGRAMMINGHEADERDIP" x="13.5128" y="17.0561" rot="R90"/>
 </elements>
 <signals>
@@
 <contactref element="U$2" pad="20"/>
 <contactref element="U$1" pad="GND"/>
-<contactref element="JP2" pad="3"/>
 <contactref element="PAD4" pad="1"/>
 <wire x1="11.0871" y1="18.415" x2="11.0744" y2="21.9329" width="0.3048" layer="16"/>
@@
 <wire x1="12.7" y1="5.5100125" x2="13.136665625" y2="5.073346875" width="0.3048" layer="1"/>
 <wire x1="11.0871" y1="18.415" x2="12.065890625" y2="17.6022" width="0.3048" layer="16"/>
-<wire x1="12.065890625" y1="17.6022" x2="13.488290625" y2="16.51" width="0.3048" layer="16"/>
 <contactref element="S2" pad="1"/>
 <wire x1="9.7663" y1="15.0292" x2="9.7917" y2="15.0292" width="0.4064" layer="16"/>
@@
 <wire x1="8.9408" y1="13.4239" x2="9.7917" y2="13.4112" width="0.3048" layer="1"/>
 <wire x1="9.7917" y1="13.4112" x2="9.7917" y2="13.4239" width="0.3048" layer="1"/>
+<contactref element="U$3" pad="GND"/>
+<contactref element="U$3" pad="GND"/>
+<wire x1="13.5128" y1="17.0561" x2="12.611990625" y2="17.0561" width="0.3048" layer="16"/>
+<wire x1="12.611990625" y1="17.0561" x2="12.065890625" y2="17.6022" width="0.3048" layer="16"/>
 </signal>
 <signal name="N$12">
@@
 <contactref element="U$2" pad="1"/>
 <contactref element="U$1" pad="VDD"/>
-<contactref element="JP2" pad="2"/>
 <contactref element="PAD1" pad="1"/>
-<wire x1="13.488290625" y1="13.97" x2="11.9126" y2="13.97" width="0.3048" layer="1"/>
-<wire x1="11.9126" y1="13.97" x2="11.0109" y2="12.9413" width="0.3048" layer="1"/>
-<wire x1="11.0109" y1="12.9413" x2="9.4107" y2="12.192" width="0.3048" layer="1"/>
+<wire x1="11.9126" y1="13.97" x2="10.9474" y2="12.7127" width="0.3048" layer="1"/>
+<wire x1="10.9474" y1="12.7127" x2="9.4107" y2="12.192" width="0.3048" layer="1"/>
 <via x="9.4107" y="12.192" extent="1-16" drill="0.6"/>
 <wire x1="9.4107" y1="12.192" x2="7.9375" y2="12.9921" width="0.3048" layer="16"/>
@@
 <wire x1="7.239" y1="15.8369" x2="7.2644" y2="16.51" width="0.3048" layer="16"/>
 <wire x1="7.2644" y1="16.51" x2="7.2644" y2="16.9926" width="0.3048" layer="16"/>
-<wire x1="7.2644" y1="16.9926" x2="6.7564" y2="17.7673" width="0.3048" layer="16"/>
-<wire x1="6.7564" y1="17.7673" x2="0.254" y2="17.8181" width="0.3048" layer="16"/>
+<wire x1="7.2644" y1="16.9926" x2="6.7945" y2="17.8054" width="0.3048" layer="16"/>
+<wire x1="6.7945" y1="17.8054" x2="0.254" y2="17.8181" width="0.3048" layer="16"/>
 <wire x1="0.254" y1="17.8181" x2="0.2159" y2="7.4549" width="0.3048" layer="16"/>
 <wire x1="0.2159" y1="7.4549" x2="0.1651" y2="7.4041" width="0.4064" layer="16"/>
 <wire x1="0.1651" y1="7.4041" x2="2.7813" y2="7.4041" width="0.3048" layer="16"/>
 <wire x1="2.7813" y1="7.4041" x2="2.9464" y2="7.5692" width="0.4064" layer="16"/>
+<contactref element="U$3" pad="VDD"/>
+<contactref element="U$3" pad="VDD"/>
+<wire x1="13.2628" y1="15.0561" x2="12.9453" y2="15.0027" width="0.3048" layer="1"/>
+<wire x1="12.9453" y1="15.0027" x2="11.9126" y2="13.97" width="0.3048" layer="1"/>
 </signal>
 <signal name="N$18">
 <contactref element="U$2" pad="19"/>
-<contactref element="JP2" pad="4"/>
-<wire x1="13.488290625" y1="19.05" x2="12.7635" y2="19.05" width="0.3048" layer="16"/>
 <wire x1="12.7635" y1="19.05" x2="11.5824" y2="20.3581" width="0.3048" layer="16"/>
 <wire x1="11.5824" y1="20.3581" x2="11.5697" y2="22.3266" width="0.3048" layer="16"/>
@@
 <wire x1="6.5405" y1="23.2537" x2="6.3009" y2="23.0268" width="0.3048" layer="16"/>
 <wire x1="6.3009" y1="23.0268" x2="6.3009" y2="22.0273" width="0.3048" layer="16"/>
-</signal>
-<signal name="N$19">
-<contactref element="U$2" pad="18"/>
-<contactref element="JP2" pad="5"/>
-<wire x1="13.488290625" y1="21.59" x2="13.2461" y2="21.5138" width="0.3048" layer="16"/>
-<wire x1="13.2461" y1="21.5138" x2="10.8585" y2="23.8633" width="0.3048" layer="16"/>
-<wire x1="10.8585" y1="23.8633" x2="6.2611" y2="23.8633" width="0.3048" layer="16"/>
-<wire x1="6.2611" y1="23.8633" x2="5.6382" y2="23.1515" width="0.3048" layer="16"/>
-<wire x1="5.6382" y1="23.1515" x2="5.6509" y2="22.0273" width="0.3048" layer="16"/>
+<contactref element="U$3" pad="PGD"/>
+<wire x1="13.2628" y1="19.0561" x2="12.7696" y2="19.0561" width="0.3048" layer="16"/>
+<wire x1="12.7696" y1="19.0561" x2="12.7635" y2="19.05" width="0.3048" layer="16"/>
 </signal>
 <signal name="N$16">
@@
 <wire x1="6.2484" y1="10.1346" x2="6.7183" y2="10.6045" width="0.254" layer="1"/>
 <wire x1="6.7183" y1="10.6045" x2="6.7564" y2="12.1539" width="0.254" layer="1"/>
-<wire x1="6.7564" y1="12.1539" x2="4.9403" y2="13.1953" width="0.254" layer="1"/>
-<wire x1="4.9403" y1="13.1953" x2="4.826" y2="20.4343" width="0.254" layer="1"/>
-<wire x1="4.826" y1="20.4343" x2="4.9276" y2="21.4503" width="0.254" layer="1"/>
+<wire x1="6.7564" y1="12.1539" x2="5.0165" y2="13.2207" width="0.254" layer="1"/>
+<wire x1="5.0165" y1="13.2207" x2="4.8768" y2="20.4597" width="0.254" layer="1"/>
+<wire x1="4.8768" y1="20.4597" x2="4.9276" y2="21.4503" width="0.254" layer="1"/>
 <wire x1="4.9276" y1="21.4503" x2="4.8641" y2="23.5458" width="0.254" layer="1"/>
 <via x="4.8641" y="23.5458" extent="1-16" drill="0.6"/>
@@
 <signal name="N$25">
 <contactref element="U$2" pad="4"/>
-<contactref element="JP2" pad="1"/>
-<wire x1="13.488290625" y1="11.43" x2="11.7475" y2="11.43" width="0.3048" layer="1"/>
-<wire x1="11.7475" y1="11.43" x2="11.3919" y2="11.0744" width="0.3048" layer="1"/>
-<wire x1="11.3919" y1="11.0744" x2="9.7663" y2="10.9601" width="0.3048" layer="1"/>
+<wire x1="11.3919" y1="10.9855" x2="9.7663" y2="10.9601" width="0.3048" layer="1"/>
 <via x="9.7663" y="10.9601" extent="1-16" drill="0.6"/>
 <wire x1="9.7663" y1="10.9601" x2="9.2329" y2="11.0744" width="0.3048" layer="16"/>
@@
 <wire x1="6.5151" y1="13.0048" x2="5.0517" y2="13.757" width="0.3048" layer="16"/>
 <wire x1="5.0517" y1="13.757" x2="5.0009" y2="14.7773" width="0.254" layer="16"/>
+<contactref element="U$3" pad="MCLR"/>
+<wire x1="13.5128" y1="13.0561" x2="13.1953" y2="12.8778" width="0.3048" layer="1"/>
+<wire x1="13.1953" y1="12.8778" x2="11.3919" y2="10.9855" width="0.3048" layer="1"/>
 </signal>
 <signal name="N$33">
@@
 <wire x1="8.5039" y1="21.6916" x2="9.7663" y2="20.4292" width="0.3048" layer="16"/>
 </signal>
+<signal name="N$2">
+<contactref element="U$3" pad="PGC"/>
+<contactref element="U$2" pad="18"/>
+<wire x1="5.6509" y1="22.0273" x2="5.6509" y2="23.1388" width="0.3048" layer="16"/>
+<wire x1="5.6509" y1="23.1388" x2="6.2865" y2="23.7744" width="0.3048" layer="16"/>
+<wire x1="6.2865" y1="23.7744" x2="10.8839" y2="23.7744" width="0.3048" layer="16"/>
+<wire x1="10.8839" y1="23.7744" x2="12.9159" y2="21.7424" width="0.3048" layer="16"/>
+<wire x1="12.9159" y1="21.7424" x2="12.9159" y2="21.3355" width="0.3048" layer="16"/>
+<wire x1="12.9159" y1="21.3355" x2="13.5128" y2="21.0561" width="0.3048" layer="16"/>
+</signal>
 </signals>

Commit message: fghf
Parts:
- moved C2 4.56 mm to (13.7, 9.32)
- moved U$3 0.08 mm to (13.4, 17.1)
Routing:
- net VDD: track 58.7 -> 63.2 mm
- net GND: track 26.3 -> 25.6 mm
- net N$34: track 25.4 -> 26.1 mm
- added copper zone on layer 16, net VDD
Other:
- board size 14.9 x 24.1 mm -> 14.9 x 24.2 mm
