File: Hardware/SchemasBoard/raspi.sch (EAGLE design)
At the start: 7 parts

Commit message: aa
Parts:
- removed S1: (no value), switch-dil:SD4-01
- added S2: DTSM-3, switch-tact:DTSM-3
Connections:
- net GND: now also S2.1; no longer S1.1
- net N$28: now also S2.2, U$2.RA4/AN3/T1G/OSC2/CLKOUT; no longer S1.2, U$2.RC6/AN8/SS
Changed lines of the file:
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@@
 <part name="JP2" library="pinhead" deviceset="PINHD-1X5" device="" value="Prog"/>
 <part name="JP1" library="pinhead" deviceset="PINHD-2X5" device="" value="Raspi"/>
-<part name="S1" library="switch-dil" deviceset="SD4-01" device=""/>
 <part name="C1" library="rcl" deviceset="C-EU" device="C0805"/>
 <part name="C2" library="resistor" deviceset="CPOL-EU" device="SMCA"/>
+<part name="S2" library="switch-tact" deviceset="DTSM-3" device=""/>
 </parts>
 <sheets>
@@
 <instance part="JP2" gate="A" x="162.56" y="121.92"/>
 <instance part="JP1" gate="A" x="43.18" y="78.74"/>
-<instance part="S1" gate="1" x="73.66" y="48.26"/>
 <instance part="C1" gate="G$1" x="33.02" y="114.3"/>
 <instance part="C2" gate="G$1" x="40.64" y="114.3"/>
+<instance part="S2" gate="G$1" x="73.66" y="45.72"/>
 </instances>
 <busses>
@@
 <wire x1="66.04" y1="78.74" x2="66.04" y2="30.48" width="0.1524" layer="91"/>
 <label x="106.68" y="30.48" size="1.778" layer="95"/>
-<pinref part="S1" gate="1" pin="1"/>
 <wire x1="73.66" y1="40.64" x2="73.66" y2="30.48" width="0.1524" layer="91"/>
 <junction x="73.66" y="30.48"/>
+<pinref part="S2" gate="G$1" pin="1"/>
 </segment>
 <segment>
@@
 <net name="N$28" class="0">
 <segment>
-<pinref part="U$2" gate="G$1" pin="RC6/AN8/SS"/>
-<pinref part="S1" gate="1" pin="2"/>
-<wire x1="73.66" y1="55.88" x2="73.66" y2="121.92" width="0.1524" layer="91"/>
-<wire x1="73.66" y1="121.92" x2="86.36" y2="121.92" width="0.1524" layer="91"/>
-<wire x1="86.36" y1="121.92" x2="86.36" y2="119.38" width="0.1524" layer="91"/>
+<wire x1="73.66" y1="50.8" x2="73.66" y2="139.7" width="0.1524" layer="91"/>
+<pinref part="U$2" gate="G$1" pin="RA4/AN3/T1G/OSC2/CLKOUT"/>
+<wire x1="73.66" y1="139.7" x2="121.92" y2="139.7" width="0.1524" layer="91"/>
+<wire x1="121.92" y1="139.7" x2="121.92" y2="119.38" width="0.1524" layer="91"/>
+<pinref part="S2" gate="G$1" pin="2"/>
 </segment>
 </net>

Commit message: aa
Parts:
- added S1, S3: DTSM-3, switch-tact:DTSM-3
Connections:
- new net N$1: JP1.3, S3.2
- new net N$2: JP1.5, S1.2
- net GND: now also S1.1, S3.1
Changed lines of the file:
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@@
 <part name="C2" library="resistor" deviceset="CPOL-EU" device="SMCA"/>
 <part name="S2" library="switch-tact" deviceset="DTSM-3" device=""/>
+<part name="S1" library="switch-tact" deviceset="DTSM-3" device=""/>
+<part name="S3" library="switch-tact" deviceset="DTSM-3" device=""/>
 </parts>
 <sheets>
@@
 <instance part="C2" gate="G$1" x="40.64" y="114.3"/>
 <instance part="S2" gate="G$1" x="73.66" y="45.72"/>
+<instance part="S1" gate="G$1" x="7.62" y="60.96"/>
+<instance part="S3" gate="G$1" x="22.86" y="60.96"/>
 </instances>
 <busses>
@@
 <junction x="73.66" y="30.48"/>
 <pinref part="S2" gate="G$1" pin="1"/>
+<pinref part="S1" gate="G$1" pin="1"/>
+<wire x1="66.04" y1="30.48" x2="22.86" y2="30.48" width="0.1524" layer="91"/>
+<wire x1="22.86" y1="30.48" x2="7.62" y2="30.48" width="0.1524" layer="91"/>
+<wire x1="7.62" y1="30.48" x2="7.62" y2="55.88" width="0.1524" layer="91"/>
+<pinref part="S3" gate="G$1" pin="1"/>
+<wire x1="22.86" y1="55.88" x2="22.86" y2="30.48" width="0.1524" layer="91"/>
+<junction x="66.04" y="30.48"/>
+<junction x="22.86" y="30.48"/>
 </segment>
 <segment>
@@
 </segment>
 </net>
+<net name="N$1" class="0">
+<segment>
+<pinref part="S3" gate="G$1" pin="2"/>
+<wire x1="22.86" y1="66.04" x2="22.86" y2="81.28" width="0.1524" layer="91"/>
+<pinref part="JP1" gate="A" pin="3"/>
+<wire x1="22.86" y1="81.28" x2="40.64" y2="81.28" width="0.1524" layer="91"/>
+</segment>
+</net>
+<net name="N$2" class="0">
+<segment>
+<pinref part="JP1" gate="A" pin="5"/>
+<pinref part="S1" gate="G$1" pin="2"/>
+<wire x1="40.64" y1="78.74" x2="7.62" y2="78.74" width="0.1524" layer="91"/>
+<wire x1="7.62" y1="78.74" x2="7.62" y2="66.04" width="0.1524" layer="91"/>
+</segment>
+</net>

Commit message: a
Connections:
- net N$28: now also U$2.RA5/T1CKI/OSC1/CLKIN; no longer U$2.RA4/AN3/T1G/OSC2/CLKOUT
Changed lines of the file:
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@@
 <segment>
 <wire x1="73.66" y1="50.8" x2="73.66" y2="139.7" width="0.1524" layer="91"/>
-<pinref part="U$2" gate="G$1" pin="RA4/AN3/T1G/OSC2/CLKOUT"/>
-<wire x1="73.66" y1="139.7" x2="121.92" y2="139.7" width="0.1524" layer="91"/>
-<wire x1="121.92" y1="139.7" x2="121.92" y2="119.38" width="0.1524" layer="91"/>
 <pinref part="S2" gate="G$1" pin="2"/>
+<pinref part="U$2" gate="G$1" pin="RA5/T1CKI/OSC1/CLKIN"/>
+<wire x1="73.66" y1="139.7" x2="119.38" y2="139.7" width="0.1524" layer="91"/>
+<wire x1="119.38" y1="139.7" x2="119.38" y2="119.38" width="0.1524" layer="91"/>
 </segment>
 </net>

Commit message: aaa
Parts:
- removed JP2: Prog, pinhead:PINHD-1X5
- added U$3: PROGRAMMINGHEADERDIP, rfm70:PROGRAMMINGHEADERDIP
Connections:
- net GND: now also U$3.GND; no longer JP2.3
- net N$18: now also U$3.PGD; no longer JP2.4
- net N$19: now also U$3.PGC; no longer JP2.5
- net N$25: now also U$3.MCLR; no longer JP2.1
- net VDD: now also U$3.VDD; no longer JP2.2
Changed lines of the file:
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@@
 <part name="U$1" library="rfm70" deviceset="RFM70" device=""/>
 <part name="U$2" library="microchip" deviceset="PIC16F690*" device=""/>
-<part name="JP2" library="pinhead" deviceset="PINHD-1X5" device="" value="Prog"/>
 <part name="JP1" library="pinhead" deviceset="PINHD-2X5" device="" value="Raspi"/>
 <part name="C1" library="rcl" deviceset="C-EU" device="C0805"/>
@@
 <part name="S1" library="switch-tact" deviceset="DTSM-3" device=""/>
 <part name="S3" library="switch-tact" deviceset="DTSM-3" device=""/>
+<part name="U$3" library="rfm70" deviceset="PROGRAMMINGHEADER" device="" technology="DIP"/>
 </parts>
 <sheets>
@@
 <instance part="U$1" gate="G$1" x="170.18" y="45.72" rot="R270"/>
 <instance part="U$2" gate="G$1" x="134.62" y="68.58" rot="R90"/>
-<instance part="JP2" gate="A" x="162.56" y="121.92"/>
 <instance part="JP1" gate="A" x="43.18" y="78.74"/>
 <instance part="C1" gate="G$1" x="33.02" y="114.3"/>
@@
 <instance part="S1" gate="G$1" x="7.62" y="60.96"/>
 <instance part="S3" gate="G$1" x="22.86" y="60.96"/>
+<instance part="U$3" gate="G$1" x="177.8" y="132.08"/>
 </instances>
 <busses>
@@
 <wire x1="172.72" y1="55.88" x2="177.8" y2="55.88" width="0.1524" layer="91"/>
 <wire x1="177.8" y1="55.88" x2="177.8" y2="30.48" width="0.1524" layer="91"/>
-<wire x1="160.02" y1="121.92" x2="177.8" y2="121.92" width="0.1524" layer="91"/>
 <wire x1="177.8" y1="121.92" x2="177.8" y2="55.88" width="0.1524" layer="91"/>
 <junction x="177.8" y="55.88"/>
 <junction x="132.08" y="30.48"/>
-<pinref part="JP2" gate="A" pin="3"/>
 <pinref part="JP1" gate="A" pin="6"/>
 <wire x1="48.26" y1="78.74" x2="66.04" y2="78.74" width="0.1524" layer="91"/>
@@
 <junction x="66.04" y="30.48"/>
 <junction x="22.86" y="30.48"/>
+<wire x1="177.8" y1="121.92" x2="162.56" y2="121.92" width="0.1524" layer="91"/>
+<wire x1="162.56" y1="121.92" x2="162.56" y2="132.08" width="0.1524" layer="91"/>
+<pinref part="U$3" gate="G$1" pin="GND"/>
+<wire x1="162.56" y1="132.08" x2="167.64" y2="132.08" width="0.1524" layer="91"/>
 </segment>
 <segment>
@@
 <wire x1="33.02" y1="83.82" x2="33.02" y2="60.96" width="0.1524" layer="91"/>
 <label x="58.42" y="60.96" size="1.778" layer="95"/>
-<pinref part="JP2" gate="A" pin="2"/>
 <pinref part="U$1" gate="G$1" pin="VDD"/>
 <wire x1="170.18" y1="55.88" x2="170.18" y2="60.96" width="0.1524" layer="91"/>
-<wire x1="170.18" y1="60.96" x2="170.18" y2="124.46" width="0.1524" layer="91"/>
-<wire x1="170.18" y1="124.46" x2="160.02" y2="124.46" width="0.1524" layer="91"/>
 <wire x1="33.02" y1="60.96" x2="83.82" y2="60.96" width="0.1524" layer="91"/>
 <pinref part="U$2" gate="G$1" pin="VDD"/>
-<wire x1="83.82" y1="60.96" x2="170.18" y2="60.96" width="0.1524" layer="91"/>
+<wire x1="83.82" y1="60.96" x2="167.64" y2="60.96" width="0.1524" layer="91"/>
 <wire x1="83.82" y1="66.04" x2="83.82" y2="60.96" width="0.1524" layer="91"/>
 <junction x="83.82" y="60.96"/>
-<junction x="170.18" y="60.96"/>
+<pinref part="U$3" gate="G$1" pin="VDD"/>
+<wire x1="170.18" y1="60.96" x2="167.64" y2="60.96" width="0.1524" layer="91"/>
+<wire x1="167.64" y1="60.96" x2="167.64" y2="129.54" width="0.1524" layer="91"/>
 </segment>
 <segment>
@@
 <net name="N$18" class="0">
 <segment>
-<wire x1="144.78" y1="119.38" x2="144.78" y2="132.08" width="0.1524" layer="91"/>
 <pinref part="U$2" gate="G$1" pin="RA0/AN0/C1IN+/ICSPDAT/ULPWU"/>
-<wire x1="144.78" y1="132.08" x2="132.08" y2="132.08" width="0.1524" layer="91"/>
 <wire x1="132.08" y1="132.08" x2="132.08" y2="119.38" width="0.1524" layer="91"/>
-<pinref part="JP2" gate="A" pin="4"/>
-<wire x1="160.02" y1="119.38" x2="144.78" y2="119.38" width="0.1524" layer="91"/>
+<wire x1="132.08" y1="132.08" x2="160.02" y2="132.08" width="0.1524" layer="91"/>
+<wire x1="160.02" y1="132.08" x2="160.02" y2="134.62" width="0.1524" layer="91"/>
+<pinref part="U$3" gate="G$1" pin="PGD"/>
+<wire x1="160.02" y1="134.62" x2="167.64" y2="134.62" width="0.1524" layer="91"/>
 </segment>
 </net>
 <net name="N$19" class="0">
 <segment>
-<wire x1="147.32" y1="116.84" x2="147.32" y2="134.62" width="0.1524" layer="91"/>
 <pinref part="U$2" gate="G$1" pin="RA1/AN1/C12IN0-/VREF/ICSPCLK"/>
-<wire x1="147.32" y1="134.62" x2="129.54" y2="134.62" width="0.1524" layer="91"/>
+<wire x1="157.48" y1="134.62" x2="129.54" y2="134.62" width="0.1524" layer="91"/>
 <wire x1="129.54" y1="134.62" x2="129.54" y2="119.38" width="0.1524" layer="91"/>
-<pinref part="JP2" gate="A" pin="5"/>
-<wire x1="147.32" y1="116.84" x2="160.02" y2="116.84" width="0.1524" layer="91"/>
+<wire x1="157.48" y1="134.62" x2="157.48" y2="137.16" width="0.1524" layer="91"/>
+<pinref part="U$3" gate="G$1" pin="PGC"/>
+<wire x1="157.48" y1="137.16" x2="167.64" y2="137.16" width="0.1524" layer="91"/>
 </segment>
 </net>
@@
 <pinref part="U$2" gate="G$1" pin="RA3/MCLR/VPP"/>
 <wire x1="124.46" y1="119.38" x2="124.46" y2="137.16" width="0.1524" layer="91"/>
-<pinref part="JP2" gate="A" pin="1"/>
-<wire x1="124.46" y1="137.16" x2="160.02" y2="137.16" width="0.1524" layer="91"/>
-<wire x1="160.02" y1="137.16" x2="160.02" y2="127" width="0.1524" layer="91"/>
+<wire x1="124.46" y1="137.16" x2="154.94" y2="137.16" width="0.1524" layer="91"/>
+<pinref part="U$3" gate="G$1" pin="MCLR"/>
+<wire x1="167.64" y1="127" x2="154.94" y2="127" width="0.1524" layer="91"/>
+<wire x1="154.94" y1="127" x2="154.94" y2="137.16" width="0.1524" layer="91"/>
 </segment>
 </net>
