File: Hardware/SchemasBoard/spinac.sch (EAGLE design)
At the start: 27 parts, among them IC1 LNK304, IC2 MCP1703DB, IC4 DS1820, K1 G5L, T1 BC846

Commit message: a
Parts:
- added S1: (no value), switch-dil:SD4-01
Connections:
- new net N$5: S1.2, U$2.RC6/AN8/SS
- net GND: now also S1.1
Changed lines of the file:
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@@
 <part name="IC4" library="ds1820" deviceset="DS1820" device=""/>
 <part name="C6" library="resistor" deviceset="CPOL-EU" device="SMCA" value="1uF"/>
+<part name="S1" library="switch-dil" deviceset="SD4-01" device=""/>
 </parts>
 <sheets>
@@
 <instance part="IC4" gate="G$1" x="43.18" y="134.62"/>
 <instance part="C6" gate="G$1" x="139.7" y="45.72"/>
+<instance part="S1" gate="1" x="147.32" y="99.06"/>
 </instances>
 <busses>
@@
 <wire x1="127" y1="30.48" x2="132.08" y2="30.48" width="0.1524" layer="91"/>
 <wire x1="132.08" y1="30.48" x2="139.7" y2="30.48" width="0.1524" layer="91"/>
-<wire x1="139.7" y1="30.48" x2="177.8" y2="30.48" width="0.1524" layer="91"/>
+<wire x1="139.7" y1="30.48" x2="144.78" y2="30.48" width="0.1524" layer="91"/>
+<wire x1="144.78" y1="30.48" x2="177.8" y2="30.48" width="0.1524" layer="91"/>
 <wire x1="71.12" y1="35.56" x2="71.12" y2="30.48" width="0.1524" layer="91"/>
 <junction x="71.12" y="30.48"/>
@@
 <wire x1="139.7" y1="40.64" x2="139.7" y2="30.48" width="0.1524" layer="91"/>
 <junction x="139.7" y="30.48"/>
+<pinref part="S1" gate="1" pin="1"/>
+<wire x1="147.32" y1="91.44" x2="144.78" y2="91.44" width="0.1524" layer="91"/>
+<wire x1="144.78" y1="91.44" x2="144.78" y2="30.48" width="0.1524" layer="91"/>
 </segment>
 </net>
@@
 </segment>
 </net>
+<net name="N$5" class="0">
+<segment>
+<pinref part="S1" gate="1" pin="2"/>
+<wire x1="147.32" y1="106.68" x2="149.86" y2="106.68" width="0.1524" layer="91"/>
+<wire x1="149.86" y1="106.68" x2="149.86" y2="142.24" width="0.1524" layer="91"/>
+<pinref part="U$2" gate="G$1" pin="RC6/AN8/SS"/>
+<wire x1="149.86" y1="142.24" x2="86.36" y2="142.24" width="0.1524" layer="91"/>
+<wire x1="86.36" y1="142.24" x2="86.36" y2="119.38" width="0.1524" layer="91"/>
+</segment>
+</net>

Commit message: aaa
Parts:
- removed JP1, JP2: (no value), pinhead:PINHD-1X5
- removed R7: 2 K, resistor:R-EU_M2012
- added U$3: PROGRAMMINGHEADERDIP, rfm70:PROGRAMMINGHEADERDIP
- added X1: (no value), con-ptr500:AK500/5
- C1: device resistor:CPOL-EUE5-13 -> resistor:CPOL-EUE5-10.5
- K1: value G5L -> FRS1B; device relay:G5L -> relay:FRS1B
- L1: value BC12 -> MMICC7; device inductors:BC12 -> inductors:MMICC7
- S1: value (none) -> DTS-3; device switch-dil:SD4-01 -> switch-tact:DTS-3
Connections:
- net GND: now also U$3.GND; no longer JP2.3, R7.1
- net N$17: now also U$3.VDD; no longer JP2.2
- net N$18: now also U$3.PGD; no longer JP2.4
- net N$19: now also U$3.PGC; no longer JP2.5
- net N$24: now also X1-1.KL; no longer JP1.3
- net N$25: now also U$3.MCLR; no longer JP2.1
- net N$26: no longer R7.2
- net N$36: now also X1-5.KL; no longer JP1.1
- net N$4: now also X1-4.KL; no longer JP1.2
- net N$5: now also U$2.RB5/AN11/RX/DT; no longer U$2.RC6/AN8/SS
- net N$7: now also K12.P@1, X1-2.KL; no longer JP1.5, K12.S
- net N$8: now also K12.S, X1-3.KL; no longer JP1.4, K12.P
