File: Hardware/SchemasBoard/spinac.sch (EAGLE design)
At the start: 27 parts, among them IC1 LNK304, IC2 MCP1703DB, IC4 DS1820, K1 FRS1B, T1 BC846

Commit message: New version
Parts:
- removed IC2: MCP1703DB, linear:MCP1703DB
- added IC3: MC33269ST-3.3T3, linear:MC33269ST-3.3T3
- added R6: 1 K, resistor:R-EU_M2012
- L1: value MICC10 -> 680uH; device inductors:MICC10 -> inductor-neosid:BS11
Connections:
- removed net N$17: C5.2, C6.+, IC2.VO, IC4.VDD, U$1.VDD, U$2.VDD, U$3.VDD
- new net N$28: C5.2, C6.+, IC3.OUT, IC3.OUT@1, IC4.VDD, U$1.VDD, U$2.VDD, U$3.VDD
- net GND: now also IC3.GND/ADJ, IC4.GND, R6.1; no longer IC2.GND
- net N$26: now also IC3.IN, R6.2; no longer IC2.VI
- net N$9: no longer IC4.GND
Other:
- moved on the sheet: C4, C5

Commit message: fixed power supply 22 uF C3 and differend FW diode
Parts:
- C3: value 10uF / 16 V -> 22uF / 16 V
- D3: value (none) -> UF4007
- D4: value (none) -> 1N4007GP
- L1: value 680uH -> 1mH
Changed lines of the file:
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@@
 <part name="R4" library="resistor" deviceset="R-EU_" device="M2012" value="2,05 k"/>
 <part name="R5" library="resistor" deviceset="R-EU_" device="M2012" value="1 K"/>
-<part name="C3" library="resistor" deviceset="CPOL-EU" device="E2.5-5" value="10uF / 16 V"/>
-<part name="L1" library="inductor-neosid" deviceset="BS" device="11" value="680uH"/>
+<part name="C3" library="resistor" deviceset="CPOL-EU" device="E2.5-5" value="22uF / 16 V"/>
+<part name="L1" library="inductor-neosid" deviceset="BS" device="11" value="1mH"/>
 <part name="C4" library="resistor" deviceset="CPOL-EU" device="E2.5-5" value="100uF / 6,3 V"/>
 <part name="C5" library="resistor" deviceset="C-EU" device="C2012" value="100nF"/>
 <part name="T1" library="transistor" deviceset="BC846" device=""/>
-<part name="D3" library="diode" deviceset="DIODE-" device="DO214AA"/>
-<part name="D4" library="diode" deviceset="DIODE-" device="DO214AA"/>
+<part name="D3" library="diode" deviceset="DIODE-" device="DO214AA" value="UF4007"/>
+<part name="D4" library="diode" deviceset="DIODE-" device="DO214AA" value="1N4007GP"/>
 <part name="D1" library="diode" deviceset="MBRA340T3" device=""/>
 <part name="JP3" library="pinhead" deviceset="PINHD-1X3" device=""/>

Commit message: aaa
Parts:
- removed R6: 1 K, resistor:R-EU_M2012
- added R7: 10 k, resistor:R-EU_M2012
- D3: value UF4007 -> ES1D; device diode:DIODE-DO214AA -> diode:DIODE-DO214AC
Connections:
- net GND: now also R7.1; no longer R6.1
- net N$26: no longer R6.2
- net N$32: now also R7.2
Other:
- moved on the sheet: JP3
Changed lines of the file:
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@@
 <part name="C5" library="resistor" deviceset="C-EU" device="C2012" value="100nF"/>
 <part name="T1" library="transistor" deviceset="BC846" device=""/>
-<part name="D3" library="diode" deviceset="DIODE-" device="DO214AA" value="UF4007"/>
+<part name="D3" library="diode" deviceset="DIODE-" device="DO214AC" value="ES1D"/>
 <part name="D4" library="diode" deviceset="DIODE-" device="DO214AA" value="1N4007GP"/>
 <part name="D1" library="diode" deviceset="MBRA340T3" device=""/>
@@
 <part name="U$3" library="rfm70" deviceset="PROGRAMMINGHEADER" device="" technology="DIP"/>
 <part name="X1" library="con-ptr500" deviceset="AK500/5" device=""/>
-<part name="R6" library="resistor" deviceset="R-EU_" device="M2012" value="1 K"/>
 <part name="IC3" library="linear" deviceset="MC33269ST*" device="" technology="-3.3T3"/>
+<part name="R7" library="resistor" deviceset="R-EU_" device="M2012" value="10 k"/>
 </parts>
 <sheets>
@@
 <instance part="D4" gate="G$1" x="66.04" y="78.74" rot="R180"/>
 <instance part="D1" gate="G$1" x="10.16" y="76.2" rot="R90"/>
-<instance part="JP3" gate="A" x="66.04" y="101.6"/>
+<instance part="JP3" gate="A" x="66.04" y="99.06"/>
 <instance part="IC4" gate="G$1" x="43.18" y="134.62"/>
 <instance part="C6" gate="G$1" x="139.7" y="45.72"/>
@@
 <instance part="X1" gate="-4" x="-35.56" y="55.88"/>
 <instance part="X1" gate="-5" x="-35.56" y="50.8"/>
-<instance part="R6" gate="G$1" x="96.52" y="43.18" rot="R90"/>
 <instance part="IC3" gate="G$1" x="111.76" y="50.8"/>
+<instance part="R7" gate="G$1" x="33.02" y="109.22"/>
 </instances>
 <busses>
@@
 <wire x1="22.86" y1="30.48" x2="71.12" y2="30.48" width="0.1524" layer="91"/>
 <wire x1="71.12" y1="30.48" x2="86.36" y2="30.48" width="0.1524" layer="91"/>
-<wire x1="86.36" y1="30.48" x2="96.52" y2="30.48" width="0.1524" layer="91"/>
-<wire x1="96.52" y1="30.48" x2="111.76" y2="30.48" width="0.1524" layer="91"/>
+<wire x1="86.36" y1="30.48" x2="111.76" y2="30.48" width="0.1524" layer="91"/>
 <wire x1="111.76" y1="30.48" x2="127" y2="30.48" width="0.1524" layer="91"/>
 <wire x1="127" y1="30.48" x2="132.08" y2="30.48" width="0.1524" layer="91"/>
@@
 <pinref part="D3" gate="G$1" pin="A"/>
 <pinref part="JP3" gate="A" pin="3"/>
-<wire x1="63.5" y1="99.06" x2="20.32" y2="99.06" width="0.1524" layer="91"/>
-<wire x1="20.32" y1="99.06" x2="20.32" y2="68.58" width="0.1524" layer="91"/>
+<wire x1="63.5" y1="96.52" x2="20.32" y2="96.52" width="0.1524" layer="91"/>
+<wire x1="20.32" y1="96.52" x2="20.32" y2="68.58" width="0.1524" layer="91"/>
 <junction x="20.32" y="68.58"/>
 <label x="48.26" y="30.48" size="1.778" layer="95"/>
@@
 <wire x1="180.34" y1="132.08" x2="177.8" y2="132.08" width="0.1524" layer="91"/>
 <junction x="144.78" y="30.48"/>
-<pinref part="R6" gate="G$1" pin="1"/>
-<wire x1="96.52" y1="38.1" x2="96.52" y2="30.48" width="0.1524" layer="91"/>
-<junction x="96.52" y="30.48"/>
 <pinref part="IC4" gate="G$1" pin="GND"/>
 <wire x1="20.32" y1="127" x2="43.18" y2="127" width="0.1524" layer="91"/>
-<wire x1="20.32" y1="127" x2="20.32" y2="99.06" width="0.1524" layer="91"/>
-<junction x="20.32" y="99.06"/>
+<wire x1="20.32" y1="127" x2="20.32" y2="109.22" width="0.1524" layer="91"/>
+<junction x="20.32" y="96.52"/>
 <pinref part="IC3" gate="G$1" pin="GND/ADJ"/>
+<pinref part="R7" gate="G$1" pin="1"/>
+<wire x1="20.32" y1="109.22" x2="20.32" y2="96.52" width="0.1524" layer="91"/>
+<wire x1="20.32" y1="109.22" x2="27.94" y2="109.22" width="0.1524" layer="91"/>
+<junction x="20.32" y="109.22"/>
 </segment>
 </net>
@@
 <wire x1="43.18" y1="83.82" x2="76.2" y2="83.82" width="0.1524" layer="91"/>
 <wire x1="0" y1="81.28" x2="0" y2="83.82" width="0.1524" layer="91"/>
-<wire x1="104.14" y1="55.88" x2="96.52" y2="55.88" width="0.1524" layer="91"/>
-<wire x1="96.52" y1="55.88" x2="86.36" y2="55.88" width="0.1524" layer="91"/>
+<wire x1="104.14" y1="55.88" x2="86.36" y2="55.88" width="0.1524" layer="91"/>
 <wire x1="76.2" y1="58.42" x2="86.36" y2="58.42" width="0.1524" layer="91"/>
 <wire x1="86.36" y1="58.42" x2="86.36" y2="55.88" width="0.1524" layer="91"/>
@@
 <junction x="10.16" y="83.82"/>
 <pinref part="JP3" gate="A" pin="1"/>
-<wire x1="63.5" y1="104.14" x2="43.18" y2="104.14" width="0.1524" layer="91"/>
-<wire x1="43.18" y1="104.14" x2="43.18" y2="83.82" width="0.1524" layer="91"/>
+<wire x1="63.5" y1="101.6" x2="43.18" y2="101.6" width="0.1524" layer="91"/>
+<wire x1="43.18" y1="101.6" x2="43.18" y2="83.82" width="0.1524" layer="91"/>
 <junction x="43.18" y="83.82"/>
-<pinref part="R6" gate="G$1" pin="2"/>
-<wire x1="96.52" y1="48.26" x2="96.52" y2="55.88" width="0.1524" layer="91"/>
-<junction x="96.52" y="55.88"/>
 <pinref part="IC3" gate="G$1" pin="IN"/>
 </segment>
@@
 <wire x1="73.66" y1="134.62" x2="73.66" y2="109.22" width="0.1524" layer="91"/>
 <pinref part="JP3" gate="A" pin="2"/>
-<wire x1="63.5" y1="101.6" x2="55.88" y2="101.6" width="0.1524" layer="91"/>
-<wire x1="55.88" y1="101.6" x2="55.88" y2="109.22" width="0.1524" layer="91"/>
+<wire x1="63.5" y1="99.06" x2="55.88" y2="99.06" width="0.1524" layer="91"/>
+<wire x1="55.88" y1="99.06" x2="55.88" y2="109.22" width="0.1524" layer="91"/>
 <wire x1="55.88" y1="109.22" x2="73.66" y2="109.22" width="0.1524" layer="91"/>
-</segment>
-</net>
+<wire x1="55.88" y1="109.22" x2="38.1" y2="109.22" width="0.1524" layer="91"/>
+<pinref part="R7" gate="G$1" pin="2"/>
+<junction x="55.88" y="109.22"/>
+</segment>
+</net>

Commit message: sdfg
Parts:
- added R6: 1 K, resistor:R-EU_M2012
- C3: device resistor:CPOL-EUE2.5-5 -> resistor:CPOL-EUSMCC
- R2: device resistor:R-EU_R2512W -> resistor:R-EU_0411/12
Connections:
- net GND: now also R6.1
- net N$26: now also R6.2
Changed lines of the file:
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@@
 <part name="B1" library="rectifier" deviceset="RECTIFIER-" device="S40" value="RECTIFIER"/>
 <part name="R1" library="resistor" deviceset="R-EU_" device="R2512W" value="100"/>
-<part name="R2" library="resistor" deviceset="R-EU_" device="R2512W" value="8,2"/>
+<part name="R2" library="resistor" deviceset="R-EU_" device="0411/12" value="8,2"/>
 <part name="U$1" library="rfm70" deviceset="RFM70" device=""/>
 <part name="U$2" library="microchip" deviceset="PIC16F690*" device=""/>
@@
 <part name="R4" library="resistor" deviceset="R-EU_" device="M2012" value="2,05 k"/>
 <part name="R5" library="resistor" deviceset="R-EU_" device="M2012" value="1 K"/>
-<part name="C3" library="resistor" deviceset="CPOL-EU" device="E2.5-5" value="22uF / 16 V"/>
+<part name="C3" library="resistor" deviceset="CPOL-EU" device="SMCC" value="22uF / 16 V"/>
 <part name="L1" library="inductor-neosid" deviceset="BS" device="11" value="1mH"/>
 <part name="C4" library="resistor" deviceset="CPOL-EU" device="E2.5-5" value="100uF / 6,3 V"/>
@@
 <part name="IC3" library="linear" deviceset="MC33269ST*" device="" technology="-3.3T3"/>
 <part name="R7" library="resistor" deviceset="R-EU_" device="M2012" value="10 k"/>
+<part name="R6" library="resistor" deviceset="R-EU_" device="M2012" value="1 K"/>
 </parts>
 <sheets>
@@
 <instance part="IC3" gate="G$1" x="111.76" y="50.8"/>
 <instance part="R7" gate="G$1" x="33.02" y="109.22"/>
+<instance part="R6" gate="G$1" x="104.14" y="43.18" rot="R90"/>
 </instances>
 <busses>
@@
 <wire x1="22.86" y1="30.48" x2="71.12" y2="30.48" width="0.1524" layer="91"/>
 <wire x1="71.12" y1="30.48" x2="86.36" y2="30.48" width="0.1524" layer="91"/>
-<wire x1="86.36" y1="30.48" x2="111.76" y2="30.48" width="0.1524" layer="91"/>
+<wire x1="86.36" y1="30.48" x2="104.14" y2="30.48" width="0.1524" layer="91"/>
+<wire x1="104.14" y1="30.48" x2="111.76" y2="30.48" width="0.1524" layer="91"/>
 <wire x1="111.76" y1="30.48" x2="127" y2="30.48" width="0.1524" layer="91"/>
 <wire x1="127" y1="30.48" x2="132.08" y2="30.48" width="0.1524" layer="91"/>
@@
 <wire x1="20.32" y1="109.22" x2="27.94" y2="109.22" width="0.1524" layer="91"/>
 <junction x="20.32" y="109.22"/>
+<pinref part="R6" gate="G$1" pin="1"/>
+<wire x1="104.14" y1="38.1" x2="104.14" y2="30.48" width="0.1524" layer="91"/>
+<junction x="104.14" y="30.48"/>
 </segment>
 </net>
@@
 <junction x="43.18" y="83.82"/>
 <pinref part="IC3" gate="G$1" pin="IN"/>
+<pinref part="R6" gate="G$1" pin="2"/>
+<wire x1="104.14" y1="48.26" x2="104.14" y2="55.88" width="0.1524" layer="91"/>
+<junction x="104.14" y="55.88"/>
 </segment>
 </net>
@@
 <junction x="127" y="53.34"/>
 <wire x1="139.7" y1="55.88" x2="127" y2="55.88" width="0.1524" layer="91"/>
-</segment>
-</net>
+<junction x="139.7" y="55.88"/>
+</segment>
+</net>

Commit message: abcd
abcd
Parts:
- C6: value 1uF -> 4,7uF
- L1: value 1mH -> 680uH
Changed lines of the file:
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@@
 <?xml version="1.0" encoding="utf-8"?>
 <!DOCTYPE eagle SYSTEM "eagle.dtd">
-<eagle version="6.3">
+<eagle version="6.4">
 <drawing>
 <settings>
@@
 <part name="R5" library="resistor" deviceset="R-EU_" device="M2012" value="1 K"/>
 <part name="C3" library="resistor" deviceset="CPOL-EU" device="SMCC" value="22uF / 16 V"/>
-<part name="L1" library="inductor-neosid" deviceset="BS" device="11" value="1mH"/>
+<part name="L1" library="inductor-neosid" deviceset="BS" device="11" value="680uH"/>
 <part name="C4" library="resistor" deviceset="CPOL-EU" device="E2.5-5" value="100uF / 6,3 V"/>
 <part name="C5" library="resistor" deviceset="C-EU" device="C2012" value="100nF"/>
@@
 <part name="JP3" library="pinhead" deviceset="PINHD-1X3" device=""/>
 <part name="IC4" library="ds1820" deviceset="DS1820" device=""/>
-<part name="C6" library="resistor" deviceset="CPOL-EU" device="SMCA" value="1uF"/>
+<part name="C6" library="resistor" deviceset="CPOL-EU" device="SMCA" value="4,7uF"/>
 <part name="S1" library="switch-tact" deviceset="DTS-3" device=""/>
 <part name="U$3" library="rfm70" deviceset="PROGRAMMINGHEADER" device="" technology="DIP"/>
