File: Hardware/SchemasBoard/tempSensor.sch (EAGLE design)
At the start: 9 parts, among them IC1 DS1820

Commit message: a
Parts:
- added R1: 4K7, resistor:R-EU_R1206W
Connections:
- net N$25: now also R1.1
- net VDD: now also R1.2
Changed lines of the file:
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@@
 <part name="S1" library="switch-dil" deviceset="SD4-01" device=""/>
 <part name="C2" library="resistor" deviceset="CPOL-EU" device="SMCA"/>
+<part name="R1" library="resistor" deviceset="R-EU_" device="R1206W" value="4K7"/>
 </parts>
 <sheets>
@@
 <instance part="S1" gate="1" x="73.66" y="71.12"/>
 <instance part="C2" gate="G$1" x="43.18" y="58.42"/>
+<instance part="R1" gate="G$1" x="175.26" y="134.62"/>
 </instances>
 <busses>
@@
 <junction x="170.18" y="73.66"/>
 <junction x="170.18" y="68.58"/>
+<junction x="170.18" y="124.46"/>
+<pinref part="R1" gate="G$1" pin="2"/>
+<wire x1="170.18" y1="124.46" x2="180.34" y2="124.46" width="0.1524" layer="91"/>
+<wire x1="180.34" y1="124.46" x2="180.34" y2="134.62" width="0.1524" layer="91"/>
 </segment>
 <segment>
@@
 <pinref part="JP2" gate="A" pin="1"/>
 <wire x1="124.46" y1="137.16" x2="160.02" y2="137.16" width="0.1524" layer="91"/>
-<wire x1="160.02" y1="137.16" x2="160.02" y2="127" width="0.1524" layer="91"/>
+<wire x1="160.02" y1="137.16" x2="160.02" y2="134.62" width="0.1524" layer="91"/>
+<pinref part="R1" gate="G$1" pin="1"/>
+<wire x1="160.02" y1="134.62" x2="160.02" y2="127" width="0.1524" layer="91"/>
+<wire x1="170.18" y1="134.62" x2="160.02" y2="134.62" width="0.1524" layer="91"/>
+<junction x="160.02" y="134.62"/>
 </segment>
 </net>

Commit message: added support for remote IR detector
Parts:
- added JP1: (no value), pinhead:PINHD-1X3
- added LSP3: LSP11, solpad:LSP11
- added R2: 1K, resistor:R-EU_R1206W
- added T1: BC846, transistor:BC846
Connections:
- new net N$4: U$2.RB5/AN11/RX/DT
- new net N$5: JP1.3, LSP3.MP
- new net N$6: R2.2, U$2.RB7/TX/CK
- new net N$7: R2.1, T1.B
- new net N$9: JP1.1, T1.C
- net GND: now also T1.E
Changed lines of the file:
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@@
 <part name="C2" library="resistor" deviceset="CPOL-EU" device="SMCA"/>
 <part name="R1" library="resistor" deviceset="R-EU_" device="R1206W" value="4K7"/>
+<part name="JP1" library="pinhead" deviceset="PINHD-1X3" device=""/>
+<part name="LSP3" library="solpad" deviceset="LSP11" device=""/>
+<part name="T1" library="transistor" deviceset="BC846" device=""/>
+<part name="R2" library="resistor" deviceset="R-EU_" device="R1206W" value="1K"/>
 </parts>
 <sheets>
@@
 <instance part="C2" gate="G$1" x="43.18" y="58.42"/>
 <instance part="R1" gate="G$1" x="175.26" y="134.62"/>
+<instance part="JP1" gate="A" x="33.02" y="116.84"/>
+<instance part="LSP3" gate="1" x="38.1" y="106.68"/>
+<instance part="T1" gate="G$1" x="20.32" y="96.52"/>
+<instance part="R2" gate="G$1" x="17.78" y="139.7"/>
 </instances>
 <busses>
@@
 <pinref part="JP2" gate="A" pin="3"/>
 <pinref part="IC1" gate="G$1" pin="GND"/>
-<wire x1="58.42" y1="91.44" x2="58.42" y2="30.48" width="0.1524" layer="91"/>
+<wire x1="58.42" y1="91.44" x2="58.42" y2="78.74" width="0.1524" layer="91"/>
+<wire x1="58.42" y1="78.74" x2="58.42" y2="30.48" width="0.1524" layer="91"/>
 <wire x1="58.42" y1="30.48" x2="73.66" y2="30.48" width="0.1524" layer="91"/>
 <junction x="132.08" y="30.48"/>
@@
 <junction x="73.66" y="30.48"/>
 <junction x="132.08" y="66.04"/>
+<wire x1="22.86" y1="78.74" x2="58.42" y2="78.74" width="0.1524" layer="91"/>
+<junction x="58.42" y="78.74"/>
+<pinref part="T1" gate="G$1" pin="E"/>
+<wire x1="22.86" y1="78.74" x2="22.86" y2="91.44" width="0.1524" layer="91"/>
 </segment>
 <segment>
@@
 </segment>
 </net>
+<net name="N$4" class="0">
+<segment>
+<pinref part="U$2" gate="G$1" pin="RB5/AN11/RX/DT"/>
+<wire x1="111.76" y1="119.38" x2="111.76" y2="134.62" width="0.1524" layer="91"/>
+<wire x1="111.76" y1="134.62" x2="38.1" y2="134.62" width="0.1524" layer="91"/>
+<wire x1="38.1" y1="134.62" x2="38.1" y2="116.84" width="0.1524" layer="91"/>
+<wire x1="38.1" y1="116.84" x2="33.02" y2="116.84" width="0.1524" layer="91"/>
+</segment>
+</net>
+<net name="N$7" class="0">
+<segment>
+<pinref part="T1" gate="G$1" pin="B"/>
+<wire x1="17.78" y1="96.52" x2="12.7" y2="96.52" width="0.1524" layer="91"/>
+<wire x1="12.7" y1="96.52" x2="12.7" y2="139.7" width="0.1524" layer="91"/>
+<pinref part="R2" gate="G$1" pin="1"/>
+</segment>
+</net>
+<net name="N$9" class="0">
+<segment>
+<pinref part="T1" gate="G$1" pin="C"/>
+<wire x1="22.86" y1="101.6" x2="22.86" y2="119.38" width="0.1524" layer="91"/>
+<pinref part="JP1" gate="A" pin="1"/>
+<wire x1="22.86" y1="119.38" x2="30.48" y2="119.38" width="0.1524" layer="91"/>
+</segment>
+</net>
+<net name="N$5" class="0">
+<segment>
+<pinref part="JP1" gate="A" pin="3"/>
+<wire x1="30.48" y1="114.3" x2="30.48" y2="104.14" width="0.1524" layer="91"/>
+<pinref part="LSP3" gate="1" pin="MP"/>
+<wire x1="30.48" y1="104.14" x2="38.1" y2="104.14" width="0.1524" layer="91"/>
+</segment>
+</net>
+<net name="N$6" class="0">
+<segment>
+<pinref part="R2" gate="G$1" pin="2"/>
+<pinref part="U$2" gate="G$1" pin="RB7/TX/CK"/>
+<wire x1="22.86" y1="139.7" x2="106.68" y2="139.7" width="0.1524" layer="91"/>
+<wire x1="106.68" y1="139.7" x2="106.68" y2="119.38" width="0.1524" layer="91"/>
+</segment>
+</net>

Commit message: a
Parts:
- C1: value (none) -> 100nF
- C2: value (none) -> 1uF
Changed lines of the file:
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@@
 <part name="LSP1" library="solpad" deviceset="LSP11" device=""/>
 <part name="LSP2" library="solpad" deviceset="LSP11" device=""/>
-<part name="C1" library="resistor" deviceset="C-EU" device="C2012"/>
+<part name="C1" library="resistor" deviceset="C-EU" device="C2012" value="100nF"/>
 <part name="S1" library="switch-dil" deviceset="SD4-01" device=""/>
-<part name="C2" library="resistor" deviceset="CPOL-EU" device="SMCA"/>
+<part name="C2" library="resistor" deviceset="CPOL-EU" device="SMCA" value="1uF"/>
 <part name="R1" library="resistor" deviceset="R-EU_" device="R1206W" value="4K7"/>
 <part name="JP1" library="pinhead" deviceset="PINHD-1X3" device=""/>

Commit message: aaa
Parts:
- removed JP2: Prog, pinhead:PINHD-1X5
- added R3: 1K, resistor:R-EU_R1206W
- added T2: BC846, transistor:BC846
- added U$3: PROGRAMMINGHEADERDIP, rfm70:PROGRAMMINGHEADERDIP
- LSP1, LSP2, LSP3: value LSP11 -> SE14; device solpad:LSP11 -> solpad:SE14
- S1: value (none) -> DTS-3; device switch-dil:SD4-01 -> switch-tact:DTS-3
Connections:
- removed net N$18: JP2.4, U$2.RA0/AN0/C1IN+/ICSPDAT/ULPWU
- removed net N$19: JP2.5, U$2.RA1/AN1/C12IN0-/VREF/ICSPCLK
- new net N$10: U$3.GND
- new net N$11: U$2.RA1/AN1/C12IN0-/VREF/ICSPCLK, U$3.PGC
- new net N$13: T2.C, U$1.GND
- new net N$14: R3.2, T2.B
- new net N$15: R3.1, U$2.RC1/AN5/C12IN1-
- new net N$8: U$2.RA0/AN0/C1IN+/ICSPDAT/ULPWU, U$3.PGD
- net GND: now also T2.E; no longer JP2.3, U$1.GND
- net N$2: now also U$2.RA4/AN3/T1G/OSC2/CLKOUT; no longer U$2.RC6/AN8/SS
- net N$25: now also U$3.MCLR; no longer JP2.1
- net N$4: now also JP1.2
- net VDD: no longer JP2.2
Other:
- moved on the sheet: R1
