File: Hardware/SchemasBoard/rolety.brd (EAGLE design)
At the start: 47.9 x 22.9 mm, 29 parts, among them IC1 LNK304, IC2 MCP1703DB, K1 FRS1B, K2 FRS1B, T1 BC846, T2 BC846

Commit message: hf
Parts:
- removed IC2: MCP1703DB, linear:SOT223
- added IC3: MC33269ST-3.3T3, linear:SOT223
- added R7: 1 K, resistor:M2012
Connections:
- net GND: now also IC3.1, R7.1; no longer IC2.2
- net N$17: now also IC3.2, IC3.4; no longer IC2.3
- net N$27: now also IC3.3, R7.2; no longer IC2.1
Routing:
- net N$17: track 69.4 -> 61.9 mm
- net GND: track 114.6 -> 111.7 mm
- net N$27: track 76.4 -> 75.5 mm
Changed lines of the file:
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@@
 <element name="L1" library="inductors" package="MICC10" value="MICC10" x="29.718" y="1.651"/>
 <element name="C4" library="resistor" package="E2,5-5" value="100uF / 6,3 V" x="25.273" y="9.7155" rot="R180"/>
-<element name="IC2" library="linear" package="SOT223" value="MCP1703DB" x="34.3535" y="17.653" rot="MR90"/>
 <element name="C5" library="resistor" package="C2012" value="100nF" x="45.1485" y="7.239" rot="MR270"/>
 <element name="T1" library="transistor" package="SOT23" value="BC846" x="13.208" y="1.778" rot="MR270"/>
@@
 </element>
 <element name="U$3" library="rfm70" package="PROGHEADER" value="PROGRAMMINGHEADERDIP" x="41.148" y="2.0955"/>
+<element name="IC3" library="linear" package="SOT223" value="MC33269ST-3.3T3" x="-8.9535" y="0.127"/>
+<element name="R7" library="resistor" package="M2012" value="1 K" x="-10.8585" y="-7.4295"/>
 </elements>
 <signals>
@@
 <signal name="GND">
 <contactref element="B1" pad="-"/>
-<contactref element="IC2" pad="2"/>
 <contactref element="C5" pad="1"/>
 <contactref element="U$2" pad="20"/>
@@
 <wire x1="43.307" y1="14.2875" x2="43.2435" y2="14.224" width="0.3048" layer="16"/>
 <wire x1="43.2435" y1="14.224" x2="43.3705" y2="13.97" width="0.3048" layer="16"/>
-<wire x1="31.2547" y1="17.653" x2="34.163" y2="17.653" width="0.3048" layer="16"/>
 <wire x1="34.163" y1="17.653" x2="34.2265" y2="17.7165" width="0.3048" layer="16"/>
 <wire x1="34.2265" y1="17.7165" x2="34.2265" y2="16.256" width="0.3048" layer="16"/>
@@
 <wire x1="10.658" y1="12.4485" x2="10.729" y2="12.4485" width="0.3048" layer="16"/>
 <wire x1="10.729" y1="12.4485" x2="12.3825" y2="10.795" width="0.3048" layer="16"/>
+<contactref element="IC3" pad="1"/>
+<contactref element="R7" pad="1"/>
 <wire x1="46.355" y1="11.8745" x2="46.355" y2="11.8505" width="0" layer="19" extent="16-16"/>
+<wire x1="-11.2649" y1="-2.9718" x2="11.938" y2="2.7305" width="0" layer="19" extent="1-1"/>
+<wire x1="-11.8085" y1="-7.4295" x2="-11.2649" y2="-2.9718" width="0" layer="19" extent="1-1"/>
 </signal>
 <signal name="N$11">
@@
 </signal>
 <signal name="N$17">
-<contactref element="C5" pad="2"/>
-<contactref element="IC2" pad="3"/>
-<contactref element="U$2" pad="1"/>
 <contactref element="U$1" pad="VDD"/>
 <contactref element="C6" pad="+"/>
 <wire x1="45.212" y1="10.311" x2="43.311" y2="8.66" width="0.3048" layer="16"/>
-<wire x1="43.311" y1="8.66" x2="43.311" y2="5.646" width="0.3048" layer="16"/>
 <wire x1="43.3705" y1="4.953" x2="45.085" y2="4.953" width="0.3048" layer="16"/>
-<wire x1="45.085" y1="4.953" x2="45.1485" y2="6.389" width="0.3048" layer="16"/>
 <wire x1="38.7985" y1="3.81" x2="34.163" y2="3.81" width="0.3048" layer="16"/>
 <wire x1="34.163" y1="3.81" x2="34.163" y2="7.1755" width="0.3048" layer="16"/>
@@
 <wire x1="39.148" y1="2.3455" x2="39.148" y2="3.4605" width="0.3048" layer="16"/>
 <wire x1="39.148" y1="3.4605" x2="38.7985" y2="3.81" width="0.3048" layer="16"/>
-<wire x1="31.2547" y1="19.9644" x2="34.2519" y2="19.9644" width="0.3048" layer="16"/>
 <wire x1="34.2519" y1="19.9644" x2="34.29" y2="20.0025" width="0.3048" layer="16"/>
 <via x="34.29" y="20.0025" extent="1-16" drill="0.6"/>
@@
 <wire x1="38.989" y1="13.7795" x2="35.4905" y2="13.7795" width="0.3048" layer="1"/>
 <wire x1="35.4905" y1="13.7795" x2="35.4205" y2="13.8495" width="0.3048" layer="1"/>
-<wire x1="43.3705" y1="4.953" x2="43.311" y2="5.646" width="0" layer="19" extent="16-16"/>
+<contactref element="C5" pad="2"/>
+<contactref element="U$2" pad="1"/>
+<contactref element="IC3" pad="4"/>
+<contactref element="IC3" pad="2"/>
+<wire x1="44.323" y1="13.081" x2="45.212" y2="10.311" width="0" layer="19" extent="1-16"/>
+<wire x1="43.311" y1="5.646" x2="43.3705" y2="4.953" width="0" layer="19" extent="16-16"/>
+<wire x1="45.1485" y1="6.389" x2="45.466" y2="5.08" width="0" layer="19" extent="16-16"/>
+<wire x1="-8.9535" y1="3.226" x2="33.0835" y2="8.9535" width="0" layer="19" extent="1-1"/>
+<wire x1="-8.9535" y1="-2.9718" x2="-8.9535" y2="3.226" width="0" layer="19" extent="1-1"/>
 </signal>
 <signal name="N$15">
@@
 <contactref element="L1" pad="2"/>
 <contactref element="K1" pad="1"/>
-<contactref element="IC2" pad="1"/>
 <contactref element="C4" pad="+"/>
 <contactref element="D4" pad="A"/>
@@
 <wire x1="28.565" y1="17.0915" x2="30.734" y2="14.9225" width="0.3048" layer="16"/>
 <wire x1="30.734" y1="14.9225" x2="31.2928" y2="14.9225" width="0.3048" layer="16"/>
-<wire x1="31.2928" y1="14.9225" x2="31.2547" y2="15.3416" width="0.3048" layer="16"/>
 <wire x1="26.543" y1="9.7155" x2="26.543" y2="9.906" width="0.3048" layer="16"/>
 <wire x1="26.543" y1="9.906" x2="26.2255" y2="10.2235" width="0.3048" layer="16"/>
@@
 <wire x1="40.5765" y1="16.002" x2="39.6875" y2="14.986" width="0.3048" layer="16"/>
 <wire x1="39.6875" y1="14.986" x2="31.5468" y2="14.986" width="0.3048" layer="16"/>
-<wire x1="31.5468" y1="14.986" x2="31.2547" y2="15.3416" width="0.3048" layer="16"/>
 <wire x1="26.543" y1="9.7155" x2="26.543" y2="9.2075" width="0.3048" layer="1"/>
 <wire x1="26.543" y1="9.2075" x2="25.019" y2="7.366" width="0.3048" layer="1"/>
@@
 <wire x1="21.1455" y1="6.477" x2="21.1455" y2="5.34735625" width="0.3048" layer="16"/>
 <wire x1="21.1455" y1="5.34735625" x2="21.1423" y2="5.34415625" width="0.3048" layer="16"/>
+<contactref element="IC3" pad="3"/>
+<contactref element="R7" pad="2"/>
+<wire x1="31.2928" y1="14.9225" x2="31.5468" y2="14.986" width="0" layer="19" extent="16-16"/>
+<wire x1="-6.6421" y1="-2.9718" x2="10.668" y2="9.525" width="0" layer="19" extent="1-1"/>
+<wire x1="-9.9085" y1="-7.4295" x2="-6.6421" y2="-2.9718" width="0" layer="19" extent="1-1"/>
 </signal>
 <signal name="N$6">
