File: Hardware/SchemasBoard/rolety.brd (EAGLE design)
At the start: 48.6 x 22.9 mm, 30 parts, among them IC1 LNK304, IC3 MC33269ST-3.3T3, K1 FRS1B, K2 FRS1B, T1 BC846, T2 BC846

Commit message: aaa
Parts:
- removed R7: 1 K, resistor:M2012
- D3: value (none) -> ES1D; device diode:DO214AA -> diode:DO214AC
- D4: value (none) -> 1N4007GP
- moved D3 0.06 mm to (34.0, 9.14)
Connections:
- net GND: no longer R7.1
- net N$27: no longer R7.2
Routing:
- net N$27: track 84.0 -> 77.3 mm, vias 4 -> 3
- net N$2: track 30.8 -> 32.3 mm
- net N$28: track 29.7 -> 30.2 mm
Other:
- board size 48.6 x 22.9 mm -> 48.9 x 22.9 mm
