File: Hardware/SchemasBoard/rolety.sch (EAGLE design)
At the start: 30 parts, among them IC1 LNK304, IC2 MCP1703DB, K1 FRS1B, K2 FRS1B, T1 BC846, T2 BC846

Commit message: aaa
Changed lines of the file:
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@@
 <wire x1="127" y1="66.04" x2="127" y2="55.88" width="0.1524" layer="91"/>
 <junction x="127" y="55.88"/>
-<wire x1="83.82" y1="66.04" x2="73.66" y2="66.04" width="0.1524" layer="91"/>
-<wire x1="73.66" y1="66.04" x2="73.66" y2="93.98" width="0.1524" layer="91"/>
-<wire x1="73.66" y1="93.98" x2="76.2" y2="93.98" width="0.1524" layer="91"/>
-<wire x1="76.2" y1="93.98" x2="76.2" y2="142.24" width="0.1524" layer="91"/>
-<junction x="83.82" y="66.04"/>
-<wire x1="76.2" y1="142.24" x2="33.02" y2="142.24" width="0.1524" layer="91"/>
 <wire x1="127" y1="55.88" x2="139.7" y2="55.88" width="0.1524" layer="91"/>
 <wire x1="139.7" y1="55.88" x2="147.32" y2="55.88" width="0.1524" layer="91"/>

Commit message: a
Connections:
- net N$5: now also U$2.RC6/AN8/SS
Changed lines of the file:
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@@
 <wire x1="2.54" y1="116.84" x2="2.54" y2="121.92" width="0.1524" layer="91"/>
 <wire x1="2.54" y1="121.92" x2="20.32" y2="121.92" width="0.1524" layer="91"/>
+<junction x="144.78" y="30.48"/>
 </segment>
 </net>
@@
 <wire x1="149.86" y1="106.68" x2="149.86" y2="142.24" width="0.1524" layer="91"/>
 <wire x1="149.86" y1="142.24" x2="86.36" y2="142.24" width="0.1524" layer="91"/>
-<wire x1="86.36" y1="142.24" x2="86.36" y2="116.84" width="0.1524" layer="91"/>
-</segment>
-</net>
+<wire x1="86.36" y1="142.24" x2="86.36" y2="119.38" width="0.1524" layer="91"/>
+<pinref part="U$2" gate="G$1" pin="RC6/AN8/SS"/>
+<junction x="86.36" y="119.38"/>
+<wire x1="86.36" y1="119.38" x2="86.36" y2="116.84" width="0.1524" layer="91"/>
+<junction x="147.32" y="106.68"/>
+</segment>
+</net>

Commit message: a
Parts:
- removed JP1: (no value), pinhead:PINHD-1X4
- added X1: (no value), con-ptr500:AK500/4
- L1: value BC12 -> MMICC7; device inductors:BC12 -> inductors:MMICC7
Connections:
- net N$36: now also X1-4.KL; no longer JP1.1
- net N$4: now also X1-3.KL; no longer JP1.2
- net N$7: now also X1-1.KL; no longer JP1.4
- net N$8: now also X1-2.KL; no longer JP1.3
Changed lines of the file:
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@@
 <part name="R7" library="resistor" deviceset="R-EU_" device="M2012" value="2 K"/>
 <part name="C3" library="resistor" deviceset="CPOL-EU" device="E2.5-5" value="10uF / 16 V"/>
-<part name="L1" library="inductors" deviceset="BC12" device=""/>
+<part name="L1" library="inductors" deviceset="MMICC7" device=""/>
 <part name="C4" library="resistor" deviceset="CPOL-EU" device="E2.5-5" value="100uF / 6,3 V"/>
 <part name="IC2" library="linear" deviceset="MCP1703" device="DB"/>
@@
 <part name="D4" library="diode" deviceset="DIODE-" device="DO214AA"/>
 <part name="D1" library="diode" deviceset="MBRA340T3" device=""/>
-<part name="JP1" library="pinhead" deviceset="PINHD-1X4" device=""/>
 <part name="C6" library="resistor" deviceset="CPOL-EU" device="SMCA" value="1uF"/>
 <part name="S1" library="switch-dil" deviceset="SD4-01" device=""/>
@@
 <part name="D2" library="diode" deviceset="MBRA340T3" device=""/>
 <part name="R6" library="resistor" deviceset="R-EU_" device="M2012" value="1 K"/>
+<part name="X1" library="con-ptr500" deviceset="AK500/4" device=""/>
 </parts>
 <sheets>
@@
 <instance part="R7" gate="G$1" x="93.98" y="40.64" rot="R90"/>
 <instance part="C3" gate="G$1" x="55.88" y="76.2"/>
-<instance part="L1" gate="G$1" x="76.2" y="53.34" rot="R90"/>
+<instance part="L1" gate="1" x="76.2" y="53.34" rot="R90"/>
 <instance part="C4" gate="G$1" x="86.36" y="38.1"/>
 <instance part="IC2" gate="G$1" x="111.76" y="55.88"/>
@@
 <instance part="D4" gate="G$1" x="66.04" y="78.74" rot="R180"/>
 <instance part="D1" gate="G$1" x="10.16" y="76.2" rot="R90"/>
-<instance part="JP1" gate="A" x="-22.86" y="55.88" rot="R180"/>
 <instance part="C6" gate="G$1" x="139.7" y="45.72"/>
 <instance part="S1" gate="1" x="147.32" y="99.06"/>
@@
 <instance part="D2" gate="G$1" x="10.16" y="93.98" rot="R90"/>
 <instance part="R6" gate="G$1" x="38.1" y="127"/>
+<instance part="X1" gate="-1" x="-38.1" y="63.5"/>
+<instance part="X1" gate="-2" x="-38.1" y="58.42"/>
+<instance part="X1" gate="-3" x="-38.1" y="53.34"/>
+<instance part="X1" gate="-4" x="-38.1" y="48.26"/>
 </instances>
 <busses>
@@
 <wire x1="12.7" y1="38.1" x2="-5.08" y2="38.1" width="0.1524" layer="91"/>
 <wire x1="-5.08" y1="38.1" x2="-5.08" y2="53.34" width="0.1524" layer="91"/>
-<pinref part="JP1" gate="A" pin="2"/>
-<wire x1="-20.32" y1="53.34" x2="-5.08" y2="53.34" width="0.1524" layer="91"/>
+<pinref part="X1" gate="-3" pin="KL"/>
+<wire x1="-33.02" y1="53.34" x2="-5.08" y2="53.34" width="0.1524" layer="91"/>
 </segment>
 </net>
@@
 <wire x1="71.12" y1="40.64" x2="71.12" y2="45.72" width="0.1524" layer="91"/>
 <junction x="71.12" y="48.26"/>
-<pinref part="L1" gate="G$1" pin="1"/>
+<pinref part="L1" gate="1" pin="1"/>
 <wire x1="71.12" y1="45.72" x2="71.12" y2="48.26" width="0.1524" layer="91"/>
 <wire x1="76.2" y1="45.72" x2="71.12" y2="45.72" width="0.1524" layer="91"/>
@@
 <pinref part="R2" gate="G$1" pin="1"/>
 <wire x1="-7.62" y1="55.88" x2="-5.08" y2="55.88" width="0.1524" layer="91"/>
-<pinref part="JP1" gate="A" pin="1"/>
-<wire x1="-20.32" y1="50.8" x2="-7.62" y2="50.8" width="0.1524" layer="91"/>
-<wire x1="-7.62" y1="50.8" x2="-7.62" y2="55.88" width="0.1524" layer="91"/>
+<wire x1="-7.62" y1="48.26" x2="-7.62" y2="55.88" width="0.1524" layer="91"/>
 <pinref part="K2" gate="2" pin="P@1"/>
 <wire x1="-17.78" y1="83.82" x2="-25.4" y2="83.82" width="0.1524" layer="91"/>
@@
 <wire x1="-7.62" y1="63.5" x2="-7.62" y2="55.88" width="0.1524" layer="91"/>
 <junction x="-7.62" y="55.88"/>
+<pinref part="X1" gate="-4" pin="KL"/>
+<wire x1="-33.02" y1="48.26" x2="-7.62" y2="48.26" width="0.1524" layer="91"/>
 </segment>
 </net>
@@
 <segment>
 <pinref part="K1" gate="2" pin="S"/>
-<wire x1="-20.32" y1="78.74" x2="-22.86" y2="78.74" width="0.1524" layer="91"/>
-<pinref part="JP1" gate="A" pin="4"/>
-<wire x1="-20.32" y1="58.42" x2="-22.86" y2="58.42" width="0.1524" layer="91"/>
-<wire x1="-22.86" y1="58.42" x2="-22.86" y2="78.74" width="0.1524" layer="91"/>
+<pinref part="X1" gate="-1" pin="KL"/>
+<wire x1="-33.02" y1="63.5" x2="-30.48" y2="63.5" width="0.1524" layer="91"/>
+<wire x1="-30.48" y1="63.5" x2="-30.48" y2="78.74" width="0.1524" layer="91"/>
+<wire x1="-30.48" y1="78.74" x2="-20.32" y2="78.74" width="0.1524" layer="91"/>
 </segment>
 </net>
@@
 <wire x1="0" y1="99.06" x2="10.16" y2="99.06" width="0.1524" layer="91"/>
 <wire x1="10.16" y1="99.06" x2="10.16" y2="96.52" width="0.1524" layer="91"/>
-<pinref part="L1" gate="G$1" pin="2"/>
+<pinref part="L1" gate="1" pin="2"/>
 <wire x1="68.58" y1="78.74" x2="76.2" y2="78.74" width="0.1524" layer="91"/>
 <wire x1="76.2" y1="78.74" x2="76.2" y2="60.96" width="0.1524" layer="91"/>
@@
 <net name="N$8" class="0">
 <segment>
-<pinref part="JP1" gate="A" pin="3"/>
 <pinref part="K2" gate="2" pin="S"/>
 <wire x1="-20.32" y1="91.44" x2="-27.94" y2="91.44" width="0.1524" layer="91"/>
-<wire x1="-27.94" y1="91.44" x2="-27.94" y2="55.88" width="0.1524" layer="91"/>
-<wire x1="-27.94" y1="55.88" x2="-20.32" y2="55.88" width="0.1524" layer="91"/>
-</segment>
-</net>
+<wire x1="-27.94" y1="91.44" x2="-27.94" y2="58.42" width="0.1524" layer="91"/>
+<pinref part="X1" gate="-2" pin="KL"/>
+<wire x1="-33.02" y1="58.42" x2="-27.94" y2="58.42" width="0.1524" layer="91"/>
+</segment>
+</net>

Commit message: ghj
Parts:
- S1: value (none) -> DTS-3; device switch-dil:SD4-01 -> switch-tact:DTS-3
Changed lines of the file:
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@@
 <part name="D1" library="diode" deviceset="MBRA340T3" device=""/>
 <part name="C6" library="resistor" deviceset="CPOL-EU" device="SMCA" value="1uF"/>
-<part name="S1" library="switch-dil" deviceset="SD4-01" device=""/>
+<part name="S1" library="switch-tact" deviceset="DTS-3" device=""/>
 <part name="K2" library="relay" deviceset="FRS1B" device="">
 <attribute name="MF" value=""/>
@@
 <instance part="D1" gate="G$1" x="10.16" y="76.2" rot="R90"/>
 <instance part="C6" gate="G$1" x="139.7" y="45.72"/>
-<instance part="S1" gate="1" x="147.32" y="99.06"/>
+<instance part="S1" gate="G$1" x="149.86" y="96.52"/>
 <instance part="K2" gate="1" x="0" y="93.98" smashed="yes">
 <attribute name="VALUE" x="1.27" y="96.901" size="1.778" layer="96"/>
@@
 <wire x1="139.7" y1="40.64" x2="139.7" y2="30.48" width="0.1524" layer="91"/>
 <junction x="139.7" y="30.48"/>
-<pinref part="S1" gate="1" pin="1"/>
-<wire x1="147.32" y1="91.44" x2="144.78" y2="91.44" width="0.1524" layer="91"/>
+<pinref part="S1" gate="G$1" pin="1"/>
+<wire x1="149.86" y1="91.44" x2="144.78" y2="91.44" width="0.1524" layer="91"/>
 <wire x1="144.78" y1="91.44" x2="144.78" y2="30.48" width="0.1524" layer="91"/>
 <pinref part="T2" gate="G$1" pin="E"/>
@@
 <net name="N$5" class="0">
 <segment>
-<pinref part="S1" gate="1" pin="2"/>
-<wire x1="147.32" y1="106.68" x2="149.86" y2="106.68" width="0.1524" layer="91"/>
-<wire x1="149.86" y1="106.68" x2="149.86" y2="142.24" width="0.1524" layer="91"/>
+<pinref part="S1" gate="G$1" pin="2"/>
+<wire x1="149.86" y1="101.6" x2="149.86" y2="142.24" width="0.1524" layer="91"/>
 <wire x1="149.86" y1="142.24" x2="86.36" y2="142.24" width="0.1524" layer="91"/>
 <wire x1="86.36" y1="142.24" x2="86.36" y2="119.38" width="0.1524" layer="91"/>
@@
 <junction x="86.36" y="119.38"/>
 <wire x1="86.36" y1="119.38" x2="86.36" y2="116.84" width="0.1524" layer="91"/>
-<junction x="147.32" y="106.68"/>
-</segment>
-</net>
+<junction x="149.86" y="101.6"/>
+</segment>
+</net>

Commit message: aaa
Parts:
- removed JP2: (no value), pinhead:PINHD-1X5
- removed R7: 2 K, resistor:R-EU_M2012
- added U$3: PROGRAMMINGHEADERDIP, rfm70:PROGRAMMINGHEADERDIP
- C1: device resistor:CPOL-EUE5-13 -> resistor:CPOL-EUE5-10.5
Connections:
- net GND: now also U$3.GND; no longer JP2.3, R7.1
- net N$17: now also U$3.VDD; no longer JP2.2
- net N$18: now also U$3.PGD; no longer JP2.4
- net N$19: now also U$3.PGC; no longer JP2.5
- net N$25: now also U$3.MCLR; no longer JP2.1
- net N$27: no longer R7.2
Changed lines of the file:
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@@
 <part name="U$2" library="microchip" deviceset="PIC16F690*" device=""/>
 <part name="K1" library="relay" deviceset="FRS1B" device=""/>
-<part name="C1" library="resistor" deviceset="CPOL-EU" device="E5-13" value="3,3uF"/>
-<part name="JP2" library="pinhead" deviceset="PINHD-1X5" device=""/>
+<part name="C1" library="resistor" deviceset="CPOL-EU" device="E5-10.5" value="3,3uF"/>
 <part name="C2" library="resistor" deviceset="C-EU" device="C2012" value="100nF"/>
 <part name="R3" library="resistor" deviceset="R-EU_" device="M2012" value="3.9 k"/>
 <part name="R4" library="resistor" deviceset="R-EU_" device="M2012" value="2,05 k"/>
 <part name="R5" library="resistor" deviceset="R-EU_" device="M2012" value="1 K"/>
-<part name="R7" library="resistor" deviceset="R-EU_" device="M2012" value="2 K"/>
 <part name="C3" library="resistor" deviceset="CPOL-EU" device="E2.5-5" value="10uF / 16 V"/>
 <part name="L1" library="inductors" deviceset="MMICC7" device=""/>
@@
 <part name="R6" library="resistor" deviceset="R-EU_" device="M2012" value="1 K"/>
 <part name="X1" library="con-ptr500" deviceset="AK500/4" device=""/>
+<part name="U$3" library="rfm70" deviceset="PROGRAMMINGHEADER" device="" technology="DIP"/>
 </parts>
 <sheets>
@@
 <instance part="K1" gate="2" x="-15.24" y="73.66"/>
 <instance part="C1" gate="G$1" x="22.86" y="38.1"/>
-<instance part="JP2" gate="A" x="162.56" y="121.92"/>
 <instance part="C2" gate="G$1" x="43.18" y="71.12" rot="R90"/>
 <instance part="R3" gate="G$1" x="30.48" y="58.42"/>
 <instance part="R4" gate="G$1" x="35.56" y="66.04" rot="R90"/>
 <instance part="R5" gate="G$1" x="55.88" y="116.84"/>
-<instance part="R7" gate="G$1" x="93.98" y="40.64" rot="R90"/>
 <instance part="C3" gate="G$1" x="55.88" y="76.2"/>
 <instance part="L1" gate="1" x="76.2" y="53.34" rot="R90"/>
@@
 <instance part="X1" gate="-3" x="-38.1" y="53.34"/>
 <instance part="X1" gate="-4" x="-38.1" y="48.26"/>
+<instance part="U$3" gate="G$1" x="177.8" y="134.62"/>
 </instances>
 <busses>
@@
 <wire x1="22.86" y1="30.48" x2="71.12" y2="30.48" width="0.1524" layer="91"/>
 <wire x1="71.12" y1="30.48" x2="86.36" y2="30.48" width="0.1524" layer="91"/>
-<wire x1="86.36" y1="30.48" x2="93.98" y2="30.48" width="0.1524" layer="91"/>
-<wire x1="93.98" y1="30.48" x2="111.76" y2="30.48" width="0.1524" layer="91"/>
+<wire x1="86.36" y1="30.48" x2="111.76" y2="30.48" width="0.1524" layer="91"/>
 <wire x1="111.76" y1="30.48" x2="127" y2="30.48" width="0.1524" layer="91"/>
 <wire x1="127" y1="30.48" x2="132.08" y2="30.48" width="0.1524" layer="91"/>
@@
 <wire x1="71.12" y1="35.56" x2="71.12" y2="30.48" width="0.1524" layer="91"/>
 <junction x="71.12" y="30.48"/>
-<pinref part="R7" gate="G$1" pin="1"/>
-<wire x1="93.98" y1="35.56" x2="93.98" y2="30.48" width="0.1524" layer="91"/>
-<junction x="93.98" y="30.48"/>
 <pinref part="IC2" gate="G$1" pin="GND"/>
 <wire x1="111.76" y1="48.26" x2="111.76" y2="30.48" width="0.1524" layer="91"/>
@@
 <wire x1="172.72" y1="68.58" x2="177.8" y2="68.58" width="0.1524" layer="91"/>
 <wire x1="177.8" y1="68.58" x2="177.8" y2="30.48" width="0.1524" layer="91"/>
-<wire x1="160.02" y1="121.92" x2="177.8" y2="121.92" width="0.1524" layer="91"/>
-<wire x1="177.8" y1="121.92" x2="177.8" y2="68.58" width="0.1524" layer="91"/>
 <junction x="177.8" y="68.58"/>
 <pinref part="T1" gate="G$1" pin="E"/>
+<wire x1="177.8" y1="119.38" x2="177.8" y2="68.58" width="0.1524" layer="91"/>
 <wire x1="10.16" y1="68.58" x2="20.32" y2="68.58" width="0.1524" layer="91"/>
 <wire x1="20.32" y1="68.58" x2="20.32" y2="30.48" width="0.1524" layer="91"/>
@@
 <junction x="86.36" y="30.48"/>
 <pinref part="D3" gate="G$1" pin="A"/>
-<pinref part="JP2" gate="A" pin="3"/>
 <wire x1="20.32" y1="121.92" x2="20.32" y2="68.58" width="0.1524" layer="91"/>
 <junction x="20.32" y="68.58"/>
@@
 <wire x1="2.54" y1="121.92" x2="20.32" y2="121.92" width="0.1524" layer="91"/>
 <junction x="144.78" y="30.48"/>
+<pinref part="U$3" gate="G$1" pin="GND"/>
+<wire x1="167.64" y1="134.62" x2="162.56" y2="134.62" width="0.1524" layer="91"/>
+<wire x1="162.56" y1="134.62" x2="162.56" y2="119.38" width="0.1524" layer="91"/>
+<wire x1="162.56" y1="119.38" x2="177.8" y2="119.38" width="0.1524" layer="91"/>
 </segment>
 </net>
@@
 <wire x1="139.7" y1="55.88" x2="147.32" y2="55.88" width="0.1524" layer="91"/>
 <wire x1="147.32" y1="55.88" x2="147.32" y2="73.66" width="0.1524" layer="91"/>
-<pinref part="JP2" gate="A" pin="2"/>
 <pinref part="U$1" gate="G$1" pin="VDD"/>
 <wire x1="170.18" y1="68.58" x2="170.18" y2="73.66" width="0.1524" layer="91"/>
-<wire x1="170.18" y1="73.66" x2="170.18" y2="124.46" width="0.1524" layer="91"/>
-<wire x1="170.18" y1="124.46" x2="160.02" y2="124.46" width="0.1524" layer="91"/>
+<wire x1="170.18" y1="73.66" x2="170.18" y2="106.68" width="0.1524" layer="91"/>
+<wire x1="170.18" y1="106.68" x2="160.02" y2="106.68" width="0.1524" layer="91"/>
+<wire x1="160.02" y1="106.68" x2="160.02" y2="132.08" width="0.1524" layer="91"/>
 <wire x1="147.32" y1="73.66" x2="170.18" y2="73.66" width="0.1524" layer="91"/>
 <junction x="170.18" y="73.66"/>
@@
 <wire x1="139.7" y1="48.26" x2="139.7" y2="55.88" width="0.1524" layer="91"/>
 <junction x="139.7" y="55.88"/>
-</segment>
-</net>
-<net name="N$18" class="0">
-<segment>
-<wire x1="144.78" y1="119.38" x2="144.78" y2="132.08" width="0.1524" layer="91"/>
-<pinref part="U$2" gate="G$1" pin="RA0/AN0/C1IN+/ICSPDAT/ULPWU"/>
-<wire x1="144.78" y1="132.08" x2="132.08" y2="132.08" width="0.1524" layer="91"/>
-<wire x1="132.08" y1="132.08" x2="132.08" y2="119.38" width="0.1524" layer="91"/>
-<pinref part="JP2" gate="A" pin="4"/>
-<wire x1="160.02" y1="119.38" x2="144.78" y2="119.38" width="0.1524" layer="91"/>
-</segment>
-</net>
-<net name="N$19" class="0">
-<segment>
-<wire x1="147.32" y1="116.84" x2="147.32" y2="134.62" width="0.1524" layer="91"/>
-<pinref part="U$2" gate="G$1" pin="RA1/AN1/C12IN0-/VREF/ICSPCLK"/>
-<wire x1="147.32" y1="134.62" x2="129.54" y2="134.62" width="0.1524" layer="91"/>
-<wire x1="129.54" y1="134.62" x2="129.54" y2="119.38" width="0.1524" layer="91"/>
-<pinref part="JP2" gate="A" pin="5"/>
-<wire x1="147.32" y1="116.84" x2="160.02" y2="116.84" width="0.1524" layer="91"/>
+<pinref part="U$3" gate="G$1" pin="VDD"/>
+<wire x1="160.02" y1="132.08" x2="167.64" y2="132.08" width="0.1524" layer="91"/>
 </segment>
 </net>
@@
 <pinref part="U$2" gate="G$1" pin="RA2/AN2/T0CKI/INT/C1OUT"/>
 <wire x1="127" y1="119.38" x2="127" y2="139.7" width="0.1524" layer="91"/>
-<wire x1="127" y1="139.7" x2="165.1" y2="139.7" width="0.1524" layer="91"/>
+<wire x1="127" y1="139.7" x2="157.48" y2="139.7" width="0.1524" layer="91"/>
 <pinref part="U$1" gate="G$1" pin="CE"/>
-<wire x1="165.1" y1="139.7" x2="165.1" y2="68.58" width="0.1524" layer="91"/>
+<wire x1="157.48" y1="139.7" x2="157.48" y2="101.6" width="0.1524" layer="91"/>
+<wire x1="157.48" y1="101.6" x2="165.1" y2="101.6" width="0.1524" layer="91"/>
+<wire x1="165.1" y1="101.6" x2="165.1" y2="68.58" width="0.1524" layer="91"/>
 </segment>
 </net>
@@
 <net name="N$25" class="0">
 <segment>
+<pinref part="U$3" gate="G$1" pin="MCLR"/>
+<wire x1="154.94" y1="129.54" x2="167.64" y2="129.54" width="0.1524" layer="91"/>
+<wire x1="154.94" y1="129.54" x2="154.94" y2="132.08" width="0.1524" layer="91"/>
 <pinref part="U$2" gate="G$1" pin="RA3/MCLR/VPP"/>
-<wire x1="124.46" y1="119.38" x2="124.46" y2="137.16" width="0.1524" layer="91"/>
-<pinref part="JP2" gate="A" pin="1"/>
-<wire x1="124.46" y1="137.16" x2="160.02" y2="137.16" width="0.1524" layer="91"/>
-<wire x1="160.02" y1="137.16" x2="160.02" y2="127" width="0.1524" layer="91"/>
+<wire x1="154.94" y1="132.08" x2="124.46" y2="132.08" width="0.1524" layer="91"/>
+<wire x1="124.46" y1="132.08" x2="124.46" y2="119.38" width="0.1524" layer="91"/>
 </segment>
 </net>
@@
 <wire x1="0" y1="81.28" x2="0" y2="83.82" width="0.1524" layer="91"/>
 <pinref part="IC2" gate="G$1" pin="VI"/>
-<pinref part="R7" gate="G$1" pin="2"/>
-<wire x1="93.98" y1="45.72" x2="93.98" y2="55.88" width="0.1524" layer="91"/>
-<wire x1="93.98" y1="55.88" x2="101.6" y2="55.88" width="0.1524" layer="91"/>
-<junction x="93.98" y="55.88"/>
-<wire x1="93.98" y1="55.88" x2="86.36" y2="55.88" width="0.1524" layer="91"/>
+<wire x1="101.6" y1="55.88" x2="86.36" y2="55.88" width="0.1524" layer="91"/>
 <wire x1="76.2" y1="60.96" x2="86.36" y2="60.96" width="0.1524" layer="91"/>
 <wire x1="86.36" y1="60.96" x2="86.36" y2="55.88" width="0.1524" layer="91"/>
@@
 </segment>
 </net>
+<net name="N$18" class="0">
+<segment>
+<pinref part="U$2" gate="G$1" pin="RA0/AN0/C1IN+/ICSPDAT/ULPWU"/>
+<wire x1="132.08" y1="119.38" x2="132.08" y2="137.16" width="0.1524" layer="91"/>
+<pinref part="U$3" gate="G$1" pin="PGD"/>
+<wire x1="132.08" y1="137.16" x2="167.64" y2="137.16" width="0.1524" layer="91"/>
+</segment>
+</net>
+<net name="N$19" class="0">
+<segment>
+<pinref part="U$2" gate="G$1" pin="RA1/AN1/C12IN0-/VREF/ICSPCLK"/>
+<wire x1="129.54" y1="119.38" x2="129.54" y2="134.62" width="0.1524" layer="91"/>
+<wire x1="129.54" y1="134.62" x2="160.02" y2="134.62" width="0.1524" layer="91"/>
+<wire x1="160.02" y1="134.62" x2="160.02" y2="139.7" width="0.1524" layer="91"/>
+<pinref part="U$3" gate="G$1" pin="PGC"/>
+<wire x1="160.02" y1="139.7" x2="167.64" y2="139.7" width="0.1524" layer="91"/>
+</segment>
+</net>

Commit message: a
Parts:
- L1: value MMICC7 -> MICC10; device inductors:MMICC7 -> inductors:MICC10
Changed lines of the file:
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@@
 <part name="R5" library="resistor" deviceset="R-EU_" device="M2012" value="1 K"/>
 <part name="C3" library="resistor" deviceset="CPOL-EU" device="E2.5-5" value="10uF / 16 V"/>
-<part name="L1" library="inductors" deviceset="MMICC7" device=""/>
+<part name="L1" library="inductors" deviceset="MICC10" device=""/>
 <part name="C4" library="resistor" deviceset="CPOL-EU" device="E2.5-5" value="100uF / 6,3 V"/>
 <part name="IC2" library="linear" deviceset="MCP1703" device="DB"/>
