File: Hardware/SchemasBoard/tempSensorCR2032.brd (EAGLE design)
At the start: 22.2 x 24.1 mm, 9 parts, among them IC1 DS1820

Commit message: aaa
Connections:
- removed net N$5: C1.1, R1.2, U$2.1, U$3.VDD, U$4.1
- net N$4: now also C1.1, R1.2, U$2.1, U$3.VDD, U$4.1; no longer U$2.15, U$2.6, U$2.7, U$2.8
Routing:
- net N$5: track 47.6 -> 0.00 mm, vias 2 -> 0
- net N$4: track 57.6 -> 61.3 mm
Changed lines of the file:
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@@
 </signal>
 <signal name="N$23">
-<contactref element="U$2" pad="9"/>
 <contactref element="U$1" pad="MOSI"/>
 <wire x1="9.1184" y1="9.1321" x2="7.6843" y2="9.1321" width="0.3048" layer="16"/>
@@
 <wire x1="7.4803" y1="4.9149" x2="14.3129" y2="4.9149" width="0.3048" layer="16"/>
 <wire x1="17.6403" y1="10.2235" x2="20.124" y2="10.2235" width="0.3048" layer="16"/>
-<wire x1="20.124" y1="10.2235" x2="20.1477" y2="10.2472" width="0.3048" layer="16"/>
 <wire x1="17.6403" y1="10.2235" x2="17.2085" y2="9.779" width="0.3048" layer="16"/>
 <wire x1="17.2085" y1="9.779" x2="17.1704" y2="7.7851" width="0.3048" layer="16"/>
 <wire x1="17.1704" y1="7.7851" x2="14.3129" y2="4.9149" width="0.3048" layer="16"/>
+<contactref element="U$2" pad="9"/>
+<wire x1="20.124" y1="10.2235" x2="20.1477" y2="10.2472" width="0" layer="19" extent="16-16"/>
 </signal>
 <signal name="N$25">
@@
 </signal>
 <signal name="N$4">
-<contactref element="U$2" pad="6"/>
-<contactref element="U$2" pad="7"/>
 <contactref element="U$1" pad="VDD"/>
-<contactref element="C2" pad="+"/>
-<wire x1="20.1477" y1="11.5472" x2="20.1477" y2="12.1972" width="0.3048" layer="16"/>
 <wire x1="5.08" y1="17.78" x2="8.89" y2="13.97" width="0.254" layer="16"/>
 <wire x1="3.81" y1="17.78" x2="5.08" y2="17.78" width="0.254" layer="16"/>
 <wire x1="1.27" y1="20.32" x2="3.81" y2="17.78" width="0.254" layer="16"/>
 <wire x1="8.89" y1="13.97" x2="9.1184" y2="14.3321" width="0.254" layer="16"/>
-<wire x1="1.27" y1="20.32" x2="1.8147" y2="19.8755" width="0.254" layer="16"/>
-<wire x1="20.1477" y1="12.1972" x2="18.8774" y2="12.1972" width="0.3048" layer="16"/>
-<wire x1="18.8774" y1="12.1972" x2="16.1925" y2="9.5123" width="0.3048" layer="16"/>
-<via x="16.1925" y="9.5123" extent="1-16" drill="0.6"/>
-<wire x1="16.1925" y1="9.5123" x2="16.1671" y2="7.5565" width="0.3048" layer="1"/>
-<wire x1="16.1671" y1="7.5565" x2="12.7127" y2="3.9751" width="0.3048" layer="1"/>
-<wire x1="12.7127" y1="3.9751" x2="9.8679" y2="3.9751" width="0.3048" layer="1"/>
-<wire x1="9.8679" y1="3.9751" x2="8.2042" y2="2.3114" width="0.3048" layer="1"/>
-<wire x1="8.2042" y1="2.3114" x2="6.3246" y2="2.3114" width="0.3048" layer="1"/>
-<wire x1="6.3246" y1="2.3114" x2="4.1529" y2="4.4831" width="0.3048" layer="1"/>
-<wire x1="4.1529" y1="4.4831" x2="4.1529" y2="15.1384" width="0.3048" layer="1"/>
-<wire x1="4.1529" y1="15.1384" x2="1.5875" y2="18.0848" width="0.3048" layer="1"/>
-<via x="1.5875" y="18.0848" extent="1-16" drill="0.6"/>
-<wire x1="1.5875" y1="18.0848" x2="1.2065" y2="19.534" width="0.3048" layer="16"/>
-<wire x1="1.2065" y1="19.534" x2="1.8147" y2="19.8755" width="0.3048" layer="16"/>
-<contactref element="U$2" pad="8"/>
-<contactref element="U$2" pad="15"/>
-<wire x1="16.1925" y1="9.5123" x2="14.1605" y2="9.5123" width="0.3048" layer="16"/>
-<wire x1="14.1605" y1="9.5123" x2="14.1605" y2="12.2047" width="0.3048" layer="16"/>
-<wire x1="14.1605" y1="12.2047" x2="12.8977" y2="12.2047" width="0.3048" layer="16"/>
-<wire x1="12.8977" y1="12.2047" x2="12.8977" y2="12.1972" width="0.3048" layer="16"/>
-<wire x1="20.1477" y1="11.5472" x2="20.1477" y2="10.8972" width="0.3048" layer="16"/>
-</signal>
-<signal name="N$5">
 <contactref element="U$4" pad="1"/>
 <contactref element="U$2" pad="1"/>
@@
 <contactref element="U$3" pad="VDD"/>
 <contactref element="U$3" pad="VDD"/>
+<contactref element="C1" pad="1"/>
 <wire x1="11.43" y1="2.54" x2="13.97" y2="2.54" width="0.254" layer="16"/>
 <wire x1="13.97" y1="2.54" x2="13.9315" y2="2.032" width="0.254" layer="16"/>
@@
 <wire x1="18.669" y1="15.4178" x2="18.8341" y2="15.3162" width="0.3048" layer="1"/>
 <wire x1="18.8341" y1="15.3162" x2="18.26895" y2="14.75105" width="0.3048" layer="1"/>
-<contactref element="C1" pad="1"/>
 <wire x1="14.6238" y1="18.4825" x2="14.6304" y2="18.4825" width="0.3048" layer="1"/>
 <wire x1="14.6304" y1="18.4825" x2="14.6304" y2="20.3073" width="0.3048" layer="1"/>
@@
 <via x="1.1684" y="22.2377" extent="1-16" drill="0.6"/>
 <wire x1="1.1684" y1="22.2377" x2="2.5536" y2="22.2377" width="0.3048" layer="16"/>
+<contactref element="C2" pad="+"/>
+<wire x1="1.8147" y1="19.8755" x2="1.1684" y2="19.8755" width="0.3048" layer="16"/>
+<wire x1="1.1684" y1="19.8755" x2="1.1684" y2="22.2377" width="0.3048" layer="16"/>
+<wire x1="1.1684" y1="19.8755" x2="1.27" y2="20.32" width="0" layer="19" extent="16-16"/>
 </signal>
 </signals>

Commit message: a
Parts:
- moved U$1 0.80 mm to (-4.39, 15.7)
Routing:
- net N$12: track 12.7 -> 14.0 mm
- net VD: track 45.7 -> 46.7 mm
- net N$16: track 3.97 -> 3.05 mm
- net N$20: track 4.25 -> 3.39 mm
- net N$22: track 19.6 -> 20.1 mm
