File: Hardware/SchemasBoard/tempSensorCR2032.sch (EAGLE design)
At the start: 11 parts, among them IC1 DS1820, T2 BC846

Commit message: a
Connections:
- removed net N$10: U$3.GND
- net GND: now also U$3.GND
- net VDD: now also U$3.VDD
Changed lines of the file:
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@@
 <instance part="C2" gate="G$1" x="43.18" y="58.42"/>
 <instance part="R1" gate="G$1" x="160.02" y="111.76" rot="R270"/>
-<instance part="U$3" gate="G$1" x="187.96" y="127"/>
+<instance part="U$3" gate="G$1" x="185.42" y="127"/>
 <instance part="T2" gate="G$1" x="175.26" y="35.56"/>
 <instance part="R3" gate="G$1" x="142.24" y="35.56"/>
@@
 <net name="GND" class="0">
 <segment>
-<wire x1="132.08" y1="30.48" x2="177.8" y2="30.48" width="0.1524" layer="91"/>
+<wire x1="132.08" y1="30.48" x2="147.32" y2="30.48" width="0.1524" layer="91"/>
 <pinref part="U$2" gate="G$1" pin="VSS"/>
+<wire x1="147.32" y1="30.48" x2="177.8" y2="30.48" width="0.1524" layer="91"/>
 <wire x1="132.08" y1="66.04" x2="132.08" y2="30.48" width="0.1524" layer="91"/>
 <pinref part="IC1" gate="G$1" pin="GND"/>
@@
 <wire x1="109.22" y1="40.64" x2="109.22" y2="30.48" width="0.1524" layer="91"/>
 <junction x="109.22" y="30.48"/>
+<pinref part="U$3" gate="G$1" pin="GND"/>
+<wire x1="175.26" y1="127" x2="147.32" y2="127" width="0.1524" layer="91"/>
+<wire x1="147.32" y1="127" x2="147.32" y2="30.48" width="0.1524" layer="91"/>
+<junction x="147.32" y="30.48"/>
 </segment>
 <segment>
@@
 <wire x1="160.02" y1="101.6" x2="160.02" y2="106.68" width="0.1524" layer="91"/>
 <wire x1="170.18" y1="101.6" x2="170.18" y2="124.46" width="0.1524" layer="91"/>
-<wire x1="170.18" y1="124.46" x2="180.34" y2="124.46" width="0.1524" layer="91"/>
 <junction x="170.18" y="101.6"/>
 <pinref part="G1" gate="1" pin="+"/>
 <wire x1="109.22" y1="50.8" x2="109.22" y2="63.5" width="0.1524" layer="91"/>
 <junction x="109.22" y="63.5"/>
+<pinref part="U$3" gate="G$1" pin="VDD"/>
+<wire x1="175.26" y1="124.46" x2="170.18" y2="124.46" width="0.1524" layer="91"/>
 </segment>
 <segment>
@@
 <pinref part="U$3" gate="G$1" pin="MCLR"/>
 <wire x1="160.02" y1="121.92" x2="160.02" y2="116.84" width="0.1524" layer="91"/>
-<wire x1="177.8" y1="121.92" x2="160.02" y2="121.92" width="0.1524" layer="91"/>
+<wire x1="175.26" y1="121.92" x2="160.02" y2="121.92" width="0.1524" layer="91"/>
 <junction x="160.02" y="121.92"/>
 </segment>
@@
 <wire x1="132.08" y1="119.38" x2="132.08" y2="132.08" width="0.1524" layer="91"/>
 <pinref part="U$3" gate="G$1" pin="PGD"/>
-<wire x1="177.8" y1="129.54" x2="154.94" y2="129.54" width="0.1524" layer="91"/>
+<wire x1="175.26" y1="129.54" x2="154.94" y2="129.54" width="0.1524" layer="91"/>
 <wire x1="154.94" y1="129.54" x2="154.94" y2="132.08" width="0.1524" layer="91"/>
 <wire x1="154.94" y1="132.08" x2="132.08" y2="132.08" width="0.1524" layer="91"/>
@@
 <segment>
 <pinref part="U$3" gate="G$1" pin="PGC"/>
-<wire x1="177.8" y1="132.08" x2="167.64" y2="132.08" width="0.1524" layer="91"/>
+<wire x1="175.26" y1="132.08" x2="167.64" y2="132.08" width="0.1524" layer="91"/>
 <wire x1="167.64" y1="132.08" x2="167.64" y2="134.62" width="0.1524" layer="91"/>
 <pinref part="U$2" gate="G$1" pin="RA1/AN1/C12IN0-/VREF/ICSPCLK"/>
@@
 </segment>
 </net>
-<net name="N$10" class="0">
-<segment>
-<pinref part="U$3" gate="G$1" pin="GND"/>
-<wire x1="172.72" y1="127" x2="177.8" y2="127" width="0.1524" layer="91"/>
-</segment>
-</net>

Commit message: \zxcv
Parts:
- removed G1: CR2032H, battery:CR2032H
- removed R3: 1K, resistor:R-EU_R1206W
- removed T2: BC846, transistor:BC846
- added U$4: CR2032, rfm70:CR2032
Connections:
- removed net N$13: T2.C, U$1.GND
- removed net N$14: R3.2, T2.B
- removed net N$15: R3.1, U$2.RC1/AN5/C12IN1-
- new net N$4: U$1.VDD, U$2.RC3/AN7C12IN3-/P1C, U$2.RC4/C2OUT/P1B
- net GND: now also R1.2, U$1.GND, U$2.VDD, U$3.VDD, U$4.GND, U$4.VDD; no longer G1.-, T2.E
- net VDD: no longer G1.+, R1.2, U$1.VDD, U$2.VDD, U$3.VDD
Changed lines of the file:
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@@
 <part name="R1" library="resistor" deviceset="R-EU_" device="R1206W" value="4K7"/>
 <part name="U$3" library="rfm70" deviceset="PROGRAMMINGHEADER" device="" technology="DIP"/>
-<part name="T2" library="transistor" deviceset="BC846" device=""/>
-<part name="R3" library="resistor" deviceset="R-EU_" device="R1206W" value="1K"/>
-<part name="G1" library="battery" deviceset="CR2032H" device=""/>
+<part name="U$4" library="rfm70" deviceset="CR2032" device=""/>
 </parts>
 <sheets>
@@
 <instance part="R1" gate="G$1" x="160.02" y="111.76" rot="R270"/>
 <instance part="U$3" gate="G$1" x="185.42" y="127"/>
-<instance part="T2" gate="G$1" x="175.26" y="35.56"/>
-<instance part="R3" gate="G$1" x="142.24" y="35.56"/>
-<instance part="G1" gate="1" x="109.22" y="45.72" rot="R90"/>
+<instance part="U$4" gate="G$1" x="104.14" y="50.8" rot="R180"/>
 </instances>
 <busses>
@@
 <nets>
 <net name="GND" class="0">
-<segment>
-<wire x1="132.08" y1="30.48" x2="147.32" y2="30.48" width="0.1524" layer="91"/>
-<pinref part="U$2" gate="G$1" pin="VSS"/>
-<wire x1="147.32" y1="30.48" x2="177.8" y2="30.48" width="0.1524" layer="91"/>
-<wire x1="132.08" y1="66.04" x2="132.08" y2="30.48" width="0.1524" layer="91"/>
-<pinref part="IC1" gate="G$1" pin="GND"/>
-<wire x1="58.42" y1="91.44" x2="58.42" y2="30.48" width="0.1524" layer="91"/>
-<wire x1="58.42" y1="30.48" x2="73.66" y2="30.48" width="0.1524" layer="91"/>
-<junction x="132.08" y="30.48"/>
-<wire x1="73.66" y1="30.48" x2="109.22" y2="30.48" width="0.1524" layer="91"/>
-<label x="154.94" y="30.48" size="1.778" layer="95"/>
-<pinref part="S1" gate="G$1" pin="1"/>
-<wire x1="109.22" y1="30.48" x2="132.08" y2="30.48" width="0.1524" layer="91"/>
-<wire x1="73.66" y1="66.04" x2="73.66" y2="30.48" width="0.1524" layer="91"/>
-<junction x="73.66" y="30.48"/>
-<junction x="132.08" y="66.04"/>
-<pinref part="T2" gate="G$1" pin="E"/>
-<pinref part="G1" gate="1" pin="-"/>
-<wire x1="109.22" y1="40.64" x2="109.22" y2="30.48" width="0.1524" layer="91"/>
-<junction x="109.22" y="30.48"/>
-<pinref part="U$3" gate="G$1" pin="GND"/>
-<wire x1="175.26" y1="127" x2="147.32" y2="127" width="0.1524" layer="91"/>
-<wire x1="147.32" y1="127" x2="147.32" y2="30.48" width="0.1524" layer="91"/>
-<junction x="147.32" y="30.48"/>
-</segment>
 <segment>
 <pinref part="C1" gate="G$1" pin="2"/>
@@
 <wire x1="43.18" y1="53.34" x2="43.18" y2="50.8" width="0.1524" layer="91"/>
 <junction x="43.18" y="50.8"/>
+</segment>
+<segment>
+<wire x1="83.82" y1="63.5" x2="109.22" y2="63.5" width="0.1524" layer="91"/>
+<label x="104.14" y="63.5" size="1.778" layer="95"/>
+<pinref part="U$2" gate="G$1" pin="VDD"/>
+<wire x1="109.22" y1="63.5" x2="139.7" y2="63.5" width="0.1524" layer="91"/>
+<wire x1="83.82" y1="66.04" x2="83.82" y2="63.5" width="0.1524" layer="91"/>
+<wire x1="139.7" y1="63.5" x2="139.7" y2="73.66" width="0.1524" layer="91"/>
+<wire x1="170.18" y1="73.66" x2="170.18" y2="101.6" width="0.1524" layer="91"/>
+<wire x1="170.18" y1="101.6" x2="160.02" y2="101.6" width="0.1524" layer="91"/>
+<wire x1="139.7" y1="73.66" x2="170.18" y2="73.66" width="0.1524" layer="91"/>
+<pinref part="R1" gate="G$1" pin="2"/>
+<wire x1="160.02" y1="101.6" x2="160.02" y2="106.68" width="0.1524" layer="91"/>
+<wire x1="170.18" y1="101.6" x2="170.18" y2="124.46" width="0.1524" layer="91"/>
+<junction x="170.18" y="101.6"/>
+<wire x1="109.22" y1="50.8" x2="109.22" y2="63.5" width="0.1524" layer="91"/>
+<junction x="109.22" y="63.5"/>
+<pinref part="U$3" gate="G$1" pin="VDD"/>
+<wire x1="175.26" y1="124.46" x2="170.18" y2="124.46" width="0.1524" layer="91"/>
+<pinref part="U$4" gate="G$1" pin="VDD"/>
+<wire x1="114.3" y1="40.64" x2="114.3" y2="50.8" width="0.1524" layer="91"/>
+<pinref part="U$4" gate="G$1" pin="GND"/>
+<wire x1="114.3" y1="50.8" x2="109.22" y2="50.8" width="0.1524" layer="91"/>
+<wire x1="132.08" y1="30.48" x2="147.32" y2="30.48" width="0.1524" layer="91"/>
+<pinref part="U$2" gate="G$1" pin="VSS"/>
+<wire x1="147.32" y1="30.48" x2="177.8" y2="30.48" width="0.1524" layer="91"/>
+<wire x1="132.08" y1="66.04" x2="132.08" y2="30.48" width="0.1524" layer="91"/>
+<label x="154.94" y="30.48" size="1.778" layer="95"/>
+<junction x="132.08" y="66.04"/>
+<pinref part="U$3" gate="G$1" pin="GND"/>
+<wire x1="175.26" y1="127" x2="147.32" y2="127" width="0.1524" layer="91"/>
+<wire x1="147.32" y1="127" x2="147.32" y2="30.48" width="0.1524" layer="91"/>
+<junction x="147.32" y="30.48"/>
+<wire x1="177.8" y1="30.48" x2="177.8" y2="68.58" width="0.1524" layer="91"/>
+<pinref part="U$1" gate="G$1" pin="GND"/>
+<wire x1="177.8" y1="68.58" x2="172.72" y2="68.58" width="0.1524" layer="91"/>
+<wire x1="111.76" y1="40.64" x2="111.76" y2="30.48" width="0.1524" layer="91"/>
+<wire x1="111.76" y1="30.48" x2="132.08" y2="30.48" width="0.1524" layer="91"/>
+<pinref part="S1" gate="G$1" pin="1"/>
+<wire x1="73.66" y1="66.04" x2="73.66" y2="30.48" width="0.1524" layer="91"/>
+<pinref part="IC1" gate="G$1" pin="GND"/>
+<wire x1="58.42" y1="91.44" x2="58.42" y2="30.48" width="0.1524" layer="91"/>
+<wire x1="58.42" y1="30.48" x2="73.66" y2="30.48" width="0.1524" layer="91"/>
+<wire x1="111.76" y1="30.48" x2="73.66" y2="30.48" width="0.1524" layer="91"/>
+<wire x1="114.3" y1="40.64" x2="111.76" y2="40.64" width="0.1524" layer="91"/>
 </segment>
 </net>
@@
 <net name="VDD" class="0">
 <segment>
-<wire x1="83.82" y1="63.5" x2="109.22" y2="63.5" width="0.1524" layer="91"/>
-<label x="104.14" y="63.5" size="1.778" layer="95"/>
-<pinref part="U$2" gate="G$1" pin="VDD"/>
-<wire x1="109.22" y1="63.5" x2="139.7" y2="63.5" width="0.1524" layer="91"/>
-<wire x1="83.82" y1="66.04" x2="83.82" y2="63.5" width="0.1524" layer="91"/>
-<wire x1="139.7" y1="63.5" x2="139.7" y2="73.66" width="0.1524" layer="91"/>
-<pinref part="U$1" gate="G$1" pin="VDD"/>
-<wire x1="170.18" y1="68.58" x2="170.18" y2="73.66" width="0.1524" layer="91"/>
-<wire x1="170.18" y1="73.66" x2="170.18" y2="101.6" width="0.1524" layer="91"/>
-<wire x1="170.18" y1="101.6" x2="160.02" y2="101.6" width="0.1524" layer="91"/>
-<wire x1="139.7" y1="73.66" x2="170.18" y2="73.66" width="0.1524" layer="91"/>
-<junction x="170.18" y="73.66"/>
-<pinref part="R1" gate="G$1" pin="2"/>
-<wire x1="160.02" y1="101.6" x2="160.02" y2="106.68" width="0.1524" layer="91"/>
-<wire x1="170.18" y1="101.6" x2="170.18" y2="124.46" width="0.1524" layer="91"/>
-<junction x="170.18" y="101.6"/>
-<pinref part="G1" gate="1" pin="+"/>
-<wire x1="109.22" y1="50.8" x2="109.22" y2="63.5" width="0.1524" layer="91"/>
-<junction x="109.22" y="63.5"/>
-<pinref part="U$3" gate="G$1" pin="VDD"/>
-<wire x1="175.26" y1="124.46" x2="170.18" y2="124.46" width="0.1524" layer="91"/>
-</segment>
-<segment>
 <pinref part="C1" gate="G$1" pin="1"/>
 <wire x1="35.56" y1="60.96" x2="35.56" y2="63.5" width="0.1524" layer="91"/>
@@
 </segment>
 </net>
-<net name="N$13" class="0">
-<segment>
-<pinref part="T2" gate="G$1" pin="C"/>
-<wire x1="177.8" y1="40.64" x2="177.8" y2="68.58" width="0.1524" layer="91"/>
-<pinref part="U$1" gate="G$1" pin="GND"/>
-<wire x1="177.8" y1="68.58" x2="172.72" y2="68.58" width="0.1524" layer="91"/>
-</segment>
-</net>
-<net name="N$14" class="0">
-<segment>
-<pinref part="T2" gate="G$1" pin="B"/>
-<pinref part="R3" gate="G$1" pin="2"/>
-<wire x1="147.32" y1="35.56" x2="172.72" y2="35.56" width="0.1524" layer="91"/>
-</segment>
-</net>
-<net name="N$15" class="0">
-<segment>
-<pinref part="U$2" gate="G$1" pin="RC1/AN5/C12IN1-"/>
-<wire x1="99.06" y1="119.38" x2="99.06" y2="121.92" width="0.1524" layer="91"/>
-<wire x1="99.06" y1="121.92" x2="76.2" y2="121.92" width="0.1524" layer="91"/>
-<wire x1="76.2" y1="121.92" x2="76.2" y2="35.56" width="0.1524" layer="91"/>
-<pinref part="R3" gate="G$1" pin="1"/>
-<wire x1="76.2" y1="35.56" x2="137.16" y2="35.56" width="0.1524" layer="91"/>
-</segment>
-</net>
+<net name="N$4" class="0">
+<segment>
+<pinref part="U$2" gate="G$1" pin="RC4/C2OUT/P1B"/>
+<pinref part="U$2" gate="G$1" pin="RC3/AN7C12IN3-/P1C"/>
+<wire x1="91.44" y1="119.38" x2="93.98" y2="119.38" width="0.1524" layer="91"/>
+<wire x1="93.98" y1="119.38" x2="93.98" y2="139.7" width="0.1524" layer="91"/>
+<wire x1="93.98" y1="139.7" x2="124.46" y2="139.7" width="0.1524" layer="91"/>
+<wire x1="124.46" y1="139.7" x2="124.46" y2="142.24" width="0.1524" layer="91"/>
+<wire x1="124.46" y1="142.24" x2="195.58" y2="142.24" width="0.1524" layer="91"/>
+<wire x1="195.58" y1="142.24" x2="195.58" y2="76.2" width="0.1524" layer="91"/>
+<wire x1="195.58" y1="76.2" x2="172.72" y2="76.2" width="0.1524" layer="91"/>
+<wire x1="172.72" y1="76.2" x2="172.72" y2="71.12" width="0.1524" layer="91"/>
+<pinref part="U$1" gate="G$1" pin="VDD"/>
+<wire x1="172.72" y1="71.12" x2="170.18" y2="71.12" width="0.1524" layer="91"/>
+<wire x1="170.18" y1="71.12" x2="170.18" y2="68.58" width="0.1524" layer="91"/>
+<junction x="91.44" y="119.38"/>
+<junction x="93.98" y="119.38"/>
+</segment>
+</net>
