File: Hardware/SchemasBoard/6relayBoard.brd (EAGLE design)
At the start: 48.6 x 22.9 mm, 30 parts, among them IC1 LNK304, IC3 MC33269ST-3.3T3, K1 FRS1B, K2 FRS1B, T1 BC846, T2 BC846

Commit message: aa
Parts:
- added D5, D6, D7, D8: MBRA340T3, diode:SMA
- added K3, K4, K5, K6: FRS1B, relay:FRS1B
- added R10, R11, R8, R9: 1 K, resistor:M2012
- added T3, T4, T5, T6: BC846, transistor:SOT23
- added X2: (no value), con-ptr500:AK500/4
- moved C6 4.62 mm to (50.5, 13.8)
- moved S1 4.58 mm to (46.6, 22.5)
- moved C5 4.57 mm to (50.5, 8.70)
- moved U$3 4.18 mm to (46.8, 18.7)
- moved U$2 3.43 mm to (43.6, 11.6)
- moved U$1 2.86 mm to (48.6, 1.21)
- moved R7 1.42 mm to (44.1, 6.54)
Connections:
- new net N$30: D5.A, K5.2, T3.3
- new net N$31: D6.A, K4.2, T4.3
- new net N$32: D7.A, K3.2, T5.3
- new net N$33: D8.A, K6.2, T6.3
- new net N$34: K6.S, X2.1
- new net N$37: K3.S, X2.2
- new net N$38: K5.S, X2.4
- new net N$39: K4.S, X2.3
- new net N$41: R8.2, T3.1
- new net N$42: R9.2, T4.1
- new net N$43: R10.2, T5.1
- new net N$44: R11.2, T6.1
- new net N$45: R10.1, U$2.5
- new net N$46: R9.1, U$2.6
- new net N$47: R8.1, U$2.7
- net GND: now also T3.2, T4.2, T5.2, T6.2
- net N$27: now also D5.C, D6.C, D7.C, D8.C, K4.1, K5.1, K6.1
- net N$29: now also R11.1
- net N$36: now also K3.P, K3.P@, K4.P, K4.P@, K5.P, K5.P@, K6.P, K6.P@
Routing:
- net N$36: track 9.35 -> 79.4 mm
- net N$17: track 59.3 -> 6.20 mm
- net N$38: track 0.00 -> 52.9 mm
- net N$39: track 0.00 -> 39.6 mm
- net GND: track 113.4 -> 74.0 mm, vias 4 -> 2
- net N$18: track 34.4 -> 0.00 mm, vias 1 -> 0
- net N$37: track 0.00 -> 28.5 mm
- net N$47: track 0.00 -> 27.0 mm
- net N$5: track 22.8 -> 0.00 mm, vias 1 -> 0
- net N$19: track 16.3 -> 0.00 mm, vias 1 -> 0
- net N$16: track 15.5 -> 0.00 mm, vias 1 -> 0
- net N$20: track 11.2 -> 0.00 mm, vias 1 -> 0
- net N$21: track 10.6 -> 0.00 mm, vias 1 -> 0
- net N$25: track 10.1 -> 0.00 mm
- net N$12: track 9.71 -> 0.00 mm, vias 1 -> 0
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Other:
- board size 48.6 x 22.9 mm -> 53.1 x 41.8 mm

Commit message: aaa
Parts:
- moved R11 7.80 mm to (20.4, 24.4)
- moved D5 6.06 mm to (43.0, 34.5), turned to 90 degrees
- moved D6 5.21 mm to (31.9, 35.0), turned to 90 degrees
- moved D7 3.70 mm to (20.8, 34.9), turned to 270 degrees
- moved R10 2.55 mm to (23.2, 29.5), turned to 90 degrees
- moved T5 2.41 mm to (26.4, 33.2), turned to 90 degrees
- moved T6 1.53 mm to (15.6, 32.8), turned to 90 degrees
- moved C5 0.32 mm to (50.8, 8.70)
- moved T3 0.19 mm to (49.6, 33.3)
- moved U$3 0.19 mm to (46.6, 18.7)
- moved R9 0.13 mm to (34.6, 30.5)
- moved C6 0.06 mm to (50.6, 13.8)
- turned D8 to 180 degrees
Connections:
- net N$27: now also K3.1
Routing:
- net GND: track 74.0 -> 199.4 mm, vias 2 -> 6
- net N$27: track 85.2 -> 198.8 mm, vias 4 -> 6
- net N$17: track 6.20 -> 52.8 mm, vias 0 -> 4
- net N$45: track 0.00 -> 34.9 mm
- net N$29: track 0.00 -> 30.7 mm, vias 0 -> 2
- net N$21: track 0.00 -> 27.9 mm, vias 0 -> 1
- net N$46: track 0.00 -> 24.1 mm
- net N$18: track 0.00 -> 15.4 mm, vias 0 -> 1
- net N$31: track 0.00 -> 14.8 mm, vias 0 -> 2
- net N$20: track 0.00 -> 14.6 mm, vias 0 -> 1
- net N$44: track 0.00 -> 13.8 mm
- net N$5: track 0.00 -> 12.9 mm
- net N$16: track 0.00 -> 12.7 mm, vias 0 -> 1
- net N$12: track 0.00 -> 11.5 mm, vias 0 -> 1
- net N$19: track 0.00 -> 11.0 mm, vias 0 -> 1
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