File: Hardware/SchemasBoard/6relayBoard.brd (EAGLE design)
At the start: 53.1 x 41.8 mm, 47 parts, among them IC1 LNK304, IC3 MC33269ST-3.3T3, K1 FRS1B, K2 FRS1B, K3 FRS1B, K4 FRS1B, K5 FRS1B, K6 FRS1B, T1 BC846, T2 BC846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

Commit message: aaa
Parts:
- removed R7: 1 K, resistor:M2012
- D3: value (none) -> ES1D; device diode:DO214AA -> diode:DO214AC
- D4: value (none) -> 1N4007GP
Connections:
- net GND: no longer R7.1
- net N$27: no longer R7.2
Routing:
- net N$27: track 198.8 -> 188.7 mm, vias 6 -> 5
- net GND: track 217.9 -> 215.3 mm
- net N$13: track 32.3 -> 32.8 mm
Changed lines of the file:
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@@
 <grid distance="0.0635" unitdist="mm" unit="mm" style="lines" multiple="1" display="no" altdistance="1" altunitdist="mm" altunit="mm"/>
 <layers>
-<layer number="1" name="Top" color="1" fill="1" visible="no" active="yes"/>
+<layer number="1" name="Top" color="1" fill="1" visible="yes" active="yes"/>
 <layer number="16" name="Bottom" color="12" fill="1" visible="yes" active="yes"/>
 <layer number="17" name="Pads" color="2" fill="1" visible="yes" active="yes"/>
@@
 <element name="C5" library="resistor" package="C2012" value="100nF" x="50.8" y="8.6995" rot="MR270"/>
 <element name="T1" library="transistor" package="SOT23" value="BC846" x="13.208" y="1.778" rot="MR270"/>
-<element name="D3" library="diode" package="DO214AA" value="" x="33.9725" y="9.2075" rot="MR90"/>
-<element name="D4" library="diode" package="DO214AA" value="" x="23.9395" y="14.732" rot="MR90"/>
+<element name="D3" library="diode" package="DO214AC" value="ES1D" x="33.9725" y="9.2075" rot="MR90"/>
+<element name="D4" library="diode" package="DO214AA" value="1N4007GP" x="23.9395" y="14.732" rot="MR90"/>
 <element name="D1" library="diode" package="SMA" value="MBRA340T3" x="17.399" y="3.3655" rot="MR270"/>
 <element name="C6" library="resistor" package="SMC_A" value="1uF" x="50.6095" y="13.7795" rot="MR270"/>
@@
 <element name="U$3" library="rfm70" package="PROGHEADER" value="PROGRAMMINGHEADERDIP" x="46.609" y="18.669"/>
 <element name="IC3" library="linear" package="SOT223" value="MC33269ST-3.3T3" x="32.893" y="18.034" rot="MR180"/>
-<element name="R7" library="resistor" package="M2012" value="1 K" x="44.069" y="6.5405" rot="MR0"/>
 <element name="L2" library="inductor-neosid" package="BS11" value="680uH" x="28.5115" y="8.3185">
 <attribute name="OC_NEWARK" value="unknown" x="28.5115" y="8.3185" size="1.778" layer="27" display="off"/>
@@
 <wire x1="10.729" y1="12.4485" x2="12.3825" y2="10.795" width="0.3048" layer="16"/>
 <contactref element="IC3" pad="1"/>
-<contactref element="R7" pad="1"/>
 <wire x1="23.307" y1="19.855" x2="23.307" y2="19.3015" width="0.3048" layer="16"/>
 <wire x1="23.307" y1="19.3015" x2="24.003" y2="18.6055" width="0.3048" layer="16"/>
@@
 <wire x1="30.607" y1="13.3985" x2="33.7185" y2="13.3985" width="0.3048" layer="16"/>
 <wire x1="33.7185" y1="13.3985" x2="33.9725" y2="12.954" width="0.3048" layer="16"/>
-<wire x1="33.9725" y1="12.954" x2="33.9725" y2="11.7575" width="0.3048" layer="16"/>
+<wire x1="33.9725" y1="12.954" x2="33.9725" y2="11.2575" width="0.3048" layer="16"/>
 <contactref element="T3" pad="2"/>
 <contactref element="T4" pad="2"/>
@@
 <wire x1="47.309" y1="8.636" x2="47.2495" y2="8.6955" width="0.3048" layer="16"/>
 <wire x1="47.2495" y1="8.6955" x2="47.174" y2="8.6955" width="0.3048" layer="16"/>
-<wire x1="47.174" y1="8.6955" x2="45.019" y2="6.5405" width="0.3048" layer="16"/>
 <wire x1="50.6095" y1="12.2795" x2="50.8635" y2="12.954" width="0.3048" layer="16"/>
 <wire x1="50.8635" y1="12.954" x2="51.816" y2="13.9065" width="0.3048" layer="16"/>
@@
 <wire x1="22.225" y1="1.9685" x2="22.225" y2="4.992" width="0.3048" layer="16"/>
 <wire x1="22.225" y1="4.992" x2="22.6305" y2="5.588" width="0.3048" layer="16"/>
-<wire x1="33.9725" y1="6.6575" x2="33.9725" y2="4.6355" width="0.3048" layer="16"/>
+<wire x1="33.9725" y1="7.1575" x2="33.9725" y2="4.6355" width="0.3048" layer="16"/>
 <wire x1="33.9725" y1="4.6355" x2="33.2105" y2="3.8735" width="0.3048" layer="16"/>
 <wire x1="33.2105" y1="3.8735" x2="32.0675" y2="3.8735" width="0.3048" layer="16"/>
@@
 <wire x1="18.796" y1="10.668" x2="18.415" y2="11.049" width="0.3048" layer="16"/>
 <contactref element="IC3" pad="3"/>
-<contactref element="R7" pad="2"/>
 <contactref element="L2" pad="2"/>
 <wire x1="18.542" y1="13.2715" x2="18.542" y2="16.129" width="0.3048" layer="16"/>
@@
 <wire x1="18.9865" y1="4.953" x2="18.9545" y2="5.0165" width="0.3048" layer="16"/>
 <wire x1="18.9545" y1="5.0165" x2="18.796" y2="5.3655" width="0.3048" layer="16"/>
-<wire x1="43.119" y1="6.5405" x2="41.722" y2="7.1095" width="0.3048" layer="16"/>
-<wire x1="41.722" y1="7.1095" x2="40.894" y2="7.5565" width="0.3048" layer="16"/>
-<via x="40.894" y="7.5565" extent="1-16" drill="0.6"/>
-<wire x1="40.894" y1="7.5565" x2="34.6075" y2="7.5565" width="0.3048" layer="1"/>
-<wire x1="34.6075" y1="7.5565" x2="33.8455" y2="8.636" width="0.3048" layer="1"/>
 <via x="33.8455" y="8.636" extent="1-16" drill="0.6"/>
 <wire x1="33.8455" y1="8.636" x2="31.4325" y2="8.636" width="0.3048" layer="16"/>

Commit message: asd
Parts:
- moved R2 0.32 mm to (13.1, 21.1)
Routing:
- net N$36: track 79.5 -> 80.3 mm
- net N$2: track 30.8 -> 31.4 mm
Changed lines of the file:
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@@
 <element name="B1" library="rectifier" package="TO-269AA" value="RECTIFIER" x="11.938" y="15.3035" rot="MR0"/>
 <element name="R1" library="resistor" package="R2512W" value="100" x="9.906" y="5.715" rot="MR180"/>
-<element name="R2" library="resistor" package="R2512W" value="8,2" x="13.1445" y="20.828" rot="MR180"/>
+<element name="R2" library="resistor" package="R2512W" value="8,2" x="13.1445" y="21.1455" rot="MR180"/>
 <element name="U$1" library="rfm70" package="RFM70" value="RFM70" x="48.5775" y="1.2065" rot="R180"/>
 <element name="U$2" library="microchip" package="SSOP20" value="PIC16F690" x="43.6245" y="11.6205" rot="MR90"/>
@@
 <wire x1="13.716" y1="8.3185" x2="12.192" y2="7.747" width="0.3048" layer="16"/>
 <wire x1="12.192" y1="7.747" x2="7.01" y2="5.715" width="0.3048" layer="16"/>
-<wire x1="13.208" y1="14.859" x2="14.351" y2="14.859" width="0.3048" layer="16"/>
-<wire x1="14.351" y1="14.859" x2="17.5895" y2="18.415" width="0.3048" layer="16"/>
-<wire x1="17.5895" y1="18.415" x2="21.717" y2="18.4785" width="0.3048" layer="16"/>
+<wire x1="13.208" y1="14.859" x2="16.1925" y2="14.859" width="0.3048" layer="16"/>
+<wire x1="16.1925" y1="14.859" x2="18.161" y2="18.4785" width="0.3048" layer="16"/>
+<wire x1="18.161" y1="18.4785" x2="21.717" y2="18.4785" width="0.3048" layer="16"/>
 <via x="21.717" y="18.4785" extent="1-16" drill="0.6"/>
 <wire x1="21.717" y1="18.4785" x2="26.2255" y2="18.415" width="0.3048" layer="1"/>
@@
 <contactref element="R2" pad="2"/>
 <contactref element="B1" pad="AC1"/>
-<wire x1="13.218" y1="18.1585" x2="13.208" y2="20.828" width="0.4064" layer="16"/>
-<wire x1="13.208" y1="20.828" x2="16.0405" y2="20.828" width="0.4064" layer="16"/>
+<wire x1="13.218" y1="18.1585" x2="16.002" y2="18.161" width="0.4064" layer="16"/>
+<wire x1="16.002" y1="18.161" x2="16.0405" y2="21.1455" width="0.4064" layer="16"/>
 </signal>
 <signal name="N$4">
@@
 <wire x1="8.382" y1="39.878" x2="8.382" y2="34.163" width="1.4224" layer="16"/>
 <wire x1="8.382" y1="34.163" x2="11.2395" y2="31.3055" width="1.4224" layer="16"/>
-<wire x1="11.2395" y1="31.3055" x2="11.2395" y2="21.819" width="1.4224" layer="16"/>
-<wire x1="11.2395" y1="21.819" x2="10.2485" y2="20.828" width="1.4224" layer="16"/>
-<wire x1="10.2485" y1="20.828" x2="8.509" y2="20.8915" width="1.4224" layer="16"/>
+<wire x1="11.2395" y1="31.3055" x2="11.176" y2="24.7015" width="1.4224" layer="16"/>
+<wire x1="11.176" y1="24.7015" x2="10.287" y2="24.7015" width="1.4224" layer="16"/>
+<wire x1="10.287" y1="24.7015" x2="10.287" y2="20.93" width="1.4224" layer="16"/>
+<wire x1="10.287" y1="20.7395" x2="10.287" y2="20.93" width="1.4224" layer="16"/>
+<wire x1="10.287" y1="20.93" x2="10.2485" y2="21.1455" width="1.4224" layer="16"/>
+<wire x1="10.2485" y1="21.1455" x2="8.509" y2="20.8915" width="1.4224" layer="16"/>
 <wire x1="8.509" y1="20.8915" x2="8.382" y2="20.8915" width="1.27" layer="16"/>
 </signal>

Commit message: aaa
Parts:
- added R7: 1 K, resistor:M2012
- C3: device resistor:E2,5-5 -> resistor:SMC_C
- R2: device resistor:R2512W -> resistor:0411/12
- moved R2 31.4 mm to (44.5, 23.4), turned to 0 degrees
- moved S1 17.4 mm to (50.1, 5.40), turned to 270 degrees
- moved C5 3.40 mm to (50.0, 5.40), turned to 0 degrees
- moved U$1 2.35 mm to (46.4, 1.97)
- moved D3 2.03 mm to (34.0, 11.2)
- moved C3 1.89 mm to (33.5, 3.87), flipped to the bottom
- moved C6 1.61 mm to (50.9, 15.4)
- moved R6 1.57 mm to (37.1, 8.06)
- moved R1 1.33 mm to (11.2, 5.71)
- moved U$3 0.83 mm to (46.5, 19.5)
- moved IC3 0.64 mm to (32.9, 18.7)
Connections:
- net GND: now also R7.1
- net N$27: now also R7.2
- net N$36: now also X1.1; no longer X1.4
- net N$4: now also X1.2; no longer X1.3
- net N$7: now also X1.3; no longer X1.1
- net N$8: now also X1.4; no longer X1.2
Routing:
- net N$36: track 80.3 -> 110.0 mm
- net N$3: track 5.77 -> 29.6 mm, vias 0 -> 1
- net GND: track 215.3 -> 236.1 mm, vias 7 -> 8
- net N$4: track 13.2 -> 33.8 mm, vias 0 -> 1
- net N$27: track 188.7 -> 205.0 mm, vias 5 -> 7
- net N$38: track 52.9 -> 63.3 mm
- net N$28: track 29.9 -> 24.2 mm
- net N$17: track 52.8 -> 58.1 mm, vias 4 -> 2
- net N$46: track 24.1 -> 28.9 mm
- net N$45: track 34.9 -> 39.7 mm
- net N$22: track 5.17 -> 9.67 mm
- net N$26: track 16.1 -> 20.5 mm
- net N$8: track 25.9 -> 21.8 mm
- net N$23: track 3.70 -> 7.49 mm
- net N$5: track 12.9 -> 16.3 mm, vias 0 -> 1
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Other:
- outline, holes or cut-outs redrawn

Commit message: fghf
Parts:
- moved R4 0.44 mm to (23.3, 2.22)
- moved C4 0.19 mm to (25.3, 2.79)
- moved D3 0.18 mm to (33.9, 11.1)
- moved C3 0.13 mm to (33.5, 4.00)
Routing:
- net N$27: track 205.0 -> 204.4 mm
- net N$35: track 48.4 -> 47.9 mm

Commit message: fixed bug.
Routing:
- net GND: track 236.0 -> 238.9 mm
Changed lines of the file:
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@@
 <?xml version="1.0" encoding="utf-8"?>
 <!DOCTYPE eagle SYSTEM "eagle.dtd">
-<eagle version="6.3">
+<eagle version="6.4">
 <drawing>
 <settings>
@@
 <wire x1="47.244" y1="21.6535" x2="46.609" y2="21.0185" width="0.3048" layer="16"/>
 <wire x1="46.609" y1="19.558" x2="46.5455" y2="19.4945" width="0.3048" layer="16"/>
-<wire x1="47.117" y1="8.636" x2="47.174" y2="8.6955" width="0" layer="19" extent="1-16"/>
+<wire x1="47.2495" y1="8.6955" x2="50.09" y2="8.6955" width="0.3048" layer="16"/>
+<wire x1="50.09" y1="8.6955" x2="50.09" y2="8.636" width="0.3048" layer="16"/>
 </signal>
 <signal name="N$11">
@@
 <wire x1="41.402" y1="7.8105" x2="40.5115" y2="8.382" width="0.3048" layer="16"/>
 <wire x1="40.5115" y1="8.382" x2="39.9995" y2="8.6955" width="0.3048" layer="16"/>
-<wire x1="44.704" y1="7.4295" x2="41.3385" y2="7.366" width="0.3048" layer="1"/>
+<wire x1="44.704" y1="7.366" x2="41.3385" y2="7.366" width="0.3048" layer="1"/>
 <wire x1="41.3385" y1="7.366" x2="41.3385" y2="7.6835" width="0.3048" layer="1"/>
 <wire x1="41.3385" y1="7.6835" x2="41.402" y2="7.8105" width="0.3048" layer="1"/>
 <wire x1="45.974" y1="10.414" x2="44.704" y2="9.017" width="0.3048" layer="1"/>
-<wire x1="44.704" y1="9.017" x2="44.704" y2="7.4295" width="0.3048" layer="1"/>
+<wire x1="44.704" y1="9.017" x2="44.704" y2="7.366" width="0.3048" layer="1"/>
 <wire x1="45.155" y1="16.2685" x2="45.155" y2="17.9005" width="0.3048" layer="1"/>
 <wire x1="45.155" y1="17.9005" x2="44.5135" y2="18.542" width="0.3048" layer="1"/>

Commit message: fixed bug
Parts:
- moved D3 0.19 mm to (33.7, 11.1)
Routing:
- net GND: track 238.9 -> 237.6 mm, vias 8 -> 7
- net N$29: track 31.0 -> 30.3 mm
Changed lines of the file:
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@@
 <element name="C5" library="resistor" package="C2012" value="100nF" x="49.9745" y="5.3975" rot="MR0"/>
 <element name="T1" library="transistor" package="SOT23" value="BC846" x="13.208" y="1.778" rot="MR270"/>
-<element name="D3" library="diode" package="DO214AC" value="ES1D" x="33.909" y="11.1125" rot="MR90"/>
+<element name="D3" library="diode" package="DO214AC" value="ES1D" x="33.7185" y="11.1125" rot="MR90"/>
 <element name="D4" library="diode" package="DO214AA" value="1N4007GP" x="23.9395" y="14.732" rot="MR90"/>
 <element name="D1" library="diode" package="SMA" value="MBRA340T3" x="17.399" y="3.3655" rot="MR270"/>
@@
 <wire x1="30.607" y1="13.3985" x2="33.7185" y2="13.3985" width="0.3048" layer="16"/>
 <wire x1="33.7185" y1="13.3985" x2="33.9725" y2="12.954" width="0.3048" layer="16"/>
-<wire x1="33.9725" y1="12.954" x2="33.909" y2="13.1625" width="0.3048" layer="16"/>
+<wire x1="33.9725" y1="12.954" x2="33.7185" y2="13.1625" width="0.3048" layer="16"/>
 <contactref element="T3" pad="2"/>
 <contactref element="T4" pad="2"/>
@@
 <wire x1="50.189" y1="14.6685" x2="50.8635" y2="13.867" width="0.3048" layer="16"/>
 <wire x1="50.8635" y1="13.867" x2="50.8635" y2="11.049" width="0.3048" layer="16"/>
-<wire x1="50.09" y1="8.636" x2="50.1015" y2="8.6475" width="0.3048" layer="16"/>
 <wire x1="50.1015" y1="8.6475" x2="50.1015" y2="10.287" width="0.3048" layer="16"/>
 <wire x1="50.1015" y1="10.287" x2="50.8635" y2="11.049" width="0.3048" layer="16"/>
@@
 <wire x1="50.8245" y1="7.9245" x2="50.1015" y2="8.6475" width="0.3048" layer="16"/>
 <wire x1="46.609" y1="21.0185" x2="46.609" y2="19.558" width="0.3048" layer="16"/>
-<via x="50.09" y="8.636" extent="1-16" drill="0.6"/>
-<wire x1="50.09" y1="8.636" x2="47.117" y2="8.636" width="0.3048" layer="1"/>
+<wire x1="48.566" y1="8.001" x2="47.117" y2="8.636" width="0.3048" layer="1"/>
 <wire x1="47.117" y1="8.636" x2="45.339" y2="6.858" width="0.3048" layer="1"/>
 <wire x1="45.339" y1="6.858" x2="40.259" y2="6.858" width="0.3048" layer="1"/>
@@
 <wire x1="47.244" y1="21.6535" x2="46.609" y2="21.0185" width="0.3048" layer="16"/>
 <wire x1="46.609" y1="19.558" x2="46.5455" y2="19.4945" width="0.3048" layer="16"/>
-<wire x1="47.2495" y1="8.6955" x2="50.09" y2="8.6955" width="0.3048" layer="16"/>
-<wire x1="50.09" y1="8.6955" x2="50.09" y2="8.636" width="0.3048" layer="16"/>
+<wire x1="47.2495" y1="8.6955" x2="50.1015" y2="8.6955" width="0.3048" layer="16"/>
+<wire x1="50.1015" y1="8.6955" x2="50.1015" y2="8.6475" width="0.3048" layer="16"/>
+<wire x1="47.117" y1="8.636" x2="47.174" y2="8.6955" width="0" layer="19" extent="1-16"/>
 </signal>
 <signal name="N$11">
@@
 <wire x1="22.1615" y1="1.9685" x2="22.1615" y2="4.992" width="0.3048" layer="16"/>
 <wire x1="22.1615" y1="4.992" x2="22.6305" y2="5.588" width="0.3048" layer="16"/>
-<wire x1="33.909" y1="9.0625" x2="34.036" y2="6.945" width="0.3048" layer="16"/>
+<wire x1="33.7185" y1="9.0625" x2="34.036" y2="6.945" width="0.3048" layer="16"/>
 <wire x1="34.036" y1="6.945" x2="33.4645" y2="6.5005" width="0.3048" layer="16"/>
 <wire x1="32.004" y1="10.795" x2="34.29" y2="8.382" width="0.3048" layer="1"/>
@@
 <wire x1="32.893" y1="15.57" x2="35.9285" y2="15.57" width="0.3048" layer="16"/>
 <wire x1="35.9285" y1="15.57" x2="35.8775" y2="14.4145" width="0.3048" layer="16"/>
-<wire x1="35.8775" y1="14.4145" x2="35.8775" y2="10.922" width="0.3048" layer="16"/>
-<via x="35.8775" y="10.922" extent="1-16" drill="0.6"/>
-<wire x1="35.8775" y1="10.922" x2="36.322" y2="10.3505" width="0.3048" layer="1"/>
-<wire x1="36.322" y1="10.3505" x2="41.402" y2="7.8105" width="0.3048" layer="1"/>
+<wire x1="35.8775" y1="14.4145" x2="35.433" y2="12.954" width="0.3048" layer="16"/>
+<via x="35.433" y="12.954" extent="1-16" drill="0.6"/>
+<wire x1="35.433" y1="12.954" x2="38.5445" y2="9.7155" width="0.3048" layer="1"/>
+<wire x1="38.5445" y1="9.7155" x2="41.402" y2="7.8105" width="0.3048" layer="1"/>
 <via x="41.402" y="7.8105" extent="1-16" drill="0.6"/>
 <wire x1="41.402" y1="7.8105" x2="40.5115" y2="8.382" width="0.3048" layer="16"/>
@@
 <wire x1="43.1165" y1="10.0965" x2="41.91" y2="10.0965" width="0.3048" layer="16"/>
 <via x="41.91" y="10.0965" extent="1-16" drill="0.6"/>
-<wire x1="41.91" y1="10.0965" x2="38.9255" y2="10.0965" width="0.3048" layer="1"/>
-<wire x1="38.9255" y1="10.0965" x2="36.7665" y2="12.2555" width="0.3048" layer="1"/>
-<wire x1="36.7665" y1="12.2555" x2="35.7505" y2="12.2555" width="0.3048" layer="1"/>
-<wire x1="35.7505" y1="12.2555" x2="35.179" y2="12.827" width="0.3048" layer="1"/>
-<wire x1="35.179" y1="12.827" x2="35.179" y2="16.5735" width="0.3048" layer="1"/>
+<wire x1="41.91" y1="10.0965" x2="39.3065" y2="10.0965" width="0.3048" layer="1"/>
+<wire x1="39.3065" y1="10.0965" x2="36.7665" y2="14.0335" width="0.3048" layer="1"/>
+<wire x1="36.7665" y1="14.0335" x2="35.179" y2="14.0335" width="0.3048" layer="1"/>
+<wire x1="35.179" y1="14.0335" x2="35.179" y2="16.5735" width="0.3048" layer="1"/>
 <wire x1="35.179" y1="16.5735" x2="34.925" y2="16.891" width="0.3048" layer="1"/>
 <wire x1="34.925" y1="16.891" x2="34.925" y2="18.034" width="0.3048" layer="1"/>
@@
 <wire x1="39.9995" y1="9.9955" x2="35.941" y2="10.033" width="0.3048" layer="16"/>
 <wire x1="35.4965" y1="10.033" x2="34.925" y2="10.6045" width="0.3048" layer="16"/>
-<wire x1="34.925" y1="10.6045" x2="34.925" y2="11.9005" width="0.3048" layer="16"/>
-<wire x1="34.925" y1="11.9005" x2="32.9305" y2="11.9005" width="0.3048" layer="16"/>
-<wire x1="32.9305" y1="11.9005" x2="32.258" y2="12.065" width="0.3048" layer="16"/>
-<wire x1="32.258" y1="12.065" x2="32.258" y2="12.827" width="0.3048" layer="16"/>
-<wire x1="32.258" y1="12.827" x2="28.8925" y2="12.827" width="0.3048" layer="16"/>
+<wire x1="34.925" y1="10.6045" x2="34.925" y2="11.837" width="0.3048" layer="16"/>
+<wire x1="34.925" y1="11.837" x2="32.9305" y2="11.837" width="0.3048" layer="16"/>
+<wire x1="32.9305" y1="11.837" x2="32.0675" y2="11.811" width="0.3048" layer="16"/>
+<wire x1="32.0675" y1="11.811" x2="32.0675" y2="12.827" width="0.3048" layer="16"/>
+<wire x1="32.0675" y1="12.827" x2="28.8925" y2="12.827" width="0.3048" layer="16"/>
 <wire x1="28.8925" y1="12.827" x2="28.5115" y2="12.446" width="0.3048" layer="16"/>
 <via x="28.5115" y="12.446" extent="1-16" drill="0.6"/>
@@
 <wire x1="18.9865" y1="4.953" x2="18.9545" y2="5.0165" width="0.3048" layer="16"/>
 <wire x1="18.9545" y1="5.0165" x2="18.796" y2="5.3655" width="0.3048" layer="16"/>
-<via x="33.9725" y="11.049" extent="1-16" drill="0.6"/>
-<wire x1="33.9725" y1="11.049" x2="31.115" y2="11.049" width="0.3048" layer="16"/>
+<via x="33.9725" y="10.922" extent="1-16" drill="0.6"/>
+<wire x1="33.9725" y1="10.922" x2="31.115" y2="11.049" width="0.3048" layer="16"/>
 <wire x1="31.115" y1="11.049" x2="31.0115" y2="11.049" width="0.3048" layer="16"/>
 <wire x1="31.0115" y1="11.049" x2="31.0115" y2="8.3185" width="0.3048" layer="16"/>
@@
 <wire x1="35.2044" y1="19.8374" x2="33.9725" y2="18.6055" width="0.3048" layer="16"/>
 <via x="33.9725" y="18.6055" extent="1-16" drill="0.6"/>
-<wire x1="33.9725" y1="18.6055" x2="33.9725" y2="11.049" width="0.3048" layer="1"/>
+<wire x1="33.9725" y1="18.6055" x2="33.9725" y2="10.922" width="0.3048" layer="1"/>
 <wire x1="35.2044" y1="23.7744" x2="35.2044" y2="21.7678" width="0.3048" layer="16"/>
 </signal>
@@
 <wire x1="26.035" y1="19.4765" x2="25.207" y2="19.855" width="0.3048" layer="16"/>
 <wire x1="39.624" y1="7.62" x2="37.211" y2="7.62" width="0.3048" layer="1"/>
-<wire x1="37.211" y1="7.62" x2="34.7345" y2="10.0965" width="0.3048" layer="1"/>
-<wire x1="34.7345" y1="10.0965" x2="33.4645" y2="10.0965" width="0.3048" layer="1"/>
-<wire x1="33.4645" y1="10.0965" x2="32.893" y2="10.795" width="0.3048" layer="1"/>
+<wire x1="37.211" y1="7.62" x2="34.925" y2="9.906" width="0.3048" layer="1"/>
+<wire x1="34.925" y1="9.906" x2="33.655" y2="9.906" width="0.3048" layer="1"/>
+<wire x1="33.655" y1="9.906" x2="32.893" y2="10.795" width="0.3048" layer="1"/>
 <wire x1="32.893" y1="10.795" x2="32.893" y2="11.7475" width="0.3048" layer="1"/>
 </signal>
@@
 <wire x1="36.3855" y1="24.7015" x2="36.3855" y2="17.7165" width="0.3048" layer="16"/>
 <via x="35.941" y="17.7165" extent="1-16" drill="0.6"/>
-<wire x1="35.941" y1="17.7165" x2="35.941" y2="13.5255" width="0.3048" layer="1"/>
-<wire x1="35.941" y1="13.5255" x2="38.354" y2="13.5255" width="0.3048" layer="1"/>
-<via x="38.354" y="13.5255" extent="1-16" drill="0.6"/>
-<wire x1="38.354" y1="13.5255" x2="38.608" y2="13.5255" width="0.3048" layer="16"/>
+<wire x1="35.941" y1="17.7165" x2="35.941" y2="14.605" width="0.3048" layer="1"/>
+<wire x1="35.941" y1="14.605" x2="37.0205" y2="14.605" width="0.3048" layer="1"/>
+<wire x1="37.0205" y1="14.605" x2="38.4175" y2="13.9065" width="0.3048" layer="1"/>
+<via x="38.4175" y="13.9065" extent="1-16" drill="0.6"/>
+<wire x1="38.4175" y1="13.9065" x2="38.608" y2="13.5255" width="0.3048" layer="16"/>
 <wire x1="38.608" y1="13.5255" x2="38.9255" y2="13.208" width="0.3048" layer="16"/>
 <wire x1="38.9255" y1="13.208" x2="40.037" y2="13.208" width="0.3048" layer="16"/>
@@
 <wire x1="40.005" y1="19.4945" x2="39.6875" y2="19.2405" width="0.3048" layer="16"/>
 <wire x1="39.6875" y1="19.2405" x2="37.719" y2="17.5895" width="0.3048" layer="16"/>
-<wire x1="37.5285" y1="17.399" x2="36.449" y2="16.5735" width="0.3048" layer="16"/>
-<wire x1="36.449" y1="16.5735" x2="36.449" y2="11.811" width="0.3048" layer="16"/>
-<wire x1="36.449" y1="11.811" x2="36.957" y2="11.303" width="0.3048" layer="16"/>
+<wire x1="37.5285" y1="17.399" x2="36.5125" y2="16.637" width="0.3048" layer="16"/>
+<wire x1="36.5125" y1="16.637" x2="36.5125" y2="11.8745" width="0.3048" layer="16"/>
+<wire x1="36.5125" y1="11.8745" x2="36.957" y2="11.303" width="0.3048" layer="16"/>
 <wire x1="36.957" y1="11.303" x2="39.9995" y2="11.303" width="0.3048" layer="16"/>
 <wire x1="39.9995" y1="11.303" x2="39.9995" y2="11.2955" width="0.3048" layer="16"/>
