File: Hardware/SchemasBoard/heatingHeader.sch (EAGLE design)
At the start: 30 parts, among them IC1 DS1820

Commit message: a
Parts:
- added Q1: BSS123, transistor-small-signal:BSS123
Connections:
- new net N$11: JP1.1, Q1.D
- new net N$28: Q1.G, U$2.RB5/AN11/RX/DT
- net VDD: now also Q1.S; no longer JP1.1
Changed lines of the file:
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@@
 <part name="C1" library="resistor" deviceset="CPOL-EU" device="SMCA" value="1uF"/>
 <part name="C2" library="resistor" deviceset="C-EU" device="C2012" value="100nF"/>
+<part name="Q1" library="transistor-small-signal" deviceset="BSS123" device=""/>
 </parts>
 <sheets>
@@
 <instance part="C1" gate="G$1" x="10.16" y="50.8"/>
 <instance part="C2" gate="G$1" x="25.4" y="50.8"/>
+<instance part="Q1" gate="G$1" x="0" y="78.74"/>
 </instances>
 <busses>
@@
 <segment>
 <pinref part="U$2" gate="G$1" pin="VDD"/>
-<wire x1="0" y1="134.62" x2="0" y2="66.04" width="0.1524" layer="91"/>
 <wire x1="83.82" y1="66.04" x2="93.98" y2="66.04" width="0.1524" layer="91"/>
 <wire x1="93.98" y1="66.04" x2="144.78" y2="66.04" width="0.1524" layer="91"/>
@@
 <wire x1="10.16" y1="66.04" x2="25.4" y2="66.04" width="0.1524" layer="91"/>
 <wire x1="25.4" y1="66.04" x2="83.82" y2="66.04" width="0.1524" layer="91"/>
-<wire x1="0" y1="134.62" x2="5.08" y2="134.62" width="0.1524" layer="91"/>
-<pinref part="JP1" gate="A" pin="1"/>
 <label x="30.48" y="66.04" size="1.778" layer="95"/>
 <pinref part="C1" gate="G$1" pin="+"/>
@@
 <junction x="25.4" y="66.04"/>
 <junction x="170.18" y="66.04"/>
+<pinref part="Q1" gate="G$1" pin="S"/>
+<wire x1="0" y1="66.04" x2="0" y2="73.66" width="0.1524" layer="91"/>
 </segment>
 <segment>
@@
 </segment>
 </net>
+<net name="N$11" class="0">
+<segment>
+<pinref part="JP1" gate="A" pin="1"/>
+<wire x1="0" y1="134.62" x2="5.08" y2="134.62" width="0.1524" layer="91"/>
+<pinref part="Q1" gate="G$1" pin="D"/>
+<wire x1="0" y1="83.82" x2="0" y2="134.62" width="0.1524" layer="91"/>
+</segment>
+</net>
+<net name="N$28" class="0">
+<segment>
+<pinref part="U$2" gate="G$1" pin="RB5/AN11/RX/DT"/>
+<wire x1="111.76" y1="119.38" x2="111.76" y2="142.24" width="0.1524" layer="91"/>
+<wire x1="111.76" y1="142.24" x2="182.88" y2="142.24" width="0.1524" layer="91"/>
+<wire x1="182.88" y1="142.24" x2="182.88" y2="35.56" width="0.1524" layer="91"/>
+<pinref part="Q1" gate="G$1" pin="G"/>
+<wire x1="182.88" y1="35.56" x2="-5.08" y2="35.56" width="0.1524" layer="91"/>
+<wire x1="-5.08" y1="35.56" x2="-5.08" y2="76.2" width="0.1524" layer="91"/>
+</segment>
+</net>

Commit message: a
Parts:
- added R6: 4K7, resistor:R-EU_R1206W
Connections:
- net N$25: now also R6.1
- net VDD: now also R6.2
Changed lines of the file:
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@@
 <part name="C2" library="resistor" deviceset="C-EU" device="C2012" value="100nF"/>
 <part name="Q1" library="transistor-small-signal" deviceset="BSS123" device=""/>
+<part name="R6" library="resistor" deviceset="R-EU_" device="R1206W" value="4K7"/>
 </parts>
 <sheets>
@@
 <instance part="C2" gate="G$1" x="25.4" y="50.8"/>
 <instance part="Q1" gate="G$1" x="0" y="78.74"/>
+<instance part="R6" gate="G$1" x="172.72" y="134.62"/>
 </instances>
 <busses>
@@
 <pinref part="JP2" gate="A" pin="1"/>
 <wire x1="124.46" y1="137.16" x2="160.02" y2="137.16" width="0.1524" layer="91"/>
-<wire x1="160.02" y1="137.16" x2="160.02" y2="127" width="0.1524" layer="91"/>
+<wire x1="160.02" y1="137.16" x2="160.02" y2="134.62" width="0.1524" layer="91"/>
 <junction x="124.46" y="119.38"/>
+<pinref part="R6" gate="G$1" pin="1"/>
+<wire x1="160.02" y1="134.62" x2="160.02" y2="127" width="0.1524" layer="91"/>
+<wire x1="167.64" y1="134.62" x2="160.02" y2="134.62" width="0.1524" layer="91"/>
+<junction x="160.02" y="134.62"/>
 </segment>
 </net>
@@
 <wire x1="170.18" y1="68.58" x2="170.18" y2="124.46" width="0.1524" layer="91"/>
 <wire x1="170.18" y1="124.46" x2="160.02" y2="124.46" width="0.1524" layer="91"/>
-</segment>
-</net>
+<pinref part="R6" gate="G$1" pin="2"/>
+<wire x1="177.8" y1="134.62" x2="177.8" y2="124.46" width="0.1524" layer="91"/>
+<wire x1="177.8" y1="124.46" x2="170.18" y2="124.46" width="0.1524" layer="91"/>
+<junction x="170.18" y="124.46"/>
+</segment>
+</net>

Commit message: a
Parts:
- Q1: value BSS123 -> BSS84; device transistor-small-signal:BSS123 -> transistor-small-signal:BSS84
Changed lines of the file:
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@@
 <part name="C1" library="resistor" deviceset="CPOL-EU" device="SMCA" value="1uF"/>
 <part name="C2" library="resistor" deviceset="C-EU" device="C2012" value="100nF"/>
-<part name="Q1" library="transistor-small-signal" deviceset="BSS123" device=""/>
+<part name="Q1" library="transistor-small-signal" deviceset="BSS84" device=""/>
 <part name="R6" library="resistor" deviceset="R-EU_" device="R1206W" value="4K7"/>
 </parts>
@@
 <instance part="C1" gate="G$1" x="10.16" y="50.8"/>
 <instance part="C2" gate="G$1" x="25.4" y="50.8"/>
-<instance part="Q1" gate="G$1" x="0" y="78.74"/>
+<instance part="Q1" gate="G$1" x="0" y="78.74" rot="R180"/>
 <instance part="R6" gate="G$1" x="172.72" y="134.62"/>
 </instances>
@@
 <pinref part="PAD1" gate="G$1" pin="P"/>
 <junction x="93.98" y="66.04"/>
-<wire x1="0" y1="66.04" x2="10.16" y2="66.04" width="0.1524" layer="91"/>
 <junction x="83.82" y="66.04"/>
 <wire x1="10.16" y1="66.04" x2="25.4" y2="66.04" width="0.1524" layer="91"/>
@@
 <pinref part="C2" gate="G$1" pin="1"/>
 <wire x1="25.4" y1="53.34" x2="25.4" y2="66.04" width="0.1524" layer="91"/>
-<junction x="10.16" y="66.04"/>
 <junction x="25.4" y="66.04"/>
 <junction x="170.18" y="66.04"/>
 <pinref part="Q1" gate="G$1" pin="S"/>
-<wire x1="0" y1="66.04" x2="0" y2="73.66" width="0.1524" layer="91"/>
+<wire x1="0" y1="73.66" x2="0" y2="66.04" width="0.1524" layer="91"/>
+<wire x1="0" y1="66.04" x2="10.16" y2="66.04" width="0.1524" layer="91"/>
+<junction x="10.16" y="66.04"/>
 </segment>
 <segment>
@@
 <wire x1="182.88" y1="142.24" x2="182.88" y2="35.56" width="0.1524" layer="91"/>
 <pinref part="Q1" gate="G$1" pin="G"/>
-<wire x1="182.88" y1="35.56" x2="-5.08" y2="35.56" width="0.1524" layer="91"/>
-<wire x1="-5.08" y1="35.56" x2="-5.08" y2="76.2" width="0.1524" layer="91"/>
-</segment>
-</net>
+<wire x1="182.88" y1="35.56" x2="5.08" y2="35.56" width="0.1524" layer="91"/>
+<wire x1="5.08" y1="35.56" x2="5.08" y2="76.2" width="0.1524" layer="91"/>
+</segment>
+</net>

Commit message: a
Parts:
- removed JP2: Prog, pinhead:PINHD-1X5
- removed Q1: BSS84, transistor-small-signal:BSS84
- added C3: 100nF, resistor:C-EUC2012
- added PAD8, PAD9: WIREPADSMD5-2,5, wirepad:WIREPADSMD5-2,5
- added R9: 1K, resistor:R-EU_R1206
- added T5: BC846, transistor:BC846
- added U$3: PROGRAMMINGHEADERDIP, rfm70:PROGRAMMINGHEADERDIP
- S1: value (none) -> DTS-3; device switch-dil:SD4-01 -> switch-tact:DTS-3
Connections:
- new net N$5: R9.1, T5.B
- net GND: now also PAD9.P, T5.E, U$3.GND; no longer JP2.3, U$1.GND
- net N$10: now also U$2.RB5/AN11/RX/DT; no longer U$2.RC6/AN8/SS
- net N$11: now also R9.2, U$2.RC6/AN8/SS; no longer JP1.1, Q1.D
- net N$18: now also U$3.PGD; no longer JP2.4
- net N$19: now also U$3.PGC; no longer JP2.5
- net N$25: now also U$3.MCLR; no longer JP2.1
- net N$28: now also T5.C, U$1.GND; no longer Q1.G, U$2.RB5/AN11/RX/DT
- net N$7: now also C3.1
- net N$8: now also C3.2
- net VDD: now also JP1.1, PAD8.P, U$3.VDD; no longer JP2.2, Q1.S
Other:
- moved on the sheet: R6

Commit message: dfg
Parts:
- removed R9: 1K, resistor:R-EU_R1206
- removed T5: BC846, transistor:BC846
Connections:
- removed net N$11: R9.2, U$2.RC6/AN8/SS
- removed net N$28: T5.C, U$1.GND
- removed net N$5: R9.1, T5.B
- net GND: now also U$1.GND; no longer T5.E
Changed lines of the file:
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@@
 <part name="R6" library="resistor" deviceset="R-EU_" device="R1206W" value="4K7"/>
 <part name="U$3" library="rfm70" deviceset="PROGRAMMINGHEADER" device="" technology="DIP"/>
-<part name="T5" library="transistor" deviceset="BC846" device=""/>
-<part name="R9" library="resistor" deviceset="R-EU_" device="R1206" value="1K"/>
 <part name="C3" library="resistor" deviceset="C-EU" device="C2012" value="100nF"/>
 <part name="PAD8" library="wirepad" deviceset="WIREPAD" device="SMD5-2,5"/>
@@
 <instance part="R6" gate="G$1" x="160.02" y="109.22" rot="R270"/>
 <instance part="U$3" gate="G$1" x="185.42" y="121.92"/>
-<instance part="T5" gate="G$1" x="185.42" y="43.18"/>
-<instance part="R9" gate="G$1" x="182.88" y="55.88" rot="R90"/>
 <instance part="C3" gate="G$1" x="30.48" y="99.06" rot="R90"/>
 <instance part="PAD8" gate="G$1" x="73.66" y="38.1"/>
@@
 <wire x1="132.08" y1="66.04" x2="132.08" y2="30.48" width="0.1524" layer="91"/>
 <pinref part="IC1" gate="G$1" pin="GND"/>
-<wire x1="187.96" y1="38.1" x2="187.96" y2="30.48" width="0.1524" layer="91"/>
 <wire x1="58.42" y1="91.44" x2="58.42" y2="86.36" width="0.1524" layer="91"/>
 <wire x1="58.42" y1="86.36" x2="58.42" y2="30.48" width="0.1524" layer="91"/>
@@
 <wire x1="203.2" y1="30.48" x2="187.96" y2="30.48" width="0.1524" layer="91"/>
 <junction x="187.96" y="30.48"/>
-<pinref part="T5" gate="G$1" pin="E"/>
-<junction x="187.96" y="38.1"/>
 <pinref part="PAD9" gate="G$1" pin="P"/>
 <junction x="101.6" y="45.72"/>
+<pinref part="U$1" gate="G$1" pin="GND"/>
+<wire x1="172.72" y1="71.12" x2="172.72" y2="68.58" width="0.1524" layer="91"/>
+<wire x1="187.96" y1="71.12" x2="172.72" y2="71.12" width="0.1524" layer="91"/>
+<wire x1="187.96" y1="71.12" x2="187.96" y2="30.48" width="0.1524" layer="91"/>
 </segment>
 </net>
@@
 </segment>
 </net>
-<net name="N$5" class="0">
-<segment>
-<pinref part="R9" gate="G$1" pin="1"/>
-<pinref part="T5" gate="G$1" pin="B"/>
-<wire x1="182.88" y1="50.8" x2="182.88" y2="43.18" width="0.1524" layer="91"/>
-</segment>
-</net>
-<net name="N$11" class="0">
-<segment>
-<pinref part="R9" gate="G$1" pin="2"/>
-<wire x1="182.88" y1="60.96" x2="193.04" y2="60.96" width="0.1524" layer="91"/>
-<wire x1="193.04" y1="60.96" x2="193.04" y2="142.24" width="0.1524" layer="91"/>
-<wire x1="193.04" y1="142.24" x2="104.14" y2="142.24" width="0.1524" layer="91"/>
-<wire x1="104.14" y1="142.24" x2="104.14" y2="121.92" width="0.1524" layer="91"/>
-<pinref part="U$2" gate="G$1" pin="RC6/AN8/SS"/>
-<wire x1="104.14" y1="121.92" x2="86.36" y2="121.92" width="0.1524" layer="91"/>
-<wire x1="86.36" y1="121.92" x2="86.36" y2="119.38" width="0.1524" layer="91"/>
-</segment>
-</net>
-<net name="N$28" class="0">
-<segment>
-<pinref part="U$1" gate="G$1" pin="GND"/>
-<wire x1="172.72" y1="71.12" x2="172.72" y2="68.58" width="0.1524" layer="91"/>
-<pinref part="T5" gate="G$1" pin="C"/>
-<wire x1="187.96" y1="48.26" x2="187.96" y2="71.12" width="0.1524" layer="91"/>
-<wire x1="187.96" y1="71.12" x2="172.72" y2="71.12" width="0.1524" layer="91"/>
-</segment>
-</net>
