File: Hardware/SchemasBoard/spinac.brd (EAGLE design)
At the start: 41.5 x 26.9 mm, 29 parts, among them IC1 LNK304, IC3 MC33269ST-3.3T3, IC4 DS1820, K1 FRS1B, T1 BC846

Commit message: fghf
Changed lines of the file:
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@@
 <contactref element="U$2" pad="13"/>
 <wire x1="25.197" y1="17.192" x2="26.4325" y2="17.192" width="0.3048" layer="1"/>
-<wire x1="26.4325" y1="17.192" x2="27.813" y2="15.8115" width="0.3048" layer="1"/>
-<wire x1="27.813" y1="15.8115" x2="32.4485" y2="15.8115" width="0.3048" layer="1"/>
-<wire x1="32.4485" y1="15.8115" x2="32.766" y2="16.129" width="0.3048" layer="1"/>
+<wire x1="26.4325" y1="17.192" x2="27.813" y2="16.129" width="0.3048" layer="1"/>
+<wire x1="27.813" y1="16.129" x2="32.766" y2="16.129" width="0.3048" layer="1"/>
 <wire x1="32.766" y1="16.129" x2="32.766" y2="18.3515" width="0.3048" layer="1"/>
 <via x="32.766" y="18.3515" extent="1-16" drill="0.6"/>
@@
 <wire x1="38.9575" y1="10.8265" x2="38.354" y2="12.1285" width="0.3048" layer="16"/>
 <wire x1="38.354" y1="12.1285" x2="38.1" y2="12.8905" width="0.3048" layer="16"/>
-<wire x1="38.1" y1="12.8905" x2="30.861" y2="12.8905" width="0.3048" layer="16"/>
-<wire x1="30.861" y1="12.8905" x2="28.829" y2="14.859" width="0.3048" layer="16"/>
-<wire x1="28.829" y1="14.859" x2="28.829" y2="16.8745" width="0.3048" layer="16"/>
+<wire x1="38.1" y1="12.8905" x2="30.6705" y2="12.8905" width="0.3048" layer="16"/>
+<wire x1="30.6705" y1="12.8905" x2="28.829" y2="14.5415" width="0.3048" layer="16"/>
+<wire x1="28.829" y1="14.5415" x2="28.829" y2="16.8745" width="0.3048" layer="16"/>
 <wire x1="28.829" y1="16.8745" x2="28.84" y2="16.8855" width="0.4064" layer="16"/>
 </signal>
@@
 <wire x1="40.005" y1="12.763" x2="40.005" y2="13.4615" width="0.4064" layer="16"/>
 <wire x1="40.005" y1="13.4615" x2="37.338" y2="13.462" width="0.3048" layer="16"/>
-<wire x1="37.338" y1="13.462" x2="31.0515" y2="13.462" width="0.3048" layer="16"/>
-<wire x1="31.0515" y1="13.462" x2="29.5275" y2="14.986" width="0.3048" layer="16"/>
-<wire x1="29.5275" y1="14.986" x2="29.5275" y2="16.848" width="0.3048" layer="16"/>
-<wire x1="29.5275" y1="16.848" x2="29.49" y2="16.8855" width="0.3048" layer="16"/>
+<wire x1="37.338" y1="13.462" x2="30.988" y2="13.462" width="0.3048" layer="16"/>
+<wire x1="30.988" y1="13.462" x2="29.464" y2="14.7955" width="0.3048" layer="16"/>
+<wire x1="29.464" y1="14.7955" x2="29.464" y2="16.848" width="0.3048" layer="16"/>
+<wire x1="29.464" y1="16.848" x2="29.49" y2="16.8855" width="0.3048" layer="16"/>
 </signal>
 <signal name="N$15">
@@
 <wire x1="27.0745" y1="22.392" x2="28.067" y2="21.3995" width="0.3048" layer="1"/>
 <via x="28.067" y="21.3995" extent="1-16" drill="0.6"/>
-<wire x1="28.067" y1="21.3995" x2="28.3845" y2="20.2565" width="0.3048" layer="16"/>
-<wire x1="28.3845" y1="20.2565" x2="30.099" y2="18.0975" width="0.3048" layer="16"/>
+<wire x1="28.067" y1="21.3995" x2="28.702" y2="20.2565" width="0.3048" layer="16"/>
+<wire x1="28.702" y1="20.2565" x2="30.099" y2="18.0975" width="0.3048" layer="16"/>
 <wire x1="30.099" y1="18.0975" x2="30.099" y2="16.9265" width="0.3048" layer="16"/>
 <wire x1="30.099" y1="16.9265" x2="30.14" y2="16.8855" width="0.3048" layer="16"/>
@@
 <wire x1="26.533" y1="21.092" x2="27.178" y2="20.447" width="0.3048" layer="1"/>
 <wire x1="27.178" y1="20.447" x2="29.4005" y2="20.447" width="0.3048" layer="1"/>
-<wire x1="29.4005" y1="20.447" x2="29.4005" y2="20.6375" width="0.3048" layer="1"/>
-<wire x1="29.4005" y1="20.6375" x2="30.353" y2="20.6375" width="0.3048" layer="1"/>
-<via x="30.353" y="20.6375" extent="1-16" drill="0.6"/>
-<wire x1="30.353" y1="20.6375" x2="30.353" y2="18.796" width="0.3048" layer="16"/>
-<wire x1="30.353" y1="18.796" x2="30.7975" y2="18.3515" width="0.3048" layer="16"/>
+<wire x1="29.4005" y1="20.447" x2="29.4005" y2="20.828" width="0.3048" layer="1"/>
+<wire x1="29.4005" y1="20.828" x2="30.1625" y2="20.828" width="0.3048" layer="1"/>
+<via x="30.1625" y="20.828" extent="1-16" drill="0.6"/>
+<wire x1="30.1625" y1="20.828" x2="30.1625" y2="19.2405" width="0.3048" layer="16"/>
+<wire x1="30.1625" y1="19.2405" x2="30.7975" y2="18.3515" width="0.3048" layer="16"/>
 <wire x1="30.7975" y1="18.3515" x2="30.7975" y2="16.893" width="0.3048" layer="16"/>
 <wire x1="30.7975" y1="16.893" x2="30.79" y2="16.8855" width="0.3048" layer="16"/>
@@
 <wire x1="30.8248" y1="4.9657" x2="30.84925" y2="4.62375" width="0.3048" layer="16"/>
 <wire x1="30.84925" y1="4.62375" x2="30.861" y2="6.644" width="0.3048" layer="16"/>
-<wire x1="40.1955" y1="1.8415" x2="36.3855" y2="4.3815" width="0.3048" layer="1"/>
-<wire x1="36.3855" y1="4.3815" x2="31.623" y2="4.3815" width="0.3048" layer="1"/>
+<wire x1="40.1955" y1="1.8415" x2="37.973" y2="4.3815" width="0.3048" layer="1"/>
+<wire x1="37.973" y1="4.3815" x2="31.623" y2="4.3815" width="0.3048" layer="1"/>
 <wire x1="31.623" y1="4.3815" x2="31.369" y2="3.937" width="0.3048" layer="1"/>
 <via x="31.369" y="3.937" extent="1-16" drill="0.6"/>
@@
 <wire x1="32.8295" y1="14.478" x2="32.385" y2="15.24" width="0.3048" layer="1"/>
 <wire x1="32.385" y1="15.24" x2="31.3055" y2="15.24" width="0.3048" layer="1"/>
-<wire x1="31.3055" y1="15.24" x2="30.734" y2="14.986" width="0.3048" layer="1"/>
-<via x="30.734" y="14.986" extent="1-16" drill="0.6"/>
-<wire x1="30.734" y1="14.986" x2="31.115" y2="15.24" width="0.3048" layer="16"/>
+<wire x1="31.3055" y1="15.24" x2="30.734" y2="15.1765" width="0.3048" layer="1"/>
+<via x="30.734" y="15.1765" extent="1-16" drill="0.6"/>
+<wire x1="30.734" y1="15.1765" x2="31.115" y2="15.24" width="0.3048" layer="16"/>
 <wire x1="31.115" y1="15.24" x2="31.4325" y2="15.5575" width="0.3048" layer="16"/>
 <wire x1="31.4325" y1="15.5575" x2="31.4325" y2="16.878" width="0.3048" layer="16"/>
@@
 <contactref element="X1" pad="5"/>
 <wire x1="21.250334375" y1="1.0160375" x2="21.250334375" y2="0.930334375" width="0.6096" layer="1"/>
-<wire x1="21.250334375" y1="0.930334375" x2="20.701" y2="0.381" width="0.6096" layer="1"/>
-<wire x1="20.701" y1="0.381" x2="5.715" y2="0.381" width="0.6096" layer="1"/>
-<wire x1="5.715" y1="0.381" x2="3.683" y2="2.413" width="0.6096" layer="1"/>
-<wire x1="3.683" y1="2.413" x2="3.683" y2="4.0259" width="0.6096" layer="1"/>
+<wire x1="21.250334375" y1="0.930334375" x2="20.701" y2="0.381" width="0.4064" layer="1"/>
+<wire x1="20.701" y1="0.381" x2="5.715" y2="0.381" width="0.4064" layer="1"/>
+<wire x1="5.715" y1="0.381" x2="3.683" y2="2.413" width="0.4064" layer="1"/>
+<wire x1="3.683" y1="2.413" x2="3.683" y2="4.0259" width="0.4064" layer="1"/>
 </signal>
 <signal name="N$6">
