File: Hardware/SchemasBoard/6relayBoard.sch (EAGLE design)
At the start: 30 parts, among them IC1 LNK304, IC3 MC33269ST-3.3T3, K1 FRS1B, K2 FRS1B, T1 BC846, T2 BC846

Commit message: aa
Parts:
- added D5, D6, D7, D8: MBRA340T3, diode:MBRA340T3
- added K3, K4, K5, K6: FRS1B, relay:FRS1B
- added R10, R11, R8, R9: 1 K, resistor:R-EU_M2012
- added T3, T4, T5, T6: BC846, transistor:BC846
- added X2: (no value), con-ptr500:AK500/4
Connections:
- new net N$30: D5.A, K51.2, T3.C
- new net N$31: D6.A, K41.2, T4.C
- new net N$32: D7.A, K31.2, T5.C
- new net N$33: D8.A, K61.2, T6.C
- new net N$34: K62.S, X2-1.KL
- new net N$37: K32.S, X2-2.KL
- new net N$38: K52.S, X2-4.KL
- new net N$39: K42.S, X2-3.KL
- new net N$41: R8.2, T3.B
- new net N$42: R9.2, T4.B
- new net N$43: R10.2, T5.B
- new net N$44: R11.2, T6.B
- new net N$45: R10.1, U$2.RC5/CCP1/P1A
- new net N$46: R9.1, U$2.RC4/C2OUT/P1B
- new net N$47: R8.1, U$2.RC3/AN7C12IN3-/P1C
- net GND: now also T3.E, T4.E, T5.E, T6.E
- net N$27: now also D5.C, D6.C, D7.C, D8.C, K41.1, K51.1, K61.1
- net N$29: now also R11.1
- net N$36: now also K32.P, K32.P@1, K42.P, K42.P@1, K52.P, K52.P@1, K62.P, K62.P@1

Commit message: aaa
Connections:
- net N$27: now also K31.1
Changed lines of the file:
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@@
 <junction x="0" y="139.7"/>
 <junction x="0" y="154.94"/>
+<pinref part="K3" gate="1" pin="1"/>
+<junction x="-35.56" y="152.4"/>
 </segment>
 </net>

Commit message: aaa
Parts:
- removed R7: 1 K, resistor:R-EU_M2012
- D3: value (none) -> ES1D; device diode:DIODE-DO214AA -> diode:DIODE-DO214AC
- D4: value (none) -> 1N4007GP
Connections:
- net GND: no longer R7.1
- net N$27: no longer R7.2
Changed lines of the file:
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@@
 <grid distance="0.1" unitdist="inch" unit="inch" style="lines" multiple="1" display="no" altdistance="0.01" altunitdist="inch" altunit="inch"/>
 <layers>
-<layer number="1" name="Top" color="1" fill="1" visible="no" active="no"/>
-<layer number="16" name="Bottom" color="12" fill="1" visible="no" active="no"/>
-<layer number="17" name="Pads" color="2" fill="1" visible="no" active="no"/>
-<layer number="18" name="Vias" color="2" fill="1" visible="no" active="no"/>
-<layer number="19" name="Unrouted" color="6" fill="1" visible="no" active="no"/>
-<layer number="20" name="Dimension" color="15" fill="1" visible="no" active="no"/>
-<layer number="21" name="tPlace" color="15" fill="1" visible="no" active="no"/>
-<layer number="22" name="bPlace" color="11" fill="1" visible="no" active="no"/>
-<layer number="23" name="tOrigins" color="15" fill="1" visible="no" active="no"/>
-<layer number="24" name="bOrigins" color="15" fill="1" visible="no" active="no"/>
-<layer number="25" name="tNames" color="7" fill="1" visible="no" active="no"/>
-<layer number="26" name="bNames" color="7" fill="1" visible="no" active="no"/>
-<layer number="27" name="tValues" color="7" fill="1" visible="no" active="no"/>
-<layer number="28" name="bValues" color="7" fill="1" visible="no" active="no"/>
+<layer number="1" name="Top" color="1" fill="1" visible="yes" active="no"/>
+<layer number="16" name="Bottom" color="12" fill="1" visible="yes" active="no"/>
+<layer number="17" name="Pads" color="2" fill="1" visible="yes" active="no"/>
+<layer number="18" name="Vias" color="2" fill="1" visible="yes" active="no"/>
+<layer number="19" name="Unrouted" color="6" fill="1" visible="yes" active="no"/>
+<layer number="20" name="Dimension" color="15" fill="1" visible="yes" active="no"/>
+<layer number="21" name="tPlace" color="15" fill="1" visible="yes" active="no"/>
+<layer number="22" name="bPlace" color="11" fill="1" visible="yes" active="no"/>
+<layer number="23" name="tOrigins" color="15" fill="1" visible="yes" active="no"/>
+<layer number="24" name="bOrigins" color="15" fill="1" visible="yes" active="no"/>
+<layer number="25" name="tNames" color="7" fill="1" visible="yes" active="no"/>
+<layer number="26" name="bNames" color="7" fill="1" visible="yes" active="no"/>
+<layer number="27" name="tValues" color="7" fill="1" visible="yes" active="no"/>
+<layer number="28" name="bValues" color="7" fill="1" visible="yes" active="no"/>
 <layer number="29" name="tStop" color="7" fill="3" visible="no" active="no"/>
 <layer number="30" name="bStop" color="7" fill="6" visible="no" active="no"/>
@@
 <layer number="35" name="tGlue" color="7" fill="4" visible="no" active="no"/>
 <layer number="36" name="bGlue" color="7" fill="5" visible="no" active="no"/>
-<layer number="37" name="tTest" color="7" fill="1" visible="no" active="no"/>
-<layer number="38" name="bTest" color="7" fill="1" visible="no" active="no"/>
+<layer number="37" name="tTest" color="7" fill="1" visible="yes" active="no"/>
+<layer number="38" name="bTest" color="7" fill="1" visible="yes" active="no"/>
 <layer number="39" name="tKeepout" color="4" fill="11" visible="no" active="no"/>
 <layer number="40" name="bKeepout" color="1" fill="11" visible="no" active="no"/>
@@
 <layer number="44" name="Drills" color="7" fill="1" visible="no" active="no"/>
 <layer number="45" name="Holes" color="7" fill="1" visible="no" active="no"/>
-<layer number="46" name="Milling" color="3" fill="1" visible="no" active="no"/>
-<layer number="47" name="Measures" color="7" fill="1" visible="no" active="no"/>
-<layer number="48" name="Document" color="7" fill="1" visible="no" active="no"/>
-<layer number="49" name="Reference" color="7" fill="1" visible="no" active="no"/>
-<layer number="50" name="dxf" color="7" fill="1" visible="no" active="no"/>
-<layer number="51" name="tDocu" color="7" fill="1" visible="no" active="no"/>
-<layer number="52" name="bDocu" color="7" fill="1" visible="no" active="no"/>
+<layer number="46" name="Milling" color="3" fill="1" visible="yes" active="no"/>
+<layer number="47" name="Measures" color="7" fill="1" visible="yes" active="no"/>
+<layer number="48" name="Document" color="7" fill="1" visible="yes" active="no"/>
+<layer number="49" name="Reference" color="7" fill="1" visible="yes" active="no"/>
+<layer number="50" name="dxf" color="7" fill="1" visible="yes" active="no"/>
+<layer number="51" name="tDocu" color="7" fill="1" visible="yes" active="no"/>
+<layer number="52" name="bDocu" color="7" fill="1" visible="yes" active="no"/>
 <layer number="91" name="Nets" color="2" fill="1" visible="yes" active="yes"/>
 <layer number="92" name="Busses" color="1" fill="1" visible="yes" active="yes"/>
@@
 <part name="C5" library="resistor" deviceset="C-EU" device="C2012" value="100nF"/>
 <part name="T1" library="transistor" deviceset="BC846" device=""/>
-<part name="D3" library="diode" deviceset="DIODE-" device="DO214AA"/>
-<part name="D4" library="diode" deviceset="DIODE-" device="DO214AA"/>
+<part name="D3" library="diode" deviceset="DIODE-" device="DO214AC" value="ES1D"/>
+<part name="D4" library="diode" deviceset="DIODE-" device="DO214AA" value="1N4007GP"/>
 <part name="D1" library="diode" deviceset="MBRA340T3" device=""/>
 <part name="C6" library="resistor" deviceset="CPOL-EU" device="SMCA" value="1uF"/>
@@
 <part name="U$3" library="rfm70" deviceset="PROGRAMMINGHEADER" device="" technology="DIP"/>
 <part name="IC3" library="linear" deviceset="MC33269ST*" device="" technology="-3.3T3"/>
-<part name="R7" library="resistor" deviceset="R-EU_" device="M2012" value="1 K"/>
 <part name="L2" library="inductor-neosid" deviceset="BS" device="11" value="680uH"/>
 <part name="K3" library="relay" deviceset="FRS1B" device="">
@@
 <instance part="U$3" gate="G$1" x="177.8" y="134.62"/>
 <instance part="IC3" gate="G$1" x="104.14" y="50.8"/>
-<instance part="R7" gate="G$1" x="81.28" y="45.72" rot="R90"/>
 <instance part="L2" gate="G$1" x="76.2" y="50.8" rot="R90"/>
 <instance part="K3" gate="1" x="-35.56" y="147.32" smashed="yes">
@@
 <wire x1="20.32" y1="30.48" x2="22.86" y2="30.48" width="0.1524" layer="91"/>
 <wire x1="22.86" y1="30.48" x2="71.12" y2="30.48" width="0.1524" layer="91"/>
-<wire x1="71.12" y1="30.48" x2="81.28" y2="30.48" width="0.1524" layer="91"/>
-<wire x1="81.28" y1="30.48" x2="88.9" y2="30.48" width="0.1524" layer="91"/>
+<wire x1="71.12" y1="30.48" x2="88.9" y2="30.48" width="0.1524" layer="91"/>
 <wire x1="88.9" y1="30.48" x2="104.14" y2="30.48" width="0.1524" layer="91"/>
 <wire x1="104.14" y1="30.48" x2="127" y2="30.48" width="0.1524" layer="91"/>
@@
 <wire x1="104.14" y1="45.72" x2="104.14" y2="30.48" width="0.1524" layer="91"/>
 <junction x="104.14" y="30.48"/>
-<pinref part="R7" gate="G$1" pin="1"/>
-<wire x1="81.28" y1="40.64" x2="81.28" y2="30.48" width="0.1524" layer="91"/>
-<junction x="81.28" y="30.48"/>
 <pinref part="T3" gate="G$1" pin="E"/>
 <wire x1="-55.88" y1="101.6" x2="-71.12" y2="101.6" width="0.1524" layer="91"/>
@@
 <wire x1="0" y1="81.28" x2="0" y2="83.82" width="0.1524" layer="91"/>
 <wire x1="96.52" y1="55.88" x2="88.9" y2="55.88" width="0.1524" layer="91"/>
-<wire x1="76.2" y1="60.96" x2="81.28" y2="60.96" width="0.1524" layer="91"/>
-<wire x1="81.28" y1="60.96" x2="88.9" y2="60.96" width="0.1524" layer="91"/>
+<wire x1="76.2" y1="60.96" x2="88.9" y2="60.96" width="0.1524" layer="91"/>
 <wire x1="88.9" y1="60.96" x2="88.9" y2="55.88" width="0.1524" layer="91"/>
 <pinref part="C4" gate="G$1" pin="+"/>
@@
 <junction x="0" y="99.06"/>
 <pinref part="IC3" gate="G$1" pin="IN"/>
-<pinref part="R7" gate="G$1" pin="2"/>
-<wire x1="81.28" y1="50.8" x2="81.28" y2="60.96" width="0.1524" layer="91"/>
-<junction x="81.28" y="60.96"/>
 <pinref part="L2" gate="G$1" pin="2"/>
 <wire x1="76.2" y1="55.88" x2="76.2" y2="60.96" width="0.1524" layer="91"/>

Commit message: aaa
Parts:
- added R7: 1 K, resistor:R-EU_M2012
- C3: device resistor:CPOL-EUE2.5-5 -> resistor:CPOL-EUSMCC
- R2: device resistor:R-EU_R2512W -> resistor:R-EU_0411/12
Connections:
- net GND: now also R7.1
- net N$27: now also R7.2
- net N$36: now also X1-1.KL; no longer X1-4.KL
- net N$4: now also X1-2.KL; no longer X1-3.KL
- net N$7: now also X1-3.KL; no longer X1-1.KL
- net N$8: now also X1-4.KL; no longer X1-2.KL
Other:
- moved on the sheet: X1-1, X1-2, X1-3, X1-4
Changed lines of the file:
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@@
 <part name="B1" library="rectifier" deviceset="RECTIFIER-" device="S40" value="RECTIFIER"/>
 <part name="R1" library="resistor" deviceset="R-EU_" device="R2512W" value="100"/>
-<part name="R2" library="resistor" deviceset="R-EU_" device="R2512W" value="8,2"/>
+<part name="R2" library="resistor" deviceset="R-EU_" device="0411/12" value="8,2"/>
 <part name="U$1" library="rfm70" deviceset="RFM70" device=""/>
 <part name="U$2" library="microchip" deviceset="PIC16F690*" device=""/>
@@
 <part name="R4" library="resistor" deviceset="R-EU_" device="M2012" value="2,05 k"/>
 <part name="R5" library="resistor" deviceset="R-EU_" device="M2012" value="1 K"/>
-<part name="C3" library="resistor" deviceset="CPOL-EU" device="E2.5-5" value="10uF / 16 V"/>
+<part name="C3" library="resistor" deviceset="CPOL-EU" device="SMCC" value="10uF / 16 V"/>
 <part name="C4" library="resistor" deviceset="CPOL-EU" device="E2.5-5" value="100uF / 6,3 V"/>
 <part name="C5" library="resistor" deviceset="C-EU" device="C2012" value="100nF"/>
@@
 <attribute name="OC_NEWARK" value="unknown"/>
 </part>
+<part name="R7" library="resistor" deviceset="R-EU_" device="M2012" value="1 K"/>
 </parts>
 <sheets>
@@
 <instance part="D2" gate="G$1" x="10.16" y="93.98" rot="R90"/>
 <instance part="R6" gate="G$1" x="38.1" y="127"/>
-<instance part="X1" gate="-1" x="-38.1" y="63.5"/>
-<instance part="X1" gate="-2" x="-38.1" y="58.42"/>
-<instance part="X1" gate="-3" x="-38.1" y="53.34"/>
-<instance part="X1" gate="-4" x="-38.1" y="48.26"/>
+<instance part="X1" gate="-1" x="-43.18" y="63.5"/>
+<instance part="X1" gate="-2" x="-43.18" y="58.42"/>
+<instance part="X1" gate="-3" x="-43.18" y="53.34"/>
+<instance part="X1" gate="-4" x="-43.18" y="48.26"/>
 <instance part="U$3" gate="G$1" x="177.8" y="134.62"/>
 <instance part="IC3" gate="G$1" x="104.14" y="50.8"/>
@@
 <instance part="X2" gate="-3" x="22.86" y="154.94"/>
 <instance part="X2" gate="-4" x="22.86" y="149.86"/>
+<instance part="R7" gate="G$1" x="96.52" y="35.56" rot="R90"/>
 </instances>
 <busses>
@@
 <pinref part="B1" gate="G$1" pin="AC2"/>
 <wire x1="12.7" y1="43.18" x2="12.7" y2="38.1" width="0.1524" layer="91"/>
-<wire x1="12.7" y1="38.1" x2="-5.08" y2="38.1" width="0.1524" layer="91"/>
-<wire x1="-5.08" y1="38.1" x2="-5.08" y2="53.34" width="0.1524" layer="91"/>
-<pinref part="X1" gate="-3" pin="KL"/>
-<wire x1="-33.02" y1="53.34" x2="-5.08" y2="53.34" width="0.1524" layer="91"/>
+<wire x1="12.7" y1="38.1" x2="-12.7" y2="38.1" width="0.1524" layer="91"/>
+<pinref part="X1" gate="-2" pin="KL"/>
+<wire x1="-38.1" y1="58.42" x2="-12.7" y2="58.42" width="0.1524" layer="91"/>
+<wire x1="-12.7" y1="58.42" x2="-12.7" y2="38.1" width="0.1524" layer="91"/>
 </segment>
 </net>
@@
 <wire x1="22.86" y1="30.48" x2="71.12" y2="30.48" width="0.1524" layer="91"/>
 <wire x1="71.12" y1="30.48" x2="88.9" y2="30.48" width="0.1524" layer="91"/>
-<wire x1="88.9" y1="30.48" x2="104.14" y2="30.48" width="0.1524" layer="91"/>
+<wire x1="88.9" y1="30.48" x2="96.52" y2="30.48" width="0.1524" layer="91"/>
+<wire x1="96.52" y1="30.48" x2="104.14" y2="30.48" width="0.1524" layer="91"/>
 <wire x1="104.14" y1="30.48" x2="127" y2="30.48" width="0.1524" layer="91"/>
 <wire x1="127" y1="30.48" x2="132.08" y2="30.48" width="0.1524" layer="91"/>
@@
 <junction x="-71.12" y="147.32"/>
 <junction x="5.08" y="30.48"/>
+<pinref part="R7" gate="G$1" pin="1"/>
+<junction x="96.52" y="30.48"/>
 </segment>
 </net>
@@
 <pinref part="R2" gate="G$1" pin="1"/>
 <wire x1="-7.62" y1="55.88" x2="-5.08" y2="55.88" width="0.1524" layer="91"/>
-<wire x1="-7.62" y1="48.26" x2="-7.62" y2="55.88" width="0.1524" layer="91"/>
 <pinref part="K2" gate="2" pin="P@1"/>
 <wire x1="-17.78" y1="83.82" x2="-22.86" y2="83.82" width="0.1524" layer="91"/>
@@
 <wire x1="-25.4" y1="63.5" x2="-7.62" y2="63.5" width="0.1524" layer="91"/>
 <wire x1="-7.62" y1="63.5" x2="-7.62" y2="55.88" width="0.1524" layer="91"/>
-<junction x="-7.62" y="55.88"/>
-<pinref part="X1" gate="-4" pin="KL"/>
-<wire x1="-33.02" y1="48.26" x2="-7.62" y2="48.26" width="0.1524" layer="91"/>
 <pinref part="K6" gate="2" pin="P"/>
 <wire x1="-20.32" y1="160.02" x2="-10.16" y2="160.02" width="0.1524" layer="91"/>
@@
 <junction x="-17.78" y="144.78"/>
 <junction x="-20.32" y="160.02"/>
+<pinref part="X1" gate="-1" pin="KL"/>
+<wire x1="-38.1" y1="63.5" x2="-25.4" y2="63.5" width="0.1524" layer="91"/>
+<junction x="-25.4" y="63.5"/>
 </segment>
 </net>
@@
 <segment>
 <pinref part="K1" gate="2" pin="S"/>
-<pinref part="X1" gate="-1" pin="KL"/>
-<wire x1="-33.02" y1="63.5" x2="-30.48" y2="63.5" width="0.1524" layer="91"/>
-<wire x1="-30.48" y1="63.5" x2="-30.48" y2="78.74" width="0.1524" layer="91"/>
 <wire x1="-30.48" y1="78.74" x2="-20.32" y2="78.74" width="0.1524" layer="91"/>
+<pinref part="X1" gate="-3" pin="KL"/>
+<wire x1="-38.1" y1="53.34" x2="-30.48" y2="53.34" width="0.1524" layer="91"/>
+<wire x1="-30.48" y1="53.34" x2="-30.48" y2="78.74" width="0.1524" layer="91"/>
 </segment>
 </net>
@@
 <pinref part="K3" gate="1" pin="1"/>
 <junction x="-35.56" y="152.4"/>
+<pinref part="R7" gate="G$1" pin="2"/>
+<wire x1="96.52" y1="40.64" x2="96.52" y2="55.88" width="0.1524" layer="91"/>
+<junction x="96.52" y="55.88"/>
 </segment>
 </net>
@@
 <pinref part="K2" gate="2" pin="S"/>
 <wire x1="-20.32" y1="91.44" x2="-27.94" y2="91.44" width="0.1524" layer="91"/>
-<wire x1="-27.94" y1="91.44" x2="-27.94" y2="58.42" width="0.1524" layer="91"/>
-<pinref part="X1" gate="-2" pin="KL"/>
-<wire x1="-33.02" y1="58.42" x2="-27.94" y2="58.42" width="0.1524" layer="91"/>
-</segment>
-</net>
+<wire x1="-27.94" y1="91.44" x2="-27.94" y2="48.26" width="0.1524" layer="91"/>
+<pinref part="X1" gate="-4" pin="KL"/>
+<wire x1="-27.94" y1="48.26" x2="-38.1" y2="48.26" width="0.1524" layer="91"/>
+</segment>
+</net>
