File: Hardware/SchemasBoard/heatingHeaderEQ3.brd (EAGLE design)
At the start: 45.5 x 30.5 mm, 36 parts, among them IC1 DS1820, T5 BC846

Commit message: a
Parts:
- removed PAD8, PAD9: WIREPADSMD5-2,5, wirepad:5-2,5
- moved U$1 48.4 mm to (11.4, 43.2), turned to 0 degrees
- moved PAD3 36.0 mm to (19.1, 33.0), flipped to the top
- moved PAD4 32.5 mm to (22.9, 33.0), flipped to the top
- moved U$3 32.2 mm to (11.4, 6.35), flipped to the bottom, turned to 0 degrees
- moved PAD7 32.1 mm to (41.9, 29.2), flipped to the top
- moved R9 31.2 mm to (5.08, 34.3), flipped to the top
- moved PAD6 29.5 mm to (41.9, 22.9), flipped to the top
- moved R5 28.4 mm to (3.56, 26.5), flipped to the top
- moved PAD1 26.5 mm to (29.2, 33.0)
- moved T5 25.6 mm to (6.05, 30.9), flipped to the top, turned to 180 degrees
- moved C3 24.8 mm to (19.4, 25.3), flipped to the top
- moved T1 21.8 mm to (38.1, 31.8), flipped to the top, turned to 0 degrees
- moved PAD5 20.4 mm to (41.9, 16.5), flipped to the top
- moved R8 19.8 mm to (22.9, 3.81), flipped to the top
- moved R7 19.5 mm to (14.0, 26.5), flipped to the top
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Connections:
- net GND: no longer PAD9.1
- net VDD: no longer PAD8.1
Routing:
- net N$22: track 21.7 -> 115.9 mm, vias 0 -> 3
- net N$2: track 93.5 -> 8.53 mm, vias 3 -> 0
- net N$20: track 25.0 -> 100.2 mm, vias 0 -> 3
- net N$31: track 6.60 -> 69.8 mm, vias 0 -> 6
- net N$4: track 5.45 -> 50.6 mm, vias 0 -> 2
- net N$18: track 54.7 -> 12.0 mm
- net N$19: track 53.1 -> 12.1 mm
- net GND: track 172.3 -> 138.8 mm, vias 8 -> 0
- net N$25: track 81.0 -> 47.5 mm
- net N$27: track 34.7 -> 4.11 mm
- net N$30: track 16.1 -> 41.2 mm, vias 0 -> 4
- net N$7: track 44.6 -> 66.4 mm, vias 2 -> 4
- net N$12: track 36.5 -> 16.2 mm
- net N$15: track 46.2 -> 65.4 mm, vias 2 -> 4
- net N$6: track 19.6 -> 38.2 mm, vias 0 -> 1
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Other:
- board size 45.5 x 30.5 mm -> 44.1 x 36.8 mm

Commit message: dfg
Parts:
- removed R9: 1K, resistor:R1206
- removed T5: BC846, transistor:SOT23
- moved C2 1.04 mm to (15.0, 16.5)
Connections:
- removed net N$11: R9.2, U$2.8
- removed net N$28: T5.3, U$1.GND
- removed net N$5: R9.1, T5.1
- net GND: now also U$1.GND; no longer T5.2
Routing:
- net N$11: track 24.6 -> 0.00 mm, vias 2 -> 0
- net N$28: track 8.10 -> 0.00 mm, vias 1 -> 0
- net GND: track 138.8 -> 133.1 mm, vias 0 -> 1
- net N$22: track 115.9 -> 120.5 mm
- net N$8: track 51.7 -> 48.6 mm
- net N$5: track 2.58 -> 0.00 mm
- net N$6: track 38.2 -> 40.7 mm
- net N$21: track 25.5 -> 27.5 mm
- net N$31: track 69.8 -> 71.6 mm
- net VDD: track 106.2 -> 104.5 mm
- net N$12: track 16.2 -> 17.8 mm
- net N$23: track 12.1 -> 13.5 mm
- net N$20: track 100.2 -> 101.4 mm
- net N$16: track 48.7 -> 49.4 mm

Commit message: aaa
Parts:
- moved U$3 9.12 mm to (20.3, 4.25)
- moved R8 7.00 mm to (29.8, 2.61)
- moved R6 4.10 mm to (17.8, 1.05), turned to 0 degrees
- moved S1 2.85 mm to (24.3, 7.99)
- moved JP1 2.12 mm to (32.6, 6.05)
- moved IC1 0.90 mm to (36.8, 1.64)
Routing:
- net VDD: track 104.5 -> 81.1 mm
- net GND: track 133.1 -> 121.7 mm
- net N$25: track 47.5 -> 43.1 mm
- net N$10: track 21.2 -> 25.3 mm
- net N$2: track 8.53 -> 4.63 mm
- net N$18: track 12.0 -> 8.62 mm
- net N$3: track 47.3 -> 44.6 mm
- net N$19: track 12.1 -> 9.50 mm
- net N$15: track 65.8 -> 68.2 mm
- net N$1: track 50.9 -> 52.3 mm

Commit message: safd
Parts:
- moved U$1 41.5 mm to (6.13, 1.98), turned to 180 degrees
- moved R8 11.5 mm to (24.2, 12.6)
- moved U$3 9.47 mm to (29.6, 2.45)
- moved R6 3.95 mm to (21.7, 1.65)
- moved D4 2.40 mm to (30.3, 14.0)
- moved S1 2.04 mm to (24.7, 5.99)
- moved C2 1.50 mm to (16.2, 17.4)
- moved C1 0.85 mm to (18.6, 16.8)
- moved IC1 0.71 mm to (37.5, 1.74)
- moved JP1 0.10 mm to (32.6, 5.95)
Routing:
- net N$23: track 13.5 -> 115.3 mm
- net N$22: track 120.5 -> 20.9 mm, vias 3 -> 1
- net N$20: track 101.4 -> 7.97 mm, vias 3 -> 1
- net N$16: track 49.4 -> 4.60 mm, vias 5 -> 1
- net VDD: track 81.1 -> 124.3 mm, vias 2 -> 5
- net GND: track 121.7 -> 153.2 mm, vias 1 -> 0
- net N$6: track 40.7 -> 15.1 mm
- net N$25: track 43.1 -> 67.3 mm
- net N$18: track 8.62 -> 32.1 mm
- net N$19: track 9.50 -> 31.9 mm
- net N$2: track 4.63 -> 20.2 mm, vias 0 -> 1
- net N$3: track 44.6 -> 52.1 mm
- net N$15: track 68.2 -> 75.4 mm
- net N$10: track 25.3 -> 32.0 mm
- net N$1: track 52.3 -> 58.6 mm
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