File: Hardware/SchemasBoard/raspi.brd (EAGLE design)
At the start: 14.9 x 30.5 mm, 7 parts

Commit message: a
Parts:
- moved JP1 0.57 mm to (7.09, 3.00), turned to 180 degrees
Routing:
- net N$33: track 3.01 -> 17.6 mm
- net N$34: track 16.5 -> 25.6 mm
- net VDD: track 42.5 -> 43.5 mm
Changed lines of the file:
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@@
 <element name="U$2" library="microchip" package="SSOP20" value="PIC16F690" x="9.922" y="10.6666"/>
 <element name="JP2" library="pinhead" package="1X05" value="Prog" x="2.0019" y="12.7889" rot="R90"/>
-<element name="JP1" library="pinhead" package="2X05" value="Raspi" x="7.62" y="2.81"/>
+<element name="JP1" library="pinhead" package="2X05" value="Raspi" x="7.0866" y="3.0005" rot="R180"/>
 <element name="S1" library="switch-dil" package="SD4-01" value="" x="2.2098" y="24.6253">
 <attribute name="OC_NEWARK" value="unknown" x="2.2098" y="24.6253" size="1.778" layer="27" display="off"/>
@@
 <wire x1="4.8133" y1="9.525" x2="4.8006" y2="8.1661" width="0.6096" layer="16"/>
 <wire x1="4.8006" y1="8.1661" x2="5.9309" y2="7.0485" width="0.6096" layer="16"/>
-<wire x1="6.07695" y1="6.69925" x2="5.0927" y2="6.223" width="0.6096" layer="16"/>
-<wire x1="5.0927" y1="6.223" x2="1.7145" y2="6.223" width="0.6096" layer="16"/>
-<wire x1="1.7145" y1="6.223" x2="0.8128" y2="5.334" width="0.6096" layer="16"/>
-<wire x1="0.8128" y1="5.334" x2="0.8128" y2="3.2672" width="0.6096" layer="16"/>
-<wire x1="0.8128" y1="3.2672" x2="2.54" y2="1.54" width="0.6096" layer="16"/>
-<wire x1="7.0035" y1="7.0543" x2="6.07695" y2="6.69925" width="0.3048" layer="1"/>
-<via x="6.07695" y="6.69925" extent="1-16" drill="0.6"/>
 <wire x1="4.71805" y1="8.08355" x2="4.8006" y2="8.1661" width="0.3048" layer="16"/>
 <wire x1="4.3118" y1="26.74" x2="4.3053" y2="26.7335" width="0.6096" layer="1"/>
@@
 <wire x1="6.02" y1="26.74" x2="4.3053" y2="26.74" width="0.6096" layer="1"/>
 <wire x1="4.3053" y1="26.74" x2="4.3053" y2="26.7335" width="0.6096" layer="1"/>
-<wire x1="4.8895" y1="7.8511" x2="4.92125" y2="6.65095" width="0.3048" layer="1"/>
-<wire x1="4.92125" y1="6.65095" x2="6.07695" y2="6.69925" width="0.3048" layer="1"/>
 <contactref element="C2" pad="+"/>
 <wire x1="4.9403" y1="11.9239" x2="4.7738" y2="11.9239" width="0.4064" layer="1"/>
 <wire x1="4.7738" y1="11.9239" x2="3.0988" y2="10.2489" width="0.4064" layer="1"/>
 <wire x1="3.0988" y1="10.2489" x2="2.0019" y2="10.2489" width="0.4064" layer="1"/>
-<wire x1="7.0035" y1="7.0543" x2="6.997" y2="7.0416" width="0" layer="19" extent="1-1"/>
-<wire x1="4.71805" y1="8.08355" x2="4.8895" y2="7.8511" width="0" layer="19" extent="1-16"/>
+<wire x1="12.1666" y1="4.2705" x2="12.1285" y2="4.2705" width="0.4064" layer="16"/>
+<wire x1="12.1285" y1="4.2705" x2="12.1285" y2="7.0358" width="0.6096" layer="16"/>
+<wire x1="12.1285" y1="7.0358" x2="5.9309" y2="7.0358" width="0.6096" layer="16"/>
+<wire x1="5.9309" y1="7.0358" x2="5.9309" y2="7.0485" width="0.4064" layer="16"/>
+<wire x1="6.997" y1="7.0416" x2="4.8895" y2="7.0416" width="0.4064" layer="1"/>
+<wire x1="4.8895" y1="7.0416" x2="4.8895" y2="7.8511" width="0.4064" layer="1"/>
+<wire x1="4.8895" y1="7.8511" x2="4.8387" y2="7.8511" width="0.3048" layer="1"/>
+<wire x1="4.8387" y1="7.8511" x2="4.8387" y2="6.5405" width="0.3048" layer="1"/>
+<via x="4.8387" y="6.5405" extent="1-16" drill="0.6"/>
+<wire x1="4.8387" y1="6.5405" x2="5.4356" y2="6.5405" width="0.3048" layer="16"/>
+<wire x1="5.4356" y1="6.5405" x2="5.9309" y2="7.0358" width="0.3048" layer="16"/>
 </signal>
 <signal name="N$18">
@@
 <contactref element="U$2" pad="4"/>
 <contactref element="JP2" pad="1"/>
-<wire x1="2.0019" y1="7.7089" x2="2.0447" y2="5.6896" width="0.3048" layer="1"/>
-<wire x1="2.0447" y1="5.6896" x2="5.9436" y2="5.6388" width="0.3048" layer="1"/>
+<wire x1="2.0019" y1="7.7089" x2="1.9939" y2="5.6515" width="0.3048" layer="1"/>
+<wire x1="1.9939" y1="5.6515" x2="5.9436" y2="5.6388" width="0.3048" layer="1"/>
 <wire x1="5.9436" y1="5.6388" x2="8.4836" y2="5.6388" width="0.3048" layer="1"/>
 <wire x1="8.4836" y1="5.6388" x2="8.9535" y2="6.0572" width="0.3048" layer="1"/>
@@
 <contactref element="U$2" pad="10"/>
 <contactref element="JP1" pad="10"/>
-<wire x1="12.7" y1="4.08" x2="12.7" y2="5.3467" width="0.3048" layer="1"/>
-<wire x1="12.7" y1="5.3467" x2="12.8397" y2="5.5499" width="0.3048" layer="1"/>
-<wire x1="12.8397" y1="5.5499" x2="12.8397" y2="6.1345" width="0.3048" layer="1"/>
+<wire x1="2.0066" y1="1.7305" x2="1.9939" y2="3.0226" width="0.3048" layer="1"/>
+<wire x1="1.9939" y1="3.0226" x2="13.589" y2="3.0226" width="0.3048" layer="1"/>
+<wire x1="13.589" y1="3.0226" x2="13.5763" y2="5.6134" width="0.3048" layer="1"/>
+<wire x1="13.5763" y1="5.6134" x2="13.5763" y2="6.1345" width="0.3048" layer="1"/>
+<wire x1="13.5763" y1="6.1345" x2="12.8397" y2="6.1345" width="0.3048" layer="1"/>
 <wire x1="12.8397" y1="6.1345" x2="12.847" y2="7.0416" width="0.3048" layer="1"/>
 </signal>
@@
 <wire x1="12.197" y1="14.2916" x2="12.1843" y2="12.3648" width="0.3048" layer="1"/>
 <wire x1="12.1843" y1="12.3648" x2="14.1986" y2="10.3759" width="0.3048" layer="1"/>
-<wire x1="14.1986" y1="10.3759" x2="14.1986" y2="3.556" width="0.3048" layer="1"/>
-<wire x1="14.1986" y1="3.556" x2="13.4366" y2="2.794" width="0.3048" layer="1"/>
-<wire x1="13.4366" y1="2.794" x2="11.446" y2="2.794" width="0.3048" layer="1"/>
-<wire x1="11.446" y1="2.794" x2="10.16" y2="4.08" width="0.3048" layer="1"/>
+<wire x1="14.1986" y1="10.3759" x2="14.1986" y2="0.4699" width="0.3048" layer="1"/>
+<wire x1="14.1986" y1="0.4699" x2="4.5499" y2="0.4699" width="0.3048" layer="1"/>
+<wire x1="4.5499" y1="0.4699" x2="4.5466" y2="1.7305" width="0.3048" layer="1"/>
 </signal>
 </signals>

Commit message: a
Parts:
- moved U$1 2.78 mm to (23.1, 27.9)
Routing:
- net N$28: track 31.5 -> 35.3 mm
- net VDD: track 43.5 -> 46.3 mm
- net GND: track 12.2 -> 15.0 mm
- net N$21: track 7.86 -> 6.91 mm
- net N$23: track 18.0 -> 17.4 mm
- net N$20: track 12.9 -> 13.4 mm, vias 2 -> 0
Changed lines of the file:
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@@
 </autorouter>
 <elements>
-<element name="U$1" library="rfm70" package="RFM70" value="RFM70" x="20.32" y="27.94" locked="yes" rot="R270"/>
+<element name="U$1" library="rfm70" package="RFM70" value="RFM70" x="23.1013" y="27.94" rot="R270"/>
 <element name="U$2" library="microchip" package="SSOP20" value="PIC16F690" x="9.922" y="10.6666"/>
 <element name="JP2" library="pinhead" package="1X05" value="Prog" x="2.0019" y="12.7889" rot="R90"/>
@@
 <vertex x="14.7701" y="30.3149"/>
 </polygon>
-<wire x1="6.02" y1="28.04" x2="6.0089" y2="28.0289" width="0.6096" layer="1"/>
+<wire x1="8.8013" y1="28.04" x2="6.0089" y2="28.0289" width="0.6096" layer="1"/>
 <wire x1="6.0089" y1="28.0289" x2="4.7752" y2="28.0289" width="0.6096" layer="1"/>
 <wire x1="4.7752" y1="28.0289" x2="4.5339" y2="28.2702" width="0.6096" layer="1"/>
@@
 <contactref element="U$1" pad="MISO"/>
 <contactref element="U$2" pad="13"/>
-<wire x1="11.547" y1="14.2916" x2="11.547" y2="16.3041" width="0.3048" layer="1"/>
-<wire x1="11.547" y1="16.3041" x2="7.6454" y2="20.2311" width="0.3048" layer="1"/>
-<wire x1="7.6454" y1="20.2311" x2="6.0289" y2="20.2311" width="0.3048" layer="1"/>
-<wire x1="6.0289" y1="20.2311" x2="6.02" y2="20.24" width="0.3048" layer="1"/>
+<wire x1="8.8013" y1="20.24" x2="8.8013" y2="20.2565" width="0.3048" layer="1"/>
+<wire x1="8.8013" y1="20.2565" x2="11.5316" y2="20.2565" width="0.3048" layer="1"/>
+<wire x1="11.5316" y1="20.2565" x2="11.5316" y2="14.2916" width="0.3048" layer="1"/>
+<wire x1="11.5316" y1="14.2916" x2="11.547" y2="14.2916" width="0.3048" layer="1"/>
 </signal>
 <signal name="VDD">
@@
 <contactref element="C1" pad="1"/>
 <wire x1="4.0894" y1="10.2489" x2="2.0019" y2="10.2489" width="0.6096" layer="16"/>
-<wire x1="6.02" y1="26.74" x2="4.3053" y2="26.74" width="0.6096" layer="1"/>
+<wire x1="8.8013" y1="26.74" x2="4.3053" y2="26.74" width="0.6096" layer="1"/>
 <wire x1="4.3053" y1="26.74" x2="4.3053" y2="26.7335" width="0.6096" layer="1"/>
 <contactref element="C2" pad="+"/>
@@
 <wire x1="8.297" y1="14.2916" x2="8.297" y2="15.3504" width="0.3048" layer="1"/>
 <wire x1="8.297" y1="15.3504" x2="6.858" y2="16.8021" width="0.3048" layer="1"/>
-<wire x1="6.858" y1="16.8021" x2="5.2451" y2="16.8021" width="0.3048" layer="1"/>
-<wire x1="5.2451" y1="16.8021" x2="4.1656" y2="17.8689" width="0.3048" layer="1"/>
+<wire x1="6.858" y1="16.8021" x2="5.7277" y2="17.8943" width="0.3048" layer="1"/>
+<wire x1="5.7277" y1="17.8943" x2="4.1656" y2="17.8689" width="0.3048" layer="1"/>
 <wire x1="4.1656" y1="17.8689" x2="2.0019" y2="17.8689" width="0.3048" layer="1"/>
 </signal>
@@
 <wire x1="8.947" y1="14.2916" x2="8.947" y2="15.5894" width="0.3048" layer="1"/>
 <wire x1="8.947" y1="15.5894" x2="7.112" y2="17.4498" width="0.3048" layer="1"/>
-<wire x1="7.112" y1="17.4498" x2="5.5245" y2="17.4498" width="0.3048" layer="1"/>
-<wire x1="5.5245" y1="17.4498" x2="4.7625" y2="18.2118" width="0.3048" layer="1"/>
-<wire x1="4.7625" y1="18.2118" x2="4.7625" y2="25.1587" width="0.3048" layer="1"/>
-<wire x1="4.7625" y1="25.1587" x2="5.0419" y2="25.4381" width="0.3048" layer="1"/>
-<wire x1="5.0419" y1="25.4381" x2="6.0181" y2="25.4381" width="0.3048" layer="1"/>
-<wire x1="6.0181" y1="25.4381" x2="6.02" y2="25.44" width="0.3048" layer="1"/>
+<wire x1="8.8013" y1="25.44" x2="5.8693" y2="25.44" width="0.3048" layer="1"/>
+<wire x1="5.8693" y1="25.44" x2="5.8293" y2="25.4" width="0.3048" layer="1"/>
+<wire x1="5.8293" y1="25.4" x2="5.8293" y2="18.7325" width="0.3048" layer="1"/>
+<wire x1="5.8293" y1="18.7325" x2="7.112" y2="17.4498" width="0.3048" layer="1"/>
 </signal>
 <signal name="N$20">
 <contactref element="U$2" pad="16"/>
 <contactref element="U$1" pad="CSN"/>
-<wire x1="9.597" y1="14.2916" x2="9.5885" y2="14.5625" width="0.3048" layer="1"/>
-<wire x1="9.5885" y1="15.4559" x2="9.8552" y2="15.7988" width="0.3048" layer="1"/>
-<via x="9.8552" y="15.7988" extent="1-16" drill="0.6"/>
-<wire x1="9.8552" y1="15.7988" x2="9.7282" y2="15.7988" width="0.3048" layer="16"/>
-<wire x1="9.7282" y1="15.7988" x2="9.144" y2="16.383" width="0.3048" layer="16"/>
-<wire x1="9.144" y1="16.383" x2="9.144" y2="22.5171" width="0.3048" layer="16"/>
-<wire x1="9.144" y1="22.5171" x2="7.5311" y2="24.13" width="0.3048" layer="16"/>
-<via x="7.5311" y="24.13" extent="1-16" drill="0.6"/>
-<wire x1="7.5311" y1="24.13" x2="7.5211" y2="24.14" width="0.3048" layer="1"/>
-<wire x1="7.5211" y1="24.14" x2="6.02" y2="24.14" width="0.3048" layer="1"/>
-<wire x1="9.5885" y1="14.5625" x2="9.5885" y2="15.5321" width="0.3048" layer="1"/>
-<wire x1="9.5885" y1="15.5321" x2="9.8552" y2="15.7988" width="0.3048" layer="1"/>
+<wire x1="9.597" y1="14.2916" x2="9.597" y2="15.7903" width="0.3048" layer="1"/>
+<wire x1="9.597" y1="15.7903" x2="6.5786" y2="18.8087" width="0.3048" layer="1"/>
+<wire x1="6.5786" y1="18.8087" x2="6.5786" y2="24.0792" width="0.3048" layer="1"/>
+<wire x1="6.5786" y1="24.0792" x2="6.5405" y2="24.1173" width="0.3048" layer="1"/>
+<wire x1="6.5405" y1="24.1173" x2="8.7786" y2="24.1173" width="0.3048" layer="1"/>
+<wire x1="8.7786" y1="24.1173" x2="8.8013" y2="24.14" width="0.3048" layer="1"/>
 </signal>
 <signal name="N$21">
 <contactref element="U$2" pad="14"/>
 <contactref element="U$1" pad="IRQ"/>
-<wire x1="10.897" y1="14.2916" x2="10.9097" y2="16.0778" width="0.3048" layer="1"/>
-<wire x1="10.9097" y1="16.0778" x2="8.0391" y2="18.9357" width="0.3048" layer="1"/>
-<wire x1="8.0391" y1="18.9357" x2="6.0243" y2="18.9357" width="0.3048" layer="1"/>
-<wire x1="6.0243" y1="18.9357" x2="6.02" y2="18.94" width="0.3048" layer="1"/>
+<wire x1="8.8013" y1="18.94" x2="8.8013" y2="19.0246" width="0.3048" layer="1"/>
+<wire x1="8.8013" y1="19.0246" x2="10.8839" y2="19.0246" width="0.3048" layer="1"/>
+<wire x1="10.8839" y1="19.0246" x2="10.8839" y2="14.2916" width="0.3048" layer="1"/>
+<wire x1="10.8839" y1="14.2916" x2="10.897" y2="14.2916" width="0.3048" layer="1"/>
 </signal>
 <signal name="N$22">
 <contactref element="U$2" pad="11"/>
 <contactref element="U$1" pad="SCK"/>
-<wire x1="7.7343" y1="22.8473" x2="6.0273" y2="22.8473" width="0.3048" layer="1"/>
-<wire x1="6.0273" y1="22.8473" x2="6.02" y2="22.84" width="0.3048" layer="1"/>
-<wire x1="7.7343" y1="22.8473" x2="12.847" y2="17.76" width="0.3048" layer="1"/>
-<wire x1="12.847" y1="17.76" x2="12.847" y2="14.2916" width="0.3048" layer="1"/>
+<wire x1="12.847" y1="22.84" x2="12.847" y2="14.2916" width="0.3048" layer="1"/>
+<wire x1="8.8013" y1="22.84" x2="12.847" y2="22.84" width="0.3048" layer="1"/>
+<wire x1="12.847" y1="22.84" x2="12.847" y2="22.8473" width="0.3048" layer="1"/>
 </signal>
 <signal name="N$23">
 <contactref element="U$2" pad="9"/>
 <contactref element="U$1" pad="MOSI"/>
-<wire x1="6.02" y1="21.54" x2="6.0208" y2="21.5392" width="0.3048" layer="1"/>
-<wire x1="6.0208" y1="21.5392" x2="7.5692" y2="21.5519" width="0.3048" layer="1"/>
-<wire x1="7.5692" y1="21.5519" x2="10.7823" y2="18.3388" width="0.3048" layer="1"/>
-<wire x1="10.7823" y1="18.3388" x2="10.8204" y2="18.3261" width="0.3048" layer="1"/>
-<via x="10.8204" y="18.3261" extent="1-16" drill="0.6"/>
-<wire x1="10.8204" y1="18.3261" x2="11.4046" y2="17.7419" width="0.3048" layer="16"/>
-<wire x1="11.4046" y1="17.7419" x2="11.4046" y2="11.6459" width="0.3048" layer="16"/>
+<via x="11.4046" y="21.5011" extent="1-16" drill="0.6"/>
+<wire x1="11.4046" y1="21.5011" x2="11.4046" y2="11.6459" width="0.3048" layer="16"/>
 <via x="11.4046" y="11.6459" extent="1-16" drill="0.6"/>
 <wire x1="11.4046" y1="11.6459" x2="11.4046" y2="11.3919" width="0.3048" layer="1"/>
 <wire x1="11.4046" y1="11.3919" x2="12.197" y2="10.6122" width="0.3048" layer="1"/>
 <wire x1="12.197" y1="10.6122" x2="12.197" y2="7.0416" width="0.3048" layer="1"/>
+<wire x1="8.8013" y1="21.54" x2="8.8013" y2="21.5519" width="0.3048" layer="1"/>
+<wire x1="8.8013" y1="21.54" x2="8.8013" y2="21.5011" width="0.3048" layer="1"/>
+<wire x1="8.8013" y1="21.5011" x2="11.4046" y2="21.5011" width="0.3048" layer="1"/>
 </signal>
 <signal name="N$25">
@@
 <wire x1="3.1115" y1="28.4353" x2="3.9878" y2="29.3116" width="0.3048" layer="1"/>
 <wire x1="3.9878" y1="29.3116" x2="7.2263" y2="29.3116" width="0.3048" layer="1"/>
-<wire x1="7.2263" y1="29.3116" x2="8.8265" y2="27.7114" width="0.3048" layer="1"/>
-<wire x1="8.8265" y1="27.7114" x2="8.8265" y2="22.8473" width="0.3048" layer="1"/>
-<wire x1="8.8265" y1="22.8473" x2="13.6525" y2="18.0213" width="0.3048" layer="1"/>
-<wire x1="13.6525" y1="18.0213" x2="13.6525" y2="12.446" width="0.3048" layer="1"/>
+<wire x1="7.2263" y1="29.3116" x2="10.5029" y2="29.2862" width="0.3048" layer="1"/>
+<wire x1="10.5029" y1="29.2862" x2="13.6525" y2="29.2862" width="0.3048" layer="1"/>
+<wire x1="13.6525" y1="29.2862" x2="13.6525" y2="12.446" width="0.3048" layer="1"/>
 <via x="13.6525" y="12.446" extent="1-16" drill="0.6"/>
 <wire x1="13.6525" y1="12.446" x2="13.6525" y2="11.8745" width="0.3048" layer="16"/>

Commit message: aa
Parts:
- removed S1: (no value), switch-dil:SD4-01
- added S2: DTSM-3, switch-tact:DTSM-3
- moved U$1 29.5 mm to (-5.19, 19.5), flipped to the bottom
- moved JP2 11.6 mm to (6.87, 23.3), flipped to the bottom, turned to 180 degrees
- moved C2 5.47 mm to (1.64, 17.8)
- moved C1 4.85 mm to (1.83, 12.6)
- moved U$2 3.03 mm to (7.09, 11.7)
Connections:
- net GND: now also S2.1; no longer S1.1
- net N$28: now also S2.2, U$2.3; no longer S1.2, U$2.8
Routing:
- net N$28: track 35.3 -> 0.00 mm, vias 2 -> 0
- net N$23: track 17.4 -> 0.00 mm, vias 2 -> 0
- net N$16: track 15.4 -> 0.00 mm
- net N$25: track 10.2 -> 24.7 mm
- net N$20: track 13.4 -> 0.00 mm
- net N$22: track 12.6 -> 0.00 mm
- net GND: track 15.0 -> 2.49 mm, vias 2 -> 1
- net N$19: track 8.40 -> 17.4 mm
- net N$12: track 8.73 -> 0.00 mm
- net N$18: track 7.33 -> 15.3 mm
- net N$21: track 6.91 -> 0.00 mm
- net N$33: track 17.6 -> 13.9 mm
- net N$34: track 25.6 -> 22.4 mm
- net VDD: track 46.3 -> 43.2 mm, vias 2 -> 1
Other:
- board size 14.9 x 30.5 mm -> 14.1 x 26 mm

Commit message: a
Parts:
- moved C1 0.75 mm to (1.80, 11.8)
Routing:
- net N$28: track 0.00 -> 13.7 mm, vias 0 -> 2
- net GND: track 2.49 -> 12.5 mm, vias 1 -> 4
- net N$21: track 0.00 -> 8.03 mm, vias 0 -> 1
- net N$20: track 0.00 -> 7.91 mm, vias 0 -> 1
- net N$23: track 0.00 -> 7.65 mm, vias 0 -> 1
- net N$12: track 0.00 -> 5.44 mm, vias 0 -> 1
- net N$16: track 0.00 -> 4.37 mm, vias 0 -> 1
- net N$22: track 0.00 -> 3.48 mm, vias 0 -> 1
- net N$34: track 22.4 -> 25.1 mm
Other:
- board size 14.1 x 26 mm -> 14.1 x 25.3 mm

Commit message: aa
Parts:
- added S1, S3: DTSM-3, switch-tact:DTSM-3
- moved S2 0.96 mm to (7.39, 19.4)
- moved U$2 0.61 mm to (6.48, 11.7)
- moved C1 0.27 mm to (1.54, 11.8)
- moved C2 0.25 mm to (1.38, 17.8)
- moved JP2 0.14 mm to (6.87, 23.5)
Connections:
- new net N$1: JP1.3, S3.2
- new net N$2: JP1.5, S1.2
- net GND: now also S1.1, S3.1
Routing:
- net N$1: track 0.00 -> 17.9 mm, vias 0 -> 1
- net N$2: track 0.00 -> 13.3 mm, vias 0 -> 1
- net N$34: track 25.1 -> 31.2 mm
- net GND: track 12.5 -> 16.5 mm, vias 4 -> 5
- net VDD: track 43.0 -> 45.7 mm
- net N$28: track 13.7 -> 15.3 mm
- net N$18: track 15.3 -> 16.3 mm
- net N$33: track 13.8 -> 13.1 mm
- net N$20: track 7.91 -> 7.29 mm
- net N$22: track 3.48 -> 4.09 mm
- net N$23: track 7.65 -> 8.24 mm
- net N$16: track 4.37 -> 4.96 mm
Other:
- board size 14.1 x 25.3 mm -> 14.2 x 25.3 mm

Commit message: a
Connections:
- net N$28: now also U$2.2; no longer U$2.3
Routing:
- net N$28: track 15.3 -> 16.2 mm
Changed lines of the file:
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@@
 </signal>
 <signal name="N$28">
-<contactref element="U$2" pad="3"/>
 <contactref element="S2" pad="2"/>
 <wire x1="4.6914" y1="19.3802" x2="6.4262" y2="19.3802" width="0.3048" layer="1"/>
@@
 <wire x1="6.4262" y1="17.3609" x2="4.9657" y2="17.3609" width="0.3048" layer="16"/>
 <wire x1="4.9657" y1="17.3609" x2="4.9657" y2="10.1981" width="0.3048" layer="16"/>
-<wire x1="4.8553" y1="8.1211" x2="4.8514" y2="9.353" width="0.3048" layer="1"/>
-<wire x1="4.8514" y1="9.353" x2="5.4356" y2="9.8044" width="0.3048" layer="1"/>
+<wire x1="4.8514" y1="9.7594" x2="5.4356" y2="9.8044" width="0.3048" layer="1"/>
 <via x="5.4356" y="9.8044" extent="1-16" drill="0.6"/>
 <wire x1="5.4356" y1="9.8044" x2="4.9657" y2="10.1981" width="0.3048" layer="16"/>
+<contactref element="U$2" pad="2"/>
+<wire x1="4.8514" y1="9.7594" x2="4.2053" y2="9.7594" width="0.3048" layer="1"/>
+<wire x1="4.2053" y1="9.7594" x2="4.2053" y2="8.1211" width="0.3048" layer="1"/>
 </signal>
 <signal name="N$33">
