File: Hardware/SchemasBoard/raspi.brd (EAGLE design)
At the start: 14.2 x 25.3 mm, 9 parts

Commit message: aaa
Parts:
- removed JP2: Prog, pinhead:1X05
- added U$3: PROGRAMMINGHEADERDIP, rfm70:PROGHEADER
- moved S2 0.20 mm to (7.19, 19.4)
Connections:
- net GND: now also U$3.GND; no longer JP2.3
- net N$18: now also U$3.PGD; no longer JP2.4
- net N$19: now also U$3.PGC; no longer JP2.5
- net N$25: now also U$3.MCLR; no longer JP2.1
- net VDD: now also U$3.VDD; no longer JP2.2
Routing:
- net N$18: track 16.3 -> 14.9 mm
- net N$19: track 17.1 -> 16.3 mm
Other:
- board size 14.2 x 25.3 mm -> 14.2 x 24.8 mm
Changed lines of the file:
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@@
 <plain>
 <wire x1="0" y1="0" x2="14.1861" y2="0" width="0" layer="20"/>
-<wire x1="14.1861" y1="0" x2="14.148" y2="25.2757" width="0" layer="20"/>
-<wire x1="14.148" y1="25.2757" x2="0" y2="25.2757" width="0" layer="20"/>
-<wire x1="0" y1="25.2757" x2="0" y2="0" width="0" layer="20"/>
+<wire x1="14.1861" y1="0" x2="14.1861" y2="24.8185" width="0" layer="20"/>
+<wire x1="14.1861" y1="24.8185" x2="0" y2="24.8185" width="0" layer="20"/>
+<wire x1="0" y1="24.8185" x2="0" y2="0" width="0" layer="20"/>
 </plain>
 <attributes>
@@
 <element name="U$1" library="rfm70" package="RFM70" value="RFM70" x="-5.1943" y="19.4818" rot="MR270"/>
 <element name="U$2" library="microchip" package="SSOP20" value="PIC16F690" x="6.4803" y="11.7461"/>
-<element name="JP2" library="pinhead" package="1X05" value="Prog" x="6.866" y="23.4696" rot="MR180"/>
 <element name="JP1" library="pinhead" package="2X05" value="Raspi" x="7.0866" y="3.0005" rot="R180"/>
 <element name="C1" library="rcl" package="C0805" value="" x="1.5367" y="11.811" rot="R90"/>
 <element name="C2" library="resistor" package="SMC_A" value="" x="1.3843" y="17.78" rot="R90"/>
-<element name="S2" library="switch-tact" package="DTSM-3" value="DTSM-3" x="7.3914" y="19.3802" rot="R180"/>
+<element name="S2" library="switch-tact" package="DTSM-3" value="DTSM-3" x="7.1882" y="19.3802" rot="R180"/>
 <element name="S1" library="switch-tact" package="DTSM-3" value="DTSM-3" x="12.2936" y="9.8806" rot="R90"/>
-<element name="S3" library="switch-tact" package="DTSM-3" value="DTSM-3" x="12.3063" y="17.6911" rot="R270"/>
+<element name="S3" library="switch-tact" package="DTSM-3" value="DTSM-3" x="12.2809" y="17.6911" rot="R270"/>
+<element name="U$3" library="rfm70" package="PROGHEADER" value="PROGRAMMINGHEADERDIP" x="5.8039" y="23.0251"/>
 </elements>
 <signals>
@@
 <contactref element="U$2" pad="20"/>
 <contactref element="U$1" pad="GND"/>
-<contactref element="JP2" pad="3"/>
 <contactref element="JP1" pad="6"/>
 <polygon width="0.254" layer="16">
@@
 <contactref element="C2" pad="-"/>
 <contactref element="S2" pad="1"/>
-<wire x1="10.0914" y1="19.3802" x2="7.6327" y2="19.3929" width="0.3048" layer="1"/>
+<wire x1="9.8882" y1="19.3802" x2="7.6327" y2="19.3929" width="0.3048" layer="1"/>
 <wire x1="7.6327" y1="19.3929" x2="7.4041" y2="19.6596" width="0.3048" layer="1"/>
 <via x="7.4041" y="19.6596" extent="1-16" drill="0.6"/>
@@
 <via x="11.9761" y="9.1186" extent="1-16" drill="0.6"/>
 <wire x1="11.9761" y1="9.1186" x2="12.319" y2="9.6139" width="0.3048" layer="16"/>
-<wire x1="12.3063" y1="20.3911" x2="11.5341" y2="20.3911" width="0.3048" layer="1"/>
-<wire x1="11.5341" y1="20.3911" x2="10.0914" y2="19.3802" width="0.3048" layer="1"/>
+<wire x1="12.2809" y1="20.3911" x2="11.5341" y2="20.3911" width="0.3048" layer="1"/>
+<wire x1="11.5341" y1="20.3911" x2="9.8882" y2="19.3802" width="0.3048" layer="1"/>
+<contactref element="U$3" pad="GND"/>
+<contactref element="U$3" pad="GND"/>
 </signal>
 <signal name="N$12">
@@
 <contactref element="U$2" pad="1"/>
 <contactref element="U$1" pad="VDD"/>
-<contactref element="JP2" pad="2"/>
 <contactref element="U$2" pad="1"/>
 <contactref element="C1" pad="1"/>
 <contactref element="C2" pad="+"/>
-<wire x1="4.326" y1="23.4696" x2="4.326" y2="21.4296" width="0.3048" layer="16"/>
-<wire x1="4.326" y1="21.4296" x2="6.28015" y2="19.47545" width="0.3048" layer="16"/>
+<wire x1="3.8039" y1="21.9517" x2="6.28015" y2="19.47545" width="0.3048" layer="16"/>
 <wire x1="6.28015" y1="19.47545" x2="7.4803" y2="18.2753" width="0.3048" layer="16"/>
 <wire x1="7.4803" y1="18.2753" x2="9.0992" y2="18.2753" width="0.3048" layer="16"/>
@@
 <wire x1="2.8321" y1="16.7894" x2="3.0861" y2="16.8148" width="0.3048" layer="16"/>
 <wire x1="3.0861" y1="16.8148" x2="6.28015" y2="19.47545" width="0.3048" layer="16"/>
+<contactref element="U$3" pad="VDD"/>
+<contactref element="U$3" pad="VDD"/>
+<wire x1="3.8039" y1="23.2751" x2="3.8039" y2="21.9517" width="0.3048" layer="16"/>
 </signal>
 <signal name="N$18">
 <contactref element="U$2" pad="19"/>
-<contactref element="JP2" pad="4"/>
-<wire x1="9.406" y1="23.4696" x2="9.4488" y2="23.3299" width="0.3048" layer="1"/>
-<wire x1="9.4488" y1="23.3299" x2="9.4488" y2="21.2344" width="0.3048" layer="1"/>
-<wire x1="9.4488" y1="21.2344" x2="2.7178" y2="21.2344" width="0.3048" layer="1"/>
-<wire x1="2.7178" y1="21.2344" x2="2.7178" y2="17.6911" width="0.3048" layer="1"/>
-<wire x1="2.7178" y1="17.6911" x2="4.1926" y2="17.6784" width="0.3048" layer="1"/>
-<wire x1="4.1926" y1="17.6784" x2="4.2053" y2="15.3711" width="0.3048" layer="1"/>
+<wire x1="7.8486" y1="21.2344" x2="7.7724" y2="21.2344" width="0.3048" layer="1"/>
+<wire x1="7.7724" y1="21.2344" x2="2.5654" y2="21.2344" width="0.3048" layer="1"/>
+<wire x1="2.5654" y1="21.2344" x2="2.5654" y2="17.6657" width="0.3048" layer="1"/>
+<wire x1="2.5654" y1="17.6657" x2="4.1926" y2="17.653" width="0.3048" layer="1"/>
+<wire x1="4.1926" y1="17.653" x2="4.2053" y2="15.3711" width="0.3048" layer="1"/>
+<contactref element="U$3" pad="PGD"/>
+<wire x1="7.8486" y1="23.3198" x2="7.8486" y2="21.3106" width="0.3048" layer="1"/>
+<wire x1="7.8486" y1="21.3106" x2="7.7724" y2="21.2344" width="0.3048" layer="1"/>
+<wire x1="7.8486" y1="23.3198" x2="7.8039" y2="23.2751" width="0" layer="19" extent="1-1"/>
 </signal>
 <signal name="N$19">
 <contactref element="U$2" pad="18"/>
-<contactref element="JP2" pad="5"/>
-<wire x1="11.946" y1="23.4696" x2="12.0142" y2="23.3299" width="0.3048" layer="1"/>
-<wire x1="12.0142" y1="23.3299" x2="10.1092" y2="20.5867" width="0.3048" layer="1"/>
-<wire x1="10.1092" y1="20.5867" x2="3.2893" y2="20.5867" width="0.3048" layer="1"/>
-<wire x1="3.2893" y1="20.5867" x2="3.2766" y2="18.2118" width="0.3048" layer="1"/>
-<wire x1="3.2766" y1="18.2118" x2="4.8553" y2="18.2118" width="0.3048" layer="1"/>
+<wire x1="9.8298" y1="20.5867" x2="3.0988" y2="20.5867" width="0.3048" layer="1"/>
+<wire x1="3.0988" y1="20.5867" x2="3.0861" y2="18.2118" width="0.3048" layer="1"/>
+<wire x1="3.0861" y1="18.2118" x2="4.8553" y2="18.2118" width="0.3048" layer="1"/>
 <wire x1="4.8553" y1="18.2118" x2="4.8553" y2="15.3711" width="0.3048" layer="1"/>
+<contactref element="U$3" pad="PGC"/>
+<wire x1="9.8298" y1="23.1775" x2="9.8298" y2="20.5867" width="0.3048" layer="1"/>
+<wire x1="9.8298" y1="23.1775" x2="9.8039" y2="23.0251" width="0" layer="19" extent="1-1"/>
 </signal>
 <signal name="N$16">
@@
 <signal name="N$25">
 <contactref element="U$2" pad="4"/>
-<contactref element="JP2" pad="1"/>
-<wire x1="1.786" y1="23.4696" x2="0.3429" y2="23.4696" width="0.3048" layer="1"/>
-<wire x1="0.3429" y1="23.4696" x2="0.3429" y2="6.9596" width="0.3048" layer="1"/>
-<wire x1="0.3429" y1="6.9596" x2="5.518" y2="6.9596" width="0.3048" layer="1"/>
+<wire x1="0.2286" y1="22.8854" x2="0.2159" y2="6.9596" width="0.3048" layer="1"/>
+<wire x1="0.2159" y1="6.9596" x2="5.518" y2="6.9596" width="0.3048" layer="1"/>
 <wire x1="5.518" y1="6.9596" x2="5.5053" y2="8.1211" width="0.3048" layer="1"/>
+<contactref element="U$3" pad="MCLR"/>
+<wire x1="1.8039" y1="23.0251" x2="0.508" y2="23.0251" width="0.3048" layer="1"/>
+<wire x1="0.508" y1="23.0251" x2="0.2286" y2="22.8854" width="0.3048" layer="1"/>
 </signal>
 <signal name="N$28">
 <contactref element="S2" pad="2"/>
-<wire x1="4.6914" y1="19.3802" x2="6.4262" y2="19.3802" width="0.3048" layer="1"/>
+<wire x1="4.4882" y1="19.3802" x2="6.4262" y2="19.3802" width="0.3048" layer="1"/>
 <wire x1="6.4262" y1="19.3802" x2="6.4262" y2="17.3609" width="0.3048" layer="1"/>
 <via x="6.4262" y="17.3609" extent="1-16" drill="0.6"/>
@@
 <contactref element="S3" pad="2"/>
 <contactref element="JP1" pad="3"/>
-<wire x1="12.3063" y1="14.9911" x2="12.3063" y2="16.5608" width="0.3048" layer="1"/>
+<wire x1="12.2809" y1="14.9911" x2="12.3063" y2="16.5608" width="0.3048" layer="1"/>
 <wire x1="12.3063" y1="16.5608" x2="12.3444" y2="16.5989" width="0.3048" layer="1"/>
 <via x="12.3444" y="16.5989" extent="1-16" drill="0.6"/>

Commit message: aaa
Parts:
- moved S3 13.2 mm to (3.87, 7.57), turned to 180 degrees
- moved C1 12.2 mm to (13.3, 15.1), flipped to the bottom, turned to 270 degrees
- moved C2 11.9 mm to (13.2, 19.5), flipped to the bottom
- moved S2 8.26 mm to (12.9, 13.4), turned to 90 degrees
- moved U$1 8.14 mm to (-5.82, 11.4), flipped to the top, turned to 90 degrees
- moved U$2 4.29 mm to (7.60, 15.9), flipped to the bottom
- moved U$3 2.81 mm to (8.34, 24.2), turned to 180 degrees
- moved S1 2.41 mm to (11.7, 7.56), turned to 0 degrees
- moved JP1 1.92 mm to (9.00, 2.91)
Routing:
- net GND: track 16.5 -> 43.6 mm, vias 5 -> 1
- net N$28: track 16.4 -> 7.20 mm, vias 2 -> 1
- net N$25: track 24.0 -> 15.1 mm, vias 0 -> 2
- net N$18: track 14.9 -> 6.00 mm
- net N$19: track 16.3 -> 8.03 mm
- net VDD: track 45.7 -> 39.0 mm
- net N$2: track 13.3 -> 6.76 mm, vias 1 -> 0
- net N$21: track 7.74 -> 3.84 mm
- net N$34: track 31.2 -> 27.6 mm, vias 0 -> 1
- net N$16: track 4.96 -> 8.21 mm
- net N$1: track 17.9 -> 20.7 mm, vias 1 -> 0
- net N$33: track 13.1 -> 15.7 mm
- net N$23: track 8.24 -> 10.7 mm
- net N$22: track 4.09 -> 6.45 mm
- added copper zone on layer 1, net VDD
Other:
- board size 14.2 x 24.8 mm -> 15.7 x 25.9 mm
