File: Hardware/SchemasBoard/tempSensorAAABat.sch (EAGLE design)
At the start: 9 parts, among them IC1 DS1820

Commit message: aaa
Parts:
- removed U$4: CR2032, rfm70:CR2032
- added GND, VDD: (no value), wirepad:SMD5
Connections:
- net N$5: now also VDD.P; no longer U$4.VDD
- net VD: now also GND.P; no longer U$4.GND
Other:
- moved on the sheet: C1

Commit message: aaa
Connections:
- removed net N$4: C2.+, U$1.VDD, U$2.RC1/AN5/C12IN1-, U$2.RC3/AN7C12IN3-/P1C, U$2.RC4/C2OUT/P1B, U$2.RC6/AN8/SS
- removed net N$5: C1.1, R1.2, U$2.VDD, U$3.VDD, VDD.P
- new net N$7: C1.1, C2.+, R1.2, U$1.VDD, U$2.VDD, U$3.VDD, VDD.P

Commit message: fghf
Connections:
- net N$7 renamed VDD
- net VD renamed GND
Changed lines of the file:
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@@
 </busses>
 <nets>
-<net name="VD" class="0">
+<net name="GND" class="0">
 <segment>
 <wire x1="132.08" y1="30.48" x2="147.32" y2="30.48" width="0.1524" layer="91"/>
@@
 </segment>
 </net>
-<net name="N$7" class="0">
+<net name="VDD" class="0">
 <segment>
 <pinref part="U$1" gate="G$1" pin="VDD"/>
